File: eagle-schematics/themis-v1/Mixer 2164D/V2164MIXER v2.sch (EAGLE design)
At the start: 32 parts

Commit message: checked connections
Connections:
- new net N$1: CONN_CURRENT_SUMMING.8
- net 2164_OUT3: no longer CONN_CURRENT_SUMMING.8
Changed lines of the file:
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@@
 <net name="2164_OUT3" class="0">
 <segment>
-<pinref part="CONN_CURRENT_SUMMING" gate="G$1" pin="8"/>
-<wire x1="337.82" y1="68.58" x2="332.74" y2="68.58" width="0.1524" layer="91"/>
-<wire x1="332.74" y1="68.58" x2="332.74" y2="-7.62" width="0.1524" layer="91"/>
 <pinref part="MIXER" gate="G$5" pin="I_OUT"/>
 <wire x1="332.74" y1="-7.62" x2="320.04" y2="-7.62" width="0.1524" layer="91"/>
@@
 </segment>
 </net>
+<net name="N$1" class="0">
+<segment>
+<pinref part="CONN_CURRENT_SUMMING" gate="G$1" pin="8"/>
+<wire x1="337.82" y1="68.58" x2="332.74" y2="68.58" width="0.1524" layer="91"/>
+</segment>
+</net>
