File: eagle-schematics/themis-v1/Mixer 2164D/V2164MIXER v2.brd (EAGLE design)
At the start: 74 x 44.4 mm, 33 parts

Commit message: Improved schematics, added analog chips library
Routing:
- net AGND: track 202.8 -> 246.1 mm
- net +15V: track 80.8 -> 79.7 mm
- net -15V: track 72.9 -> 72.2 mm
Other:
- board size 74 x 44.4 mm -> 80 x 50.4 mm
Changed lines of the file:
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@@
 <?xml version="1.0" encoding="utf-8"?>
 <!DOCTYPE eagle SYSTEM "eagle.dtd">
-<eagle version="9.3.2">
+<eagle version="9.5.0">
 <drawing>
 <settings>
@@
 <setting verticaltext="up"/>
 </settings>
-<grid distance="25" unitdist="mil" unit="mil" style="lines" multiple="1" display="no" altdistance="5" altunitdist="mil" altunit="mil"/>
+<grid distance="1" unitdist="mm" unit="mm" style="lines" multiple="1" display="yes" altdistance="5" altunitdist="mil" altunit="mil"/>
 <layers>
 <layer number="1" name="Top" color="4" fill="1" visible="yes" active="yes"/>
@@
 <layer number="45" name="Holes" color="7" fill="1" visible="no" active="yes"/>
 <layer number="46" name="Milling" color="3" fill="1" visible="no" active="yes"/>
-<layer number="47" name="Measures" color="7" fill="1" visible="no" active="yes"/>
+<layer number="47" name="Measures" color="7" fill="1" visible="yes" active="yes"/>
 <layer number="48" name="Document" color="7" fill="1" visible="no" active="yes"/>
 <layer number="49" name="Reference" color="7" fill="1" visible="no" active="yes"/>
@@
 <board>
 <plain>
-<wire x1="1.905" y1="32.385" x2="75.87" y2="32.385" width="0" layer="20"/>
-<wire x1="75.87" y1="32.385" x2="75.87" y2="76.825" width="0" layer="20"/>
-<wire x1="75.87" y1="76.825" x2="1.905" y2="76.825" width="0" layer="20"/>
-<wire x1="1.905" y1="76.825" x2="1.905" y2="32.385" width="0" layer="20"/>
-<text x="21.717" y="74.676" size="1.27" layer="1">THeMiS Mixer v2 [TOP]</text>
-<text x="43.434" y="74.676" size="1.27" layer="16" rot="MR0">THeMiS Mixer v2 [BOTTOM]</text>
+<wire x1="-1.095" y1="28.385" x2="78.87" y2="28.385" width="0" layer="20"/>
+<wire x1="78.87" y1="28.385" x2="78.87" y2="78.825" width="0" layer="20"/>
+<wire x1="78.87" y1="78.825" x2="-1.095" y2="78.825" width="0" layer="20"/>
+<wire x1="-1.095" y1="78.825" x2="-1.095" y2="28.385" width="0" layer="20"/>
+<text x="21.717" y="75.676" size="1.27" layer="1">THeMiS Mixer v2 [TOP]</text>
+<text x="43.434" y="75.676" size="1.27" layer="16" rot="MR0">THeMiS Mixer v2 [BOTTOM]</text>
+<dimension x1="-1" y1="34" x2="-1" y2="74" x3="-9" y3="54" textsize="1.778" layer="47"/>
+<dimension x1="0" y1="74" x2="0" y2="79" x3="-3" y3="76.5" textsize="1.778" layer="47"/>
+<dimension x1="-1" y1="34" x2="-1" y2="29" x3="-2" y3="31.5" textsize="1.778" layer="47"/>
+<dimension x1="4" y1="74" x2="74" y2="74" x3="39" y3="84" textsize="1.778" layer="47"/>
+<dimension x1="4" y1="84" x2="-1" y2="84" x3="1.5" y3="86" textsize="1.778" layer="47"/>
+<dimension x1="74" y1="84" x2="79" y2="84" x3="76.5" y3="86" textsize="1.778" layer="47"/>
 </plain>
 <attributes>
@@
 <wire x1="40.005" y1="68.58" x2="50.8" y2="68.58" width="0.6096" layer="16"/>
 <wire x1="50.8" y1="68.58" x2="51.435" y2="69.215" width="0.6096" layer="16"/>
-<wire x1="53.34" y1="41.275" x2="53.34" y2="45.72" width="0.508" layer="1"/>
-<wire x1="53.34" y1="45.72" x2="51.435" y2="47.625" width="0.508" layer="1"/>
-<wire x1="45.72" y1="41.275" x2="53.34" y2="41.275" width="0.508" layer="1"/>
+<wire x1="51.435" y1="47.625" x2="53.34" y2="45.72" width="0.508" layer="1"/>
+<wire x1="51.435" y1="41.275" x2="45.72" y2="41.275" width="0.508" layer="1"/>
 <wire x1="51.435" y1="47.625" x2="51.435" y2="60.96" width="0.6096" layer="1"/>
 <wire x1="51.435" y1="60.96" x2="48.895" y2="63.5" width="0.6096" layer="1"/>
 <wire x1="48.895" y1="63.5" x2="40.005" y2="63.5" width="0.6096" layer="1"/>
 <wire x1="40.005" y1="63.5" x2="37.465" y2="66.04" width="0.6096" layer="1"/>
+<wire x1="53.34" y1="43.18" x2="51.435" y2="41.275" width="0.508" layer="1"/>
+<wire x1="53.34" y1="45.72" x2="53.34" y2="43.18" width="0.508" layer="1"/>
 </signal>
 <signal name="-15V">
@@
 <wire x1="49.53" y1="66.04" x2="50.8" y2="66.04" width="0.6096" layer="16"/>
 <wire x1="50.8" y1="66.04" x2="53.975" y2="69.215" width="0.6096" layer="16"/>
-<wire x1="62.9094" y1="43.2244" x2="62.9094" y2="60.2806" width="0.508" layer="1"/>
-<wire x1="62.9094" y1="43.2244" x2="56.515" y2="36.83" width="0.508" layer="1"/>
-<wire x1="62.9094" y1="60.2806" x2="57.15" y2="66.04" width="0.6096" layer="1"/>
-<wire x1="57.15" y1="66.04" x2="46.355" y2="66.04" width="0.6096" layer="1"/>
+<wire x1="46.355" y1="66.04" x2="48.26" y2="66.04" width="0.6096" layer="1"/>
+<wire x1="58.42" y1="53.975" x2="61.595" y2="50.8" width="0.508" layer="1"/>
+<wire x1="58.42" y1="37.465" x2="57.785" y2="36.83" width="0.508" layer="1"/>
+<wire x1="57.785" y1="36.83" x2="56.515" y2="36.83" width="0.508" layer="1"/>
+<wire x1="58.42" y1="64.135" x2="58.42" y2="53.975" width="0.508" layer="1"/>
+<wire x1="61.595" y1="50.8" x2="61.595" y2="48.26" width="0.508" layer="1"/>
+<wire x1="61.595" y1="48.26" x2="58.42" y2="45.085" width="0.508" layer="1"/>
+<wire x1="58.42" y1="45.085" x2="58.42" y2="37.465" width="0.508" layer="1"/>
+<wire x1="48.26" y1="66.04" x2="49.53" y2="64.77" width="0.508" layer="1"/>
+<wire x1="57.785" y1="64.77" x2="58.42" y2="64.135" width="0.508" layer="1"/>
+<wire x1="49.53" y1="64.77" x2="57.785" y2="64.77" width="0.508" layer="1"/>
 </signal>
 <signal name="2164_IN3">
@@
 <contactref element="CONN_IN" pad="2"/>
 <polygon width="0.254" layer="1" isolate="1.016">
-<vertex x="1.905" y="76.835"/>
-<vertex x="75.565" y="76.835"/>
-<vertex x="75.565" y="33.02"/>
-<vertex x="1.905" y="33.02"/>
+<vertex x="-1.095" y="78.835"/>
+<vertex x="78.565" y="78.835"/>
+<vertex x="78.565" y="29.02"/>
+<vertex x="-1.095" y="29.02"/>
 </polygon>
 <polygon width="0.254" layer="16" isolate="1.016">
-<vertex x="1.905" y="76.835"/>
-<vertex x="75.565" y="76.835"/>
-<vertex x="75.565" y="33.02"/>
-<vertex x="1.905" y="33.02"/>
+<vertex x="-1.095" y="78.835"/>
+<vertex x="78.565" y="78.835"/>
+<vertex x="78.565" y="29.02"/>
+<vertex x="-1.095" y="29.02"/>
 </polygon>
 <contactref element="RLOAD" pad="2"/>
@@
 <wire x1="69.215" y1="53.34" x2="67.945" y2="54.61" width="0.6096" layer="16"/>
 <wire x1="69.215" y1="45.72" x2="69.215" y2="53.34" width="0.6096" layer="16"/>
-<wire x1="67.945" y1="62.23" x2="60.96" y2="69.215" width="0.6096" layer="16"/>
+<wire x1="67.945" y1="62.23" x2="65.0875" y2="65.0875" width="0.6096" layer="16"/>
+<wire x1="65.0875" y1="65.0875" x2="60.96" y2="69.215" width="0.6096" layer="16"/>
 <wire x1="60.96" y1="69.215" x2="59.055" y2="69.215" width="0.6096" layer="16"/>
 <wire x1="37.465" y1="41.86384375" x2="37.465" y2="37.465" width="0.508" layer="16"/>
@@
 <wire x1="49.53" y1="74.295" x2="56.515" y2="74.295" width="0.6096" layer="16"/>
 <wire x1="56.515" y1="74.295" x2="59.055" y2="71.755" width="0.6096" layer="16"/>
-<via x="6.985" y="72.39" extent="1-16" drill="1.016" shape="square"/>
-<via x="6.985" y="37.465" extent="1-16" drill="1.016" shape="square"/>
-<via x="71.12" y="37.465" extent="1-16" drill="1.016" shape="square"/>
-<via x="71.12" y="72.39" extent="1-16" drill="1.016" shape="square"/>
+<via x="4" y="74" extent="1-16" drill="1.016" shape="square"/>
+<via x="4" y="34" extent="1-16" drill="1.016" shape="square"/>
+<via x="74" y="34" extent="1-16" drill="1.016" shape="square"/>
+<via x="74" y="74" extent="1-16" drill="1.016" shape="square"/>
+<wire x1="74" y1="74" x2="65.0875" y2="65.0875" width="0.4" layer="16"/>
+<wire x1="66.04" y1="38.735" x2="70.775" y2="34" width="0.4" layer="16"/>
+<wire x1="70.775" y1="34" x2="74" y2="34" width="0.4" layer="16"/>
+<wire x1="10.16" y1="45.085" x2="4" y2="38.925" width="0.4" layer="16"/>
+<wire x1="4" y1="38.925" x2="4" y2="34" width="0.4" layer="16"/>
+<wire x1="4" y1="74" x2="4" y2="69" width="0.4" layer="16"/>
+<wire x1="4" y1="69" x2="5.08" y2="67.92" width="0.4" layer="16"/>
+<wire x1="5.08" y1="67.92" x2="5.08" y2="67.31" width="0.4" layer="16"/>
 </signal>
 <signal name="N$11">

Commit message: New version of DAC board based on AD5391 chip
Parts:
- removed CONN_CURRENT_SUMMING1, CONN_IN: (no value), con-lstb:MA04-2
- removed RLOAD: 27k, rcl:0204/7
- removed TP_RLOAD: (no value), 6P1_EVB:TESTPOINT_63
- added CONN_INPUT: (no value), con-lstb:MA04-1
- added CONN_IOUT, CONN_VOUT: (no value), con-lstb:MA03-1
- R1, RSTAB1: device rcl:0207/10 -> rcl:0204/7
- R2, RSTAB2: device rcl:0204/7 -> rcl:0207/10
- moved RSTAB1 9.61 mm to (21.6, 52.1)
- moved RSTAB2 9.61 mm to (22.9, 42.5)
- moved R1 8.98 mm to (21.6, 55.2)
- moved R2 8.98 mm to (22.9, 46.4)
- moved R3 6.98 mm to (21.6, 65.4)
- moved R4 6.98 mm to (21.6, 58.4)
- moved RSTAB3 6.98 mm to (21.6, 68.6)
- moved RSTAB4 6.98 mm to (21.6, 61.6)
- moved CIN3 6.35 mm to (12.7, 64.1)
- moved CIN4 6.35 mm to (12.7, 57.8)
- moved CIN1 6.35 mm to (12.7, 54.6)
- moved CIN2 6.35 mm to (12.7, 48.3)
- moved CSTAB1 6.35 mm to (12.7, 51.4)
- moved CSTAB2 6.35 mm to (12.7, 45.1)
- moved CSTAB3 6.35 mm to (12.7, 67.3)
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Connections:
- removed net N$1: CIN1.1, CONN_IN.1
- removed net N$2: CIN2.1, CONN_IN.3
- removed net N$22: RLOAD.1, TP_RLOAD.P$1
- removed net N$3: CIN4.1, CONN_IN.7
- removed net N$4: CIN3.1, CONN_IN.5
- new net IN1: CIN1.1, CONN_INPUT.2
- new net IN2: CIN2.1, CONN_INPUT.1
- new net IN3: CIN3.1, CONN_INPUT.4
- new net IN4: CIN4.1, CONN_INPUT.3
- net 2164_IN1: now also MIXER.2; no longer MIXER.7
- net 2164_IN2: now also MIXER.7; no longer MIXER.2
- net 2164_IN3: now also MIXER.10; no longer MIXER.15
- net 2164_IN4: now also MIXER.15; no longer MIXER.10
- net AGND: no longer CONN_CURRENT_SUMMING1.2, CONN_CURRENT_SUMMING1.4, CONN_CURRENT_SUMMING1.6, CONN_CURRENT_SUMMING1.8, CONN_IN.2, CONN_IN.4, CONN_IN.6, CONN_IN.8, RLOAD.2
- net CURRENT_OUT: now also CONN_IOUT.1, CONN_IOUT.2, CONN_IOUT.3; no longer CONN_CURRENT_SUMMING1.1, CONN_CURRENT_SUMMING1.3
- net VOLTAGE_OUT: now also CONN_VOUT.1, CONN_VOUT.2, CONN_VOUT.3; no longer CONN_CURRENT_SUMMING1.5, CONN_CURRENT_SUMMING1.7
Routing:
- net AGND: track 246.1 -> 199.3 mm, vias 4 -> 3
- net 2164_IN4: track 35.3 -> 22.9 mm
- net 2164_IN3: track 22.9 -> 35.3 mm
- net 2164_IN2: track 14.2 -> 26.1 mm
- net 2164_IN1: track 26.1 -> 14.2 mm
- net CURRENT_OUT: track 15.3 -> 24.4 mm
- net VOLTAGE_OUT: track 29.7 -> 38.6 mm
- net IN3: track 0.00 -> 8.82 mm
- net IN2: track 0.00 -> 8.66 mm
- net N$3: track 7.25 -> 0.00 mm
- net N$1: track 6.61 -> 0.00 mm
- net IN4: track 0.00 -> 5.37 mm
- net IN1: track 0.00 -> 5.21 mm
- net N$4: track 3.44 -> 0.00 mm
- net N$2: track 3.17 -> 0.00 mm
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
Commit message: checked connections
Connections:
- new net N$1: CONN_CURRENT_SUMMING.8
- net 2164_OUT3: no longer CONN_CURRENT_SUMMING.8
Routing:
- net 2164_OUT3: track 17.2 -> 16.0 mm
Changed lines of the file:
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@@
 <wire x1="41.9798" y1="57.7152" x2="49.43944375" y2="57.7152" width="0.508" layer="16"/>
 <wire x1="41.275" y1="58.42" x2="41.9798" y2="57.7152" width="0.508" layer="16"/>
-<contactref element="CONN_CURRENT_SUMMING" pad="8"/>
 <wire x1="50.165" y1="57.785" x2="51.435" y2="59.055" width="0.508" layer="16"/>
 <wire x1="51.435" y1="59.055" x2="51.435" y2="60.96" width="0.508" layer="16"/>
 <wire x1="51.435" y1="60.96" x2="52.705" y2="62.23" width="0.508" layer="16"/>
-<wire x1="52.705" y1="62.23" x2="53.975" y2="62.23" width="0.508" layer="16"/>
 </signal>
 <signal name="GAIN1">
@@
 <wire x1="15.24" y1="57.785" x2="15.875" y2="58.42" width="0.6096" layer="16"/>
 </signal>
+<signal name="N$1">
+<contactref element="CONN_CURRENT_SUMMING" pad="8"/>
+</signal>
 </signals>
