File: eagle-schematics/themis-v1/VCO AS3340/VCO3340 v2.1.brd (EAGLE design)
At the start: 95.8 x 55.1 mm, 47 parts

Commit message: New version of DAC board based on AD5391 chip
Parts:
- removed CONN_OUTPUT: (no value), con-lstb:MA03-2
- added CONN_OUT: (no value), con-lstb:MA03-1
- added C_FM_LIN: 100n, rcl:C050-025X075
- added R_FM_LIN: 1M, rcl:0204/7
- added R_PD_411_IN_PULSE, R_PD_411_IN_SAW: 100k, rcl:0207/10
- added R_PD_411_IN_SYNC, R_PD_411_IN_TRI: 100k, rcl:0204/7
- C1_411: device rcl:C075-032X103 -> rcl:C050-030X075
- moved C1_411 3.17 mm to (64.1, 41.9)
- moved R3S_411 1.27 mm to (88.3, 23.5)
- moved R1_PWM 0.63 mm to (76.2, 8.89)
- renumbered C5_3340 to C_CV_FREQ_STAB, R12_3340 to R_CV_FREQ_BIAS, R13_3340 to R_CV_FREQ, R14_3340 to R_CV_FREQ_STAB
Connections:
- net PULSE_IN renamed N$51
- net SAW_IN renamed N$50
- net SAW_OUT renamed N$2
- net TRI_IN renamed N$49
- new net N$1: C_FM_LIN.1, R_FM_LIN.2
- new net N$4: C_FM_LIN.2
- net 411_IN_PULSE: now also 411.8, CONN_STM32.4, R_PD_411_IN_PULSE.2; no longer 411.9, CONN_STM32.7
- net 411_IN_SAW: now also 411.9, CONN_STM32.7, R_PD_411_IN_SAW.1; no longer 411.8, CONN_STM32.4
- net 411_IN_SYNC: now also R_PD_411_IN_SYNC.1
- net 411_IN_TRI: now also R_PD_411_IN_TRI.1
- net 5V: now also R_PD_411_IN_SAW.2
- net AGND: now also R_PD_411_IN_PULSE.1, R_PD_411_IN_SYNC.2, R_PD_411_IN_TRI.2; no longer CONN_OUTPUT.1, CONN_OUTPUT.3, CONN_OUTPUT.5
- net LINEAR_CTRL: now also R_FM_LIN.1
- net OUT: now also CONN_OUT.1, CONN_OUT.2, CONN_OUT.3; no longer CONN_OUTPUT.2, CONN_OUTPUT.4, CONN_OUTPUT.6
Routing:
- net AGND: track 449.2 -> 432.2 mm
- net 411_IN_SYNC: track 39.5 -> 46.1 mm
- net 411_IN_TRI: track 38.0 -> 43.1 mm
- net TRI_3340: track 50.7 -> 46.2 mm
- net +15V: track 183.1 -> 180.5 mm
- net 411_IN_SAW: track 18.1 -> 20.0 mm
- net PULSE_OUT: track 6.35 -> 7.62 mm
- net N$49: track 12.9 -> 13.6 mm
- net OUT: track 76.4 -> 75.8 mm
Other:
- board size 95.8 x 55.1 mm -> 95.8 x 57.6 mm
