File: eagle-schematics/themis-v1/VCO AS3340/VCO3340 v2.1.sch (EAGLE design)
At the start: 32 parts

Commit message: New version of DAC board based on AD5391 chip
Parts:
- removed CAOP: 1p, rcl:C-EU050-030X075
- removed CDEC+15V, CDEC-15V, CDEC-15VPOL: 100n, rcl:C-EU050-030X075
- removed CDEC+15VPOL: 100n, rcl:C-EU075-032X103
- removed CIN1, CIN2, CIN3, CIN4: 470n, rcl:C-EU050-030X075
- removed CONN_ALIM, CONN_CURRENT_SUMMING: (no value), con-lstb:MA04-2
- removed CONN_INPUT: (no value), con-lstb:MA04-1
- removed CONN_IOUT, CONN_ITOV, CONN_VOUT: (no value), con-lstb:MA03-1
- removed CONV_ITOV: NE5534AN, linear:NE5534AN
- removed CSTAB1, CSTAB2, CSTAB3, CSTAB4: 560p, rcl:C-EU050-030X075
- removed MIXER: SSM2164_MULTI, analog-audio-chips:SSM2164_MULTI
- removed R1, R3, R4: 27k, rcl:R-EU_0204/7
- removed R2: 27k, rcl:R-EU_0207/10
- removed RAOP: 33K, rcl:R-EU_0204/7
- removed RMODE: 8.2k, rcl:R-EU_0204/7
- removed RSTAB1, RSTAB3, RSTAB4: 470, rcl:R-EU_0204/7
- removed RSTAB2: 470, rcl:R-EU_0207/10
- added 411: ADG411N, analog-devices:ADG411N
- added C1_411: 470n, rcl:C-EU050-030X075
- added C1_SYNC3340: 1n, rcl:C-EU075-032X103
- added C2_411: 470n, rcl:C-EU075-032X103
- added C2_SYNC3340: 100n, rcl:C-EU075-032X103
- added C3_411: 470n, rcl:C-EU102-043X133
- added C4_3340: 10n, rcl:C-EU050-025X075
- added CDEC_3340A, CDEC_3340B, CDEC_411B, C_FM_LIN: 100n, rcl:C-EU050-025X075
- added CDEC_3340A1, CDEC_3340B1, CDEC_411B1: 10u, rcl:C-EU050-025X075
- added CEM3340: CEM3340, analog-audio-chips:CEM3340
- added CONN_ALIM1, CONN_ALIM2: (no value), SparkFun-Connectors:CONN_04
- added CONN_OUT: (no value), con-lstb:MA03-1
- added C_3340: 1n, rcl:C-EU050-025X075
- added C_CV_FREQ_STAB: 10n, rcl:C-EU075-032X103
- added H1, H2: MOUNT-PAD-ROUND2.8, holes:MOUNT-PAD-ROUND2.8
- added R10_3340, R_CV_FREQ_STAB: 470, rcl:R-EU_0204/7
- added R11_3340: 1.8k, rcl:R-EU_0204/7
- added R1S_411, R3S_411: 1k, rcl:R-EU_0204/7
- added R1_3340: 30k, rcl:R-EU_0204/7
- added R1_411, R2_411, R_PD_411_IN_PULSE, R_PD_411_IN_SAW: 100k, rcl:R-EU_0207/10
- added R1_PWM: 68k, rcl:R-EU_0207/12
- added R2S_411: 1k, rcl:R-EU_0207/10
- added R2_3340: 5.6k, rcl:R-EU_0204/7
- added R2_PWM: 330k, rcl:R-EU_0204/7
- added R3_3340: 820, rcl:R-EU_0204/7
- added R3_411, R_PD_411_IN_SYNC, R_PD_411_IN_TRI: 100k, rcl:R-EU_0204/7
- added R5_3340: 10k, rcl:R-EU_0204/7
- added R6_3340: 33k, rcl:R-EU_0204/7
- added R7_3340: 5.6k, rcl:R-EU_0207/10
- added R8_3340: 1.5M, rcl:R-EU_0204/7
- added R_CV_FREQ: 68k, rcl:R-EU_0204/7
- added R_CV_FREQ_BIAS: 270k, rcl:R-EU_0204/7
- added R_FM_LIN: 1M, rcl:R-EU_0204/7
- added R_SYNC: 470k, rcl:R-EU_0204/7
- added SYNC_IN, TP_PULSE, TP_SAW, TP_TRI: (no value), 6P1_EVB:TESTPOINT
- CONN_STM32: device con-lstb:MA05-1 -> con-lstb:MA08-1
Connections:
- removed net +5V: CONN_ALIM.3, CONN_ALIM.4
- removed net 2164_IN1: MIXERG$2.I_IN, R1.1, RSTAB1.1
- removed net 2164_IN2: MIXERG$3.I_IN, R2.1, RSTAB2.1
- removed net 2164_IN3: MIXERG$5.I_IN, R3.1, RSTAB3.1
- removed net 2164_IN4: MIXERG$4.I_IN, R4.1, RSTAB4.1
- removed net 2164_MODE: MIXERG$1.MODE, RMODE.2
- removed net 2164_OUT1: CONN_CURRENT_SUMMING.4, MIXERG$2.I_OUT
- removed net 2164_OUT2: CONN_CURRENT_SUMMING.2, MIXERG$3.I_OUT
- removed net 2164_OUT3: CONN_CURRENT_SUMMING.8, MIXERG$5.I_OUT
- removed net 2164_OUT4: CONN_CURRENT_SUMMING.6, MIXERG$4.I_OUT
- removed net CURRENT_OUT: CONN_IOUT.1, CONN_IOUT.2, CONN_IOUT.3, CONN_ITOV.3
- removed net GAIN1: CONN_STM32.3, MIXERG$2.GAIN_VCA
- removed net GAIN2: CONN_STM32.4, MIXERG$3.GAIN_VCA
- removed net GAIN3: CONN_STM32.1, MIXERG$5.GAIN_VCA
- removed net GAIN4: CONN_STM32.2, MIXERG$4.GAIN_VCA
- removed net IN1: CIN1.1, CONN_INPUT.2
- removed net IN2: CIN2.1, CONN_INPUT.1
- removed net IN3: CIN3.1, CONN_INPUT.4
- removed net IN4: CIN4.1, CONN_INPUT.3
- removed net MIXER_OUT: CONN_CURRENT_SUMMING.1, CONN_CURRENT_SUMMING.3, CONN_CURRENT_SUMMING.5, CONN_CURRENT_SUMMING.7, CONN_ITOV.2
- removed net N$11: CIN2.2, R2.2
- removed net N$12: CAOP.1, CONN_ITOV.1, CONV_ITOV.-IN, RAOP.1
- removed net N$33: CSTAB2.2, RSTAB2.2
- removed net N$34: CSTAB1.2, RSTAB1.2
- removed net N$35: CIN1.2, R1.2
- removed net N$41: CSTAB3.2, RSTAB3.2
- removed net N$5: CIN4.2, R4.2
- removed net N$7: CSTAB4.2, RSTAB4.2
- removed net N$71: CIN3.2, R3.2
- removed net VOLTAGE_OUT: CAOP.2, CONN_VOUT.1, CONN_VOUT.2, CONN_VOUT.3, CONV_ITOV.OUT, RAOP.2
- new net 411_IN_PULSE: 411D.IN, CONN_STM32.4, R_PD_411_IN_PULSE.2
- new net 411_IN_SAW: 411C.IN, CONN_STM32.7, R_PD_411_IN_SAW.1
- new net 411_IN_SYNC: 411B.IN, CONN_STM32.6, R_PD_411_IN_SYNC.1
- new net 411_IN_TRI: 411A.IN, CONN_STM32.5, R_PD_411_IN_TRI.1
- new net 5V: 411P.VL, CDEC_411B.1, CDEC_411B1.1, CONN_ALIM1.3, CONN_ALIM2.3, R_PD_411_IN_SAW.2
- new net CALIB: CONN_STM32.3, R5_3340.1, R6_3340.1
- new net CV_FREQ: CONN_STM32.1, R_CV_FREQ.2
- new net CV_PWM: CEM3340.PWM_CTRL, CONN_STM32.2, R1_PWM.1, R2_PWM.1
- new net FREQ_CTRL: CEM3340.FREQ_CTRL, R_CV_FREQ.1, R_CV_FREQ_BIAS.1, R_CV_FREQ_STAB.1
- new net HARD_SYNC: C1_SYNC3340.2, CEM3340.HARD_SYNC
- new net LINEAR_CTRL: CEM3340.LINEAR_CTRL, R10_3340.1, R8_3340.1, R_FM_LIN.1
- new net N$1: C_FM_LIN.1, R_FM_LIN.2
- new net N$2: 411D.S, R2S_411.2
- new net N$4: C_FM_LIN.2
- new net N$42: C_CV_FREQ_STAB.2, R_CV_FREQ_STAB.2
- new net N$45: C4_3340.1, R10_3340.2
- new net N$49: 411A.D, C1_411.2, R1_411.2
- new net N$50: 411D.D, C2_411.2, R2_411.2
- new net N$51: 411C.D, C3_411.2, R3_411.2
- new net OUT: CONN_OUT.1, CONN_OUT.2, CONN_OUT.3, R1S_411.2, R2S_411.1, R3S_411.1
- new net PULSE: C3_411.1, CEM3340.PULSE_OUT, R6_3340.2, TP_PULSE.P$1
- new net PULSE_OUT: 411C.S, R3S_411.2
- new net SAW: CEM3340.SAW_OUT, R7_3340.2
- new net SAW_3340: C2_411.1, R7_3340.1, TP_SAW.P$1
- new net SCALE: CEM3340.SCALE, R11_3340.1
- new net SOFT_SYNC: C2_SYNC3340.2, CEM3340.SOFT_SYNC
- new net SYNC_3340: 411B.D, C1_SYNC3340.1, R_SYNC.2
- new net SYNC_IN: 411B.S, SYNC_IN.P$1
- new net TEMPCO1: CEM3340.MUL_GAIN1, R1_3340.1
- new net TEMPCO2: CEM3340.MUL_GAIN2, R2_3340.1
- new net TIMING_CAP: CEM3340.TIMING_CAP, C_3340.2
- new net TRI_3340: C1_411.1, CEM3340.TRI_OUT, TP_TRI.P$1
- new net TRI_OUT: 411A.S, R1S_411.1
- new net VEE: CDEC_3340B.2, CDEC_3340B1.2, CEM3340.VEE, R1_3340.2, R2_3340.2, R3_3340.2
- net +15V: now also 411P.VDD, CDEC_3340A.2, CDEC_3340A1.2, CEM3340.VCC, CONN_ALIM1.1, CONN_ALIM2.1, R2_PWM.2, R8_3340.2, R_CV_FREQ_BIAS.2; no longer CDEC+15V.2, CDEC+15VPOL.2, CONN_ALIM.7, CONN_ALIM.8, CONV_ITOV.V+, MIXERG$1.V+, RMODE.1
- net -15V: now also 411P.VSS, CONN_ALIM1.2, CONN_ALIM2.2, R3_3340.1; no longer CDEC-15V.1, CDEC-15VPOL.1, CONN_ALIM.5, CONN_ALIM.6, CONV_ITOV.V-, MIXERG$1.V-
- net AGND: now also 411P.GND, C2_SYNC3340.1, C4_3340.2, CDEC_3340A.1, CDEC_3340A1.1, CDEC_3340B.1, CDEC_3340B1.1, CDEC_411B.2, CDEC_411B1.2, CEM3340.GND, CONN_ALIM1.4, CONN_ALIM2.4, CONN_STM32.8, C_3340.1, C_CV_FREQ_STAB.1, R11_3340.2, R1_411.1, R1_PWM.2, R2_411.1, R3_411.1, R5_3340.2, R_PD_411_IN_PULSE.1, R_PD_411_IN_SYNC.2, R_PD_411_IN_TRI.2, R_SYNC.1; no longer CDEC+15V.1, CDEC+15VPOL.1, CDEC-15V.2, CDEC-15VPOL.2, CONN_ALIM.1, CONN_ALIM.2, CONN_STM32.5, CONV_ITOV.+IN, CSTAB1.1, CSTAB2.1, CSTAB3.1, CSTAB4.1, MIXERG$1.GND
Other:
- note added: "Bloc VCO3340 + switches de sélection de forme d'onde"
- note added: "C2_SYNC protège l'entrée soft sync contre le bruit"
- note added: "FM lin non utilisée"
- note added: "SAW is the only active output when nothing is plugged from the STM32."
- note added: "Values for R?S_411 depend on the level of the signal we wanna have at V2164's output."
- note removed: "Control Voltages"
- note removed: "Input Signals"
- note removed: "Output"
- note removed: "Output mode I : 2-1 Output mode V : 2-3"
- note removed: "Power"
- note removed: "RLOAD permet de tester le bon fonctionnement de la sortie en courant du 2164"
- note removed: "current -> voltage converter"
