File: eagle-schematics/themis-v1/VCF AS3320/pcb - vcf et etage sortie v3.sch (EAGLE design)
At the start: 38 parts

Commit message: New version of DAC board based on AD5391 chip
Parts:
- added C_IN: 470n, rcl:C-EU075-032X103
- added R_PD_4TH_ORDER, R_PU_2ND_ORDER: 100k, rcl:R-EU_0204/7
Connections:
- new net GND: R_PD_4TH_ORDER.1
- new net N$1: C_IN.1, RTEST_VCF.1
- net 5V: now also R_PU_2ND_ORDER.1
- net IN_2NDORDER: now also R_PU_2ND_ORDER.2
- net IN_4THORDER: now also R_PD_4TH_ORDER.2
- net V_IN: now also C_IN.2; no longer RTEST_VCF.1

Commit message: checked connections
Parts:
- renumbered R1_VCF to R1_CV, R2 to R2_CV, R3 to R_RES
Connections:
- net N$17 renamed VCAP3
- net N$18 renamed VCAP2
- net N$24 renamed VCAP4
- net N$37 renamed VCF_FREQ_CV
- net N$5 renamed VCAP1
- net N$57 renamed OUT1
- net N$62 renamed IN2
- net N$65 renamed OUT2
- net N$69 renamed OUT4
- net N$72 renamed IN3
- net N$82 renamed OUT3
- net N$83 renamed IN4
- net N$86 renamed VIN_RES
- net N$87 renamed VCF_RES_CUR
- net VM3320 renamed VEE
- removed net GND: R_PD_4TH_ORDER.1
- net AGND: now also R_PD_4TH_ORDER.1
