File: eagle-schematics/themis-v1/VCF AS3320/pcb - vcf et etage sortie.brd (EAGLE design)
At the start: 78 x 63.8 mm, 42 parts

Commit message: checked connections
Connections:
- net N$37 renamed FREQ_CV
- net N$87 renamed RES_CUR
Changed lines of the file:
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@@
 <?xml version="1.0" encoding="utf-8"?>
 <!DOCTYPE eagle SYSTEM "eagle.dtd">
-<eagle version="9.3.1">
+<eagle version="9.5.2">
 <drawing>
 <settings>
@@
 <setting verticaltext="up"/>
 </settings>
-<grid distance="25" unitdist="mil" unit="mil" style="lines" multiple="1" display="yes" altdistance="5" altunitdist="mil" altunit="mil"/>
+<grid distance="25" unitdist="mil" unit="mil" style="lines" multiple="1" display="no" altdistance="5" altunitdist="mil" altunit="mil"/>
 <layers>
 <layer number="1" name="Top" color="4" fill="1" visible="yes" active="yes"/>
@@
 <wire x1="62.865" y1="41.275" x2="62.865" y2="36.83" width="0.6096" layer="16"/>
 </signal>
-<signal name="N$37">
+<signal name="FREQ_CV">
 <contactref element="R1_VCF" pad="1"/>
 <contactref element="R2" pad="1"/>
@@
 <wire x1="64.77" y1="10.795" x2="56.515" y2="19.05" width="0.6096" layer="1"/>
 </signal>
-<signal name="N$87">
+<signal name="RES_CUR">
 <contactref element="VCF" pad="9"/>
 <contactref element="R3" pad="1"/>
