File: eagle-schematics/themis-v2/DAC STM32 Board v5 - AD5391.brd (EAGLE design)
At the start: 161.3 x 134.6 mm, 229 parts, among them IC1 MCP23017SO, U1 ANALOG_DEVICES_AD5391BSTZ-3AN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

Commit message: Layout half way
Parts:
- removed SYNC_IN1: (no value), 6P1_EVB:TESTPOINT_63
- added JP_SYNC_3340B_TO_A: JUMPER, 6P1_EVB:HDR2X1
- moved JP_SAWOUT_VCO3340B 16.0 mm to (47.0, 125.5)
- moved JP_OUT_VCO3340A 12.0 mm to (46.9, 107.2)
- moved JP_PULSEOUT_VCO3340B 6.45 mm to (47.0, 119.1)
- moved JP_FMLIN_VCO3340B 4.73 mm to (42.0, 83.1), turned to 270 degrees
- moved JP9 3.92 mm to (92.7, 127.4)
- moved JP7 3.51 mm to (92.7, 123.6)
- moved JP_TRIOUT_VCO3340B 1.17 mm to (47.0, 116.1)
- renumbered CEM1 to 3340B, CEM3 to 3340A
Connections:
- net IN2_MIXERA: now also JP_OUT_VCO3340A.2; no longer JP_SAWOUT_VCO3340B.2
- net IN3_MIXERA: now also JP_SAWOUT_VCO3340B.2; no longer JP_PULSEOUT_VCO3340B.2
- net IN4_MIXERA: now also JP_PULSEOUT_VCO3340B.2; no longer JP_OUT_VCO3340A.2
- net SYNC_IN_VCOA: now also JP_SYNC_3340B_TO_A.1; no longer SYNC_IN1.P$1
- net VCO3340B_SAW_OUT: now also JP_SYNC_3340B_TO_A.2
Routing:
- net VCO3340B_SAW_OUT: track 27.6 -> 213.2 mm
- net VCO3340B_TRI_OUT: track 33.6 -> 74.0 mm, vias 0 -> 1
- net VCO13700_SQUARE: track 68.3 -> 47.8 mm
- net 2164_OUT4_MIXA: track 20.4 -> 0.00 mm
- net -15V: track 299.3 -> 280.1 mm
- net GAIN2_A: track 31.4 -> 14.8 mm
- net VCO3340B_PULSE_OUT: track 27.8 -> 43.1 mm
- net 2164_OUT3_MIXA: track 15.0 -> 0.00 mm
- net SYNC_IN_VCOA: track 9.83 -> 20.0 mm
- net IN4_MIXERB: track 0.00 -> 8.10 mm
- net IN3_MIXERB: track 0.00 -> 5.71 mm
- net VCO3340B_FMLIN: track 0.00 -> 5.59 mm
- net IN2_MIXERA: track 0.00 -> 4.57 mm
- net IN4_MIXERA: track 0.00 -> 4.45 mm
- net IN3_MIXERA: track 0.00 -> 4.45 mm
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