File: eagle-schematics/themis-v2/DAC STM32 Board v5 - AD5391.sch (EAGLE design)
At the start: 229 parts, among them IC1 MCP23017SO, U1 ANALOG_DEVICES_AD5391BSTZ-3AN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

Commit message: Layout half way
Parts:
- removed SYNC_IN1: (no value), 6P1_EVB:TESTPOINT
- added JP_SYNC_3340B_TO_A: JUMPER, 6P1_EVB:JUMPER
- renumbered CEM1 to 3340B, CEM3 to 3340A
Connections:
- net IN2_MIXERA: now also JP_OUT_VCO3340A.2; no longer JP_SAWOUT_VCO3340B.2
- net IN3_MIXERA: now also JP_SAWOUT_VCO3340B.2; no longer JP_PULSEOUT_VCO3340B.2
- net IN4_MIXERA: now also JP_PULSEOUT_VCO3340B.2; no longer JP_OUT_VCO3340A.2
- net SYNC_IN_VCOA: now also JP_SYNC_3340B_TO_A.1; no longer SYNC_IN1.P$1
- net VCO3340B_SAW_OUT: now also JP_SYNC_3340B_TO_A.2
