File: eagle-schematics/themis-v1/VCO LM13700/LM13700_v2.brd (EAGLE design)
At the start: 90.5 x 51.3 mm, 39 parts

Commit message: bug fix on LM13700 schematics
Parts:
- R1_EXPCONV: value 330 -> 3.3k
- R2_EXPCONV, R4_EXPCONV: value 10 -> 100
- R3_EXPCONV: value 260 -> 2.6k
Other:
- board text added: "THeMiS - VCO 13700 [v2] BOTTOM"
- board text added: "THeMiS - VCO 13700 [v2] TOP"
- board text removed: "THeMiS - VCO 13700 [v1] BOTTOM"
- board text removed: "THeMiS - VCO 13700 [v1] TOP"
Changed lines of the file:
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@@
 <?xml version="1.0" encoding="utf-8"?>
 <!DOCTYPE eagle SYSTEM "eagle.dtd">
-<eagle version="9.3.2">
+<eagle version="9.5.2">
 <drawing>
 <settings>
@@
 <wire x1="88.57" y1="49.266" x2="-1.905" y2="49.266" width="0.1524" layer="20"/>
 <wire x1="-1.905" y1="49.266" x2="-1.905" y2="-2.032" width="0.1524" layer="20"/>
-<text x="6.35" y="43.18" size="1.778" layer="1">THeMiS - VCO 13700 [v1] TOP</text>
-<text x="45.72" y="43.18" size="1.778" layer="16" rot="MR0">THeMiS - VCO 13700 [v1] BOTTOM</text>
+<text x="6.35" y="43.18" size="1.778" layer="1">THeMiS - VCO 13700 [v2] TOP</text>
+<text x="45.72" y="43.18" size="1.778" layer="16" rot="MR0">THeMiS - VCO 13700 [v2] BOTTOM</text>
 </plain>
 <attributes>
@@
 <attribute name="VALUE" x="58.0136" y="30.8864" size="0.4064" layer="27" ratio="10" rot="R180"/>
 </element>
-<element name="R1_EXPCONV" library="rcl" library_urn="urn:adsk.eagle:library:334" package="0204/7" package3d_urn="urn:adsk.eagle:package:23498/2" value="330" x="3.175" y="5.715" smashed="yes" rot="R270">
+<element name="R1_EXPCONV" library="rcl" library_urn="urn:adsk.eagle:library:334" package="0204/7" package3d_urn="urn:adsk.eagle:package:23498/2" value="3.3k" x="3.175" y="5.715" smashed="yes" rot="R270">
 <attribute name="NAME" x="4.3434" y="7.7216" size="0.4064" layer="25" ratio="10" rot="R270"/>
 <attribute name="SPICEPREFIX" value="R" x="-43.815" y="-48.895" size="1.778" layer="27" rot="R270" display="off"/>
@@
 <attribute name="VALUE" x="51.8414" y="33.2486" size="0.4064" layer="27" ratio="10"/>
 </element>
-<element name="R2_EXPCONV" library="rcl" library_urn="urn:adsk.eagle:library:334" package="0204/7" package3d_urn="urn:adsk.eagle:package:23498/2" value="10" x="8.255" y="13.97" smashed="yes" rot="R90">
+<element name="R2_EXPCONV" library="rcl" library_urn="urn:adsk.eagle:library:334" package="0204/7" package3d_urn="urn:adsk.eagle:package:23498/2" value="100" x="8.255" y="13.97" smashed="yes" rot="R90">
 <attribute name="NAME" x="7.0866" y="11.9634" size="0.4064" layer="25" ratio="10" rot="R90"/>
 <attribute name="SPICEPREFIX" value="R" x="55.245" y="82.55" size="1.778" layer="27" rot="R90" display="off"/>
 <attribute name="VALUE" x="10.5664" y="11.8364" size="0.4064" layer="27" ratio="10" rot="R90"/>
 </element>
-<element name="R3_EXPCONV" library="rcl" library_urn="urn:adsk.eagle:library:334" package="0204/7" package3d_urn="urn:adsk.eagle:package:23498/2" value="260" x="1.905" y="39.37" smashed="yes" rot="R90">
+<element name="R3_EXPCONV" library="rcl" library_urn="urn:adsk.eagle:library:334" package="0204/7" package3d_urn="urn:adsk.eagle:package:23498/2" value="2.6k" x="1.905" y="39.37" smashed="yes" rot="R90">
 <attribute name="NAME" x="0.7366" y="37.3634" size="0.4064" layer="25" ratio="10" rot="R90"/>
 <attribute name="SPICEPREFIX" value="R" x="55.245" y="63.5" size="1.778" layer="27" rot="R90" display="off"/>
 <attribute name="VALUE" x="4.2164" y="37.2364" size="0.4064" layer="27" ratio="10" rot="R90"/>
 </element>
-<element name="R4_EXPCONV" library="rcl" library_urn="urn:adsk.eagle:library:334" package="0204/7" package3d_urn="urn:adsk.eagle:package:23498/2" value="10" x="16.51" y="32.385" smashed="yes">
+<element name="R4_EXPCONV" library="rcl" library_urn="urn:adsk.eagle:library:334" package="0204/7" package3d_urn="urn:adsk.eagle:package:23498/2" value="100" x="16.51" y="32.385" smashed="yes">
 <attribute name="NAME" x="13.2334" y="33.5534" size="0.4064" layer="25" ratio="10"/>
 <attribute name="SPICEPREFIX" value="R" x="54.61" y="-20.955" size="1.778" layer="27" display="off"/>

Commit message: bug fix
Parts:
- R3_EXPCONV: value 2.6k -> 8.2k
- R5_EXPCONV: value 110 -> 220
- REE_13700: value 27k -> 47k
- RTRI_13700: value 12k -> 10k
Changed lines of the file:
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@@
 <layer number="25" name="tNames" color="7" fill="1" visible="yes" active="yes"/>
 <layer number="26" name="bNames" color="7" fill="1" visible="yes" active="yes"/>
-<layer number="27" name="tValues" color="7" fill="1" visible="no" active="yes"/>
+<layer number="27" name="tValues" color="7" fill="1" visible="yes" active="yes"/>
 <layer number="28" name="bValues" color="7" fill="1" visible="no" active="yes"/>
 <layer number="29" name="tStop" color="7" fill="3" visible="no" active="yes"/>
@@
 <attribute name="VALUE" x="10.5664" y="11.8364" size="0.4064" layer="27" ratio="10" rot="R90"/>
 </element>
-<element name="R3_EXPCONV" library="rcl" library_urn="urn:adsk.eagle:library:334" package="0204/7" package3d_urn="urn:adsk.eagle:package:23498/2" value="2.6k" x="1.905" y="39.37" smashed="yes" rot="R90">
+<element name="R3_EXPCONV" library="rcl" library_urn="urn:adsk.eagle:library:334" package="0204/7" package3d_urn="urn:adsk.eagle:package:23498/2" value="8.2k" x="1.905" y="39.37" smashed="yes" rot="R90">
 <attribute name="NAME" x="0.7366" y="37.3634" size="0.4064" layer="25" ratio="10" rot="R90"/>
 <attribute name="SPICEPREFIX" value="R" x="55.245" y="63.5" size="1.778" layer="27" rot="R90" display="off"/>
@@
 <attribute name="VALUE" x="14.3764" y="30.0736" size="0.4064" layer="27" ratio="10"/>
 </element>
-<element name="R5_EXPCONV" library="rcl" library_urn="urn:adsk.eagle:library:334" package="0204/7" package3d_urn="urn:adsk.eagle:package:23498/2" value="110" x="16.51" y="27.94" smashed="yes">
+<element name="R5_EXPCONV" library="rcl" library_urn="urn:adsk.eagle:library:334" package="0204/7" package3d_urn="urn:adsk.eagle:package:23498/2" value="220" x="16.51" y="27.94" smashed="yes">
 <attribute name="NAME" x="14.5034" y="29.1084" size="0.4064" layer="25" ratio="10"/>
 <attribute name="SPICEPREFIX" value="R" x="68.58" y="-25.4" size="1.778" layer="27" display="off"/>
@@
 <attribute name="VALUE" x="7.3914" y="14.3764" size="0.4064" layer="27" ratio="10" rot="R90"/>
 </element>
-<element name="REE_13700" library="rcl" library_urn="urn:adsk.eagle:library:334" package="0204/7" package3d_urn="urn:adsk.eagle:package:23498/2" value="27k" x="54.61" y="21.59" smashed="yes" rot="R270">
+<element name="REE_13700" library="rcl" library_urn="urn:adsk.eagle:library:334" package="0204/7" package3d_urn="urn:adsk.eagle:package:23498/2" value="47k" x="54.61" y="21.59" smashed="yes" rot="R270">
 <attribute name="NAME" x="55.7784" y="23.5966" size="0.4064" layer="25" ratio="10" rot="R270"/>
 <attribute name="SPICEPREFIX" value="R" x="-11.43" y="-1.27" size="1.778" layer="27" rot="R270" display="off"/>
@@
 <attribute name="VALUE" x="22.4536" y="38.5064" size="0.4064" layer="27" ratio="10" rot="R180"/>
 </element>
-<element name="RTRI_13700" library="rcl" library_urn="urn:adsk.eagle:library:334" package="0204/7" package3d_urn="urn:adsk.eagle:package:23498/2" value="12k" x="24.765" y="8.255" smashed="yes" rot="R270">
+<element name="RTRI_13700" library="rcl" library_urn="urn:adsk.eagle:library:334" package="0204/7" package3d_urn="urn:adsk.eagle:package:23498/2" value="10k" x="24.765" y="8.255" smashed="yes" rot="R270">
 <attribute name="NAME" x="25.9334" y="10.2616" size="0.4064" layer="25" ratio="10" rot="R270"/>
 <attribute name="SPICEPREFIX" value="R" x="-34.925" y="-53.975" size="1.778" layer="27" rot="R270" display="off"/>
