File: eagle-schematics/themis-v2/main-board/DAC STM32 Board v5 - AD5391.sch (EAGLE design)
At the start: 229 parts, among them IC1 MCP23017SO, U1 ANALOG_DEVICES_AD5391BSTZ-3AN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

Commit message: bug fix
Parts:
- removed CIN_VCA: 470n, rcl:C-EU050-030X075
- removed CSTAB_VCA: 560p, rcl:C-EU050-030X075
- removed C_FM_LIN1, C_FM_LIN3: 100n, rcl:C-EU050-025X075
- removed JP_FMLIN_VCO3340B: JUMPER, 6P1_EVB:JUMPER
- removed RIN_VCA: 27k, rcl:R-EU_0204/7
- removed RSTAB_VCA: 470, rcl:R-EU_0204/7
- removed R_FM_LIN1, R_FM_LIN3: 1M, rcl:R-EU_0204/7
- added CIN4_MIXERB1: 470n, rcl:C-EU050-030X075
- added CSTAB1: 10u, rcl:C-EU050-030X075
- added CSTAB2, CSTAB3: 560p, rcl:C-EU050-030X075
- added JP_FMLIN_VCO3340B1, JP_OUT_VCO3340A1, JP_OUT_VCO3340A2: JUMPER, 6P1_EVB:JUMPER
- added RIN4_MIXERB1: 27k, rcl:R-EU_0204/7
- added RSTAB3_MIXERB1: 51k, rcl:R-EU_0204/7
- added RSTAB3_MIXERB2, RSTAB3_MIXERB3, RSTAB3_MIXERB4, RSTAB3_MIXERB5: 10k, rcl:R-EU_0204/7
- added RSTAB4_MIXERB1, RSTAB4_MIXERB2: 470, rcl:R-EU_0204/7
- added VCO1: LM13700N, ota:LM13700N
Connections:
- removed net 2164_IN1_MIXB: MIXER_BG$2.I_IN, RIN_VCA.1, RSTAB_VCA.1
- removed net 2164_OUT1_MIXA: JP_MIXER_A.2, MIXER_AG$2.I_OUT
- removed net CSTAB3_MIXERB: CSTAB8.1
- removed net N$21: CSTAB_VCA.2, RSTAB_VCA.2
- removed net N$62: CIN_VCA.2, RIN_VCA.2
- removed net N$84: C_FM_LIN1.1, R_FM_LIN1.2
- removed net N$92: C_FM_LIN3.1, R_FM_LIN3.2
- removed net N$93: C_FM_LIN3.2
- removed net NOISE_GENE: U1A.VOUT_15
- removed net OUT_VCA: JP1.1, MIXER_BG$2.I_OUT
- removed net VCO3340B_FMLIN: C_FM_LIN1.2, JP_FMLIN_VCO3340B.1
- new net 2164_IN4_MIXB1: MIXER_BG$2.I_IN, RIN4_MIXERB1.1, RSTAB4_MIXERB2.1
- new net CV_VCA: RSTAB3_MIXERB1.1, U1A.VOUT_15
- new net IN4_MIXERB1: CIN4_MIXERB1.1, JP_OUT_VCO3340A2.2
- new net N$10: CSTAB3.2, RSTAB4_MIXERB2.2
- new net N$11: CIN4_MIXERB1.2, RIN4_MIXERB1.2
- new net N$12: RSTAB3_MIXERB4.2, RSTAB3_MIXERB5.2, VCO1OTA1.IN_N
- new net N$17: RSTAB3_MIXERB1.2, VCO1OTA1.I_BIAS
- new net N$2: JP_FMLIN_VCO3340B1.2
- new net N$4: JP_MIXER_A.4, MIXER_AG$2.I_OUT
- new net N$8: CSTAB2.2, MIXER_BG$2.I_OUT, RSTAB4_MIXERB1.2
- new net N$9: CSTAB1.1, RSTAB3_MIXERB2.2, RSTAB3_MIXERB3.1, VCO1OTA1.IN_P
- net +15V: now also RSTAB3_MIXERB2.1, RSTAB3_MIXERB4.1, VCO1SUPPLY.V+
- net 2164_OUT2_MIXA: now also JP_MIXER_A.2; no longer JP_MIXER_A.4
- net 2164_OUT3_MIXA: now also JP_MIXER_A.6; no longer JP_MIXER_A.8
- net 2164_OUT4_MIXA: now also JP_MIXER_A.8; no longer JP_MIXER_A.6
- net 411_IN_PULSE: now also IC1.GPA1; no longer IC1.GPA0
- net 411_IN_SAW: now also IC1.GPA2; no longer IC1.GPA3
- net 411_IN_SYNC: now also IC1.GPA3; no longer IC1.GPA2
- net 411_IN_TRI: now also IC1.GPA0; no longer IC1.GPA1
- net AGND: now also CSTAB3.1, CSTAB8.1, RSTAB3_MIXERB3.2, RSTAB3_MIXERB5.1, RSTAB4_MIXERB1.1, VCO1SUPPLY.V-; no longer CSTAB_VCA.1
- net CV_FREQ_3340A: now also JP_FMLIN_VCO3340B1.1
- net GAIN3_A: now also U1A.VOUT_6; no longer U1A.VOUT_5
- net GAIN4_A: now also U1A.VOUT_5; no longer U1A.VOUT_6
- net IN2_MIXERA: now also JP_OUT_VCO3340A2.1
- net INPUT_CURRENT_SUM_STG: now also JP1.1, VCO1OTA1.OUT
- net INPUT_FM_3340: now also JP_OUT_VCO3340A1.2
- net IN_VCA: now also CSTAB1.2; no longer CIN_VCA.1
- net LINEAR_CTRL_VCOA: no longer R_FM_LIN3.1
- net LINEAR_CTRL_VCOB: no longer R_FM_LIN1.1
- net N$1: now also CSTAB2.1, JP_OUT_VCO3340A1.1; no longer JP_FMLIN_VCO3340B.2
Other:
- moved on the sheet: CIN4_MIXERB, CSTAB8, JP1, RIN4_MIXERB, RSTAB4_MIXERB
