File: eagle-schematics/themis-v2/main-board/DAC STM32F446 Board SMD v7.sch (EAGLE design)
At the start: 250 parts, among them IC1 4027D, U2 AD5328BRUZ-REEL7, U3 AD5328BRUZ-REEL7

Commit message: started PCB routing with F446
Parts:
- removed BTN_RST1: BUTTON-FSM14JRT, MyComponents:BUTTON-FSM14JRT
- removed C+15VPOL_VCF, C-15VPOL_VCF: 1u, rcl:C-EUC0603
- removed C1_HSE1, C2_HSE1: 12pF, MyComponents:C-US0805
- removed C1_LSE1, C2_LSE1: 22pF, MyComponents:C-US0805
- removed C5VPOL_VCF, CDEC+15V6, CDEC+15V7, CDEC-15V6, CDEC-15V7, CDEC-VREF-1, CDEC-VREF-3, CDEC_5V4: 100n, rcl:C-EUC0603
- removed CDEC-VREF-2: 10u, rcl:CPOL-US140CLH-1014
- removed CDEC-VREF-4: 100u, rcl:CPOL-US140CLH-1014
- removed CDEC_5V1: 10u, rcl:C-EUC0603
- removed CF_2: 100nF, rcl:C-EUC0603
- removed CIN_2, C_IN2: 470n, rcl:C-EUC0603
- removed CONN_UART_RPI: (no value), con-lstb:MA03-1
- removed CONVLOG2: BC857BS, paires_diff:BC857BS
- removed C_DEC_10, C_DEC_12, C_DEC_14, C_DEC_8, C_DEC_9, C_IN_ALIM1, C_NRST1: 0.1uF, MyComponents:C-US0805
- removed C_DEC_11: 4.7uF, MyComponents:C-US0805
- removed C_DEC_13: 1.0uF, MyComponents:C-US0805
- removed C_DEC_POL3: 100 uF, MyComponents:CPOL-US1311
- removed C_DEC_POL4: 47 uF, MyComponents:CPOL-US0805
- removed C_IN_ALIM_POL1: 470 uF, MyComponents:CPOL-US2917
- removed C_VCAP1, V_CAP2: 2.2uF, MyComponents:C-US0805
- removed DEBUG_CONN1: 75867-331LF, MyComponents:MA03-2
- removed D_2: 1N4148DO35-7, diode:1N4148DO35-7
- removed EXPCONV2: TL081, linear:1AMP_P7+4D
- removed HEADER_EXPCONV2: (no value), con-amp-quick:M03
- removed IC_EEPROM: 24C04ASN, microchip:24C04ASN
- removed JP7, JP8, JP9, JP_OUT_VCO3340A1: JUMPER, 6P1_EVB:JUMPER
- removed L_3V3_OUT1: 1 uH, MyComponents:L-USL0805
- removed R1_8, R2_8, R2_VCF, RCAL_2, RF3, RF4, R_RES_VCF: 100k, rcl:R-EU_R0603
- removed R1_EXPCONV2: 330, rcl:R-EU_R0603
- removed R1_VCF, RSQU_2: 10k, rcl:R-EU_R0603
- removed R2_EXPCONV2, R4_EXPCONV2: 10, rcl:R-EU_R0603
- removed R3_EXPCONV2: 260, rcl:R-EU_R0603
- removed R5_EXPCONV2: 110, rcl:R-EU_R0603
- removed RA_2: 4.7k, rcl:R-EU_R0603
- removed RB2: 220k, rcl:R-EU_R0603
- removed RBIAS_EXPCONV2, RCAL_1: 47k, rcl:R-EU_R0603
- removed RC3, RC4: 91k, rcl:R-EU_R0603
- removed REE_2, RTEST_13700FREQ2: 27k, rcl:R-EU_R0603
- removed REGUL3V1: REG1117, MyComponents:REG1117
- removed RTEST_LOG2, R_LIM_2: 1k, rcl:R-EU_R0603
- removed RTRI_2: 12k, rcl:R-EU_R0603
- removed R_3V3_OUT1: 1, MyComponents:R-US0805
- removed R_HSE1: 100, MyComponents:R-US0805
- removed TP_13700_SQU2, TP_13700_TRI2, TP_CV_2: (no value), 6P1_EVB:TESTPOINT
- removed U2, U3: AD5328BRUZ-REEL7, AD5328:AD5328BRUZ-REEL7
- removed UC1: STM32F405RG, stm32:STM32F405RGT
- removed VCF_ANALOG_SW: DG413DJD, linear:DG413DJD
- removed VCO2: LM13700M, ota:LM13700M
- removed VREF_DAC_2V5: AD780R, analog-devices:AD780R
- removed XTAL_HSE1: 16MHz, MyComponents:Q-HSEHC-46X
- removed XTAL_LSE1: 32.7680kHz, MyComponents:Q-LSECM7V-T1A
- added C+15V_SUM_STG, C-15V_SUM_STG: 100n, rcl:C-EU075-032X103
- added C1_HSE, C2_HSE: 12pF, MyComponents:C-US0805
- added CONN_ALIM, SUM_STG_HEADER1: (no value), con-lstb:MA04-2
- added COUT_SUM_STG: 22u, resistor:CPOL-EUB45181A
- added C_DEC_1, C_DEC_2, C_DEC_3, C_DEC_4, C_DEC_5, C_NRST: 0.1uF, MyComponents:C-US0805
- added C_DEC_6: 1.0uF, MyComponents:C-US0805
- added C_DEC_ALIM_+15V, C_DEC_ALIM_-15V, C_DEC_ALIM_5V, C_IN_ALIM_POL: 10u, MyComponents:CPOL-US2917
- added C_IN_VCF: 470n, rcl:C-EUC0805
- added C_TLV_OUT: 100 uF, MyComponents:CPOL-US2917
- added C_VCAP: 2.2uF, MyComponents:C-US0805
- added DEBUG_CONN: 75867-331LF, MyComponents:MA03-2
- added I2C_PU_SCL, I2C_PU_SDA: 1k, 6P1_EVB:R-US_R0805
- added IC2: 24C04AP, microchip:24C04AP
- added JACK_SUM_STG: 1502_01, con-lumberg:1502_01
- added L_3V3: 1 uH, MyComponents:L-USL0805
- added OPAMP_SUM_STG: NE5534AN, linear:NE5534AN
- added POT_SUM_STG: 100kB, pot:3RP/1610N
- added RB2_VCF: 220k, rcl:R-EU_R0805
- added RC3_VCF, RC4_VCF: 91k, rcl:R-EU_R0805
- added REG3V3: TLV75533PDBVR, TLV75533PDBVR:TLV75533PDBVR
- added RF3_VCF, RF4_VCF: 100k, rcl:R-EU_R0805
- added ROUT_SUM_STG: 470, rcl:R-EU_0207/12
- added R_3V3: 1, MyComponents:R-US0805
- added R_HSE: 100, MyComponents:R-US0805
- added R_RST: 100k, MyComponents:R-US0805
- added SUM_STG_C: 560p, rcl:C-EU075-032X103
- added SUM_STG_R: 27k, rcl:R-EU_0207/10
- added SW_RST: (no value), switch-omron:10-XX
- added TRIM_VCF_CUT, TRIM_VCF_RES: 100k, adafruit:TRIM
- added U1: STM32F446RCT7, STM32F446RCT7:STM32F446RCT7
- added XTAL_HSE: 16MHz, MyComponents:Q-HSEHC-46X
- C+15V_VCF, C-15V_VCF, C10, C3, C4, C5, C5V_VCF, CRES_VCF: device rcl:C-EUC0603 -> rcl:C-EUC0805
- C_SW1, C_SW2: device 6P1_EVB:C-EUC0603 -> 6P1_EVB:C-EUC0805
- IC1: value 4027D -> ADG453BRZ; device 40xx:4027D -> ADG453BRZ:ADG453BRZ
- RB1_VCF, RB3_VCF, RC1_VCF, RC2_VCF, REE_VCF, RF1_VCF, RF2_VCF, RRI_VCF, R_PD_4TH_ORDER_VCF: device rcl:R-EU_R0603 -> rcl:R-EU_R0805
- R_SW1A, R_SW1B, R_SW2A, R_SW2B: device 6P1_EVB:R-US_R0603 -> 6P1_EVB:R-US_R0805
Connections:
- removed net ALIM_CONN: C_IN_ALIM1.1, C_IN_ALIM_POL1.+, REGUL3V1.VIN
- removed net BIAS_4027_VCO13700: CIN_2.1, D_2.A, R1_8.2, R2_8.1
- removed net CALIB_13700: RCAL_1.2, RCAL_2.1
- removed net CV_FREQ_13700: R1_EXPCONV2.2, TP_CV_2.P$1, U2.VOUTC
- removed net DAC_LDAC: U2.!_2, U3.!_2
- removed net DAC_SYNC_CV: U2.!
- removed net DAC_SYNC_GAIN: U3.!
- removed net FM_ENTREE_13700_VCO13700: HEADER_EXPCONV2.3, RTEST_13700FREQ2.2, VCO2OTA1.I_BIAS
- removed net IA_VCO13700: REE_2.1, VCO2OTA2.I_BIAS
- removed net INPUT_FM_3340: JP_OUT_VCO3340A1.2, RTEST_13700FREQ2.1
- removed net N$105: C2_HSE1.2, UC1MCU.OSC_OUT, XTAL_HSE1.2
- removed net N$106: R_HSE1.1, UC1MCU.OSC_IN
- removed net N$113: CRES_VCF.1, VCF_ANALOG_SWA.S, VCF_ANALOG_SWB.S
- removed net N$94: EXPCONV2.OUT, R5_EXPCONV2.2
- removed net N$95: RA_2.2, VCO2BUF2.B, VCO2OTA1.IN_P, VCO2OTA2.IN_P, VCO2OTA2.OUT
- removed net N$96: CF_2.2, VCO2BUF1.B, VCO2OTA1.OUT
- removed net N$98: D_2.C, R_LIM_2.2
- removed net N$99: HEADER_EXPCONV2.1, RTEST_LOG2.1
- removed net OUT_EXPCONV_VCO13700: CONVLOG2.C2, HEADER_EXPCONV2.2
- removed net PA0: UC1MCU.PA0-WKUP
- removed net PA1: UC1MCU.PA1
- removed net PA10: UC1MCU.PA10
- removed net PA15: UC1MCU.PA15
- removed net PA2: UC1MCU.PA2
- removed net PA3: UC1MCU.PA3
- removed net PA4: UC1MCU.PA4
- removed net PA5: UC1MCU.PA5
- removed net PA6: UC1MCU.PA6
- removed net PA7: UC1MCU.PA7
- removed net PA8: UC1MCU.PA8
- removed net PB0: UC1MCU.PB0
- removed net PB1: UC1MCU.PB1
- removed net PB10: UC1MCU.PB10
- removed net PB11: UC1MCU.PB11
- removed net PB12: UC1MCU.PB12
- removed net PB13: UC1MCU.PB13
- removed net PB14: UC1MCU.PB14
- removed net PB15: UC1MCU.PB15
- removed net PB2: UC1MCU.PB2
- removed net PB3: UC1MCU.PB3
- removed net PB4: UC1MCU.PB4
- removed net PB5: UC1MCU.PB5
- removed net PB6: UC1MCU.PB6
- removed net PB7: UC1MCU.PB7
- removed net PB8: UC1MCU.PB8
- removed net PB9: UC1MCU.PB9
- removed net PC0: UC1MCU.PC0
- removed net PC1: UC1MCU.PC1
- removed net PC10: UC1MCU.PC10
- removed net PC11: UC1MCU.PC11
- removed net PC12: UC1MCU.PC12
- removed net PC13: UC1MCU.PC13
- removed net PC2: UC1MCU.PC2
- removed net PC3: UC1MCU.PC3
- removed net PC4: UC1MCU.PC4
- removed net PC5: UC1MCU.PC5
- removed net PC6: UC1MCU.PC6
- removed net PC7: UC1MCU.PC7
- removed net PC8: UC1MCU.PC8
- removed net PC9: UC1MCU.PC9
- removed net PD2: UC1MCU.PD2
- removed net PNP1_B_VCO13700: CONVLOG2.B1, R1_EXPCONV2.1, R2_EXPCONV2.1
- removed net PNP1_C1_VCO1: CONVLOG2.C1, EXPCONV2.-IN, RBIAS_EXPCONV2.2
- removed net PNP2_B_VCO13700: CONVLOG2.B2, R3_EXPCONV2.1, R4_EXPCONV2.1
- removed net PNP_E1-VCO1_MIXB: CONVLOG2.E1, CONVLOG2.E2, R5_EXPCONV2.1
- removed net Q2M1: C2_LSE1.2, UC1MCU.PC14, XTAL_LSE1.1
- removed net Q2P1: C1_LSE1.2, UC1MCU.PC15, XTAL_LSE1.2
- removed net SPI_CLK: U2.SCLK, U3.SCLK
- removed net SPI_MOSI: U2.DIN, U3.DIN
- removed net SUBBASS_IN_VCO13700: IC1B.CLK, R_LIM_2.1
- removed net USART_RX_RPI_TX: CONN_UART_RPI.2
- removed net USART_TX_RPI_RX: CONN_UART_RPI.3
- removed net USB-DM: UC1MCU.PA11
- removed net USB-DP: UC1MCU.PA12
- removed net USB-VBUS: UC1MCU.PA9
- removed net VCAP2: UC1MCU.VCAP1, V_CAP2.2
- removed net VCO13700_SQUARE: CIN_2.2, JP8.1, RSQU_2.2, TP_13700_SQU2.P$1, VCO2BUF2.E
- removed net VCO13700_SUBBASS: IC1B.Q, JP7.1, RCAL_1.1
- removed net VCO13700_TRI: JP9.1, RTRI_2.2, TP_13700_TRI2.P$1, VCO2BUF1.E, VCO2OTA2.IN_N
- removed net VDD: C_DEC_10.2, C_DEC_11.2, C_DEC_12.2, C_DEC_13.2, C_DEC_14.2, C_DEC_8.2, C_DEC_9.2, C_DEC_POL3.+, C_DEC_POL4.+, DEBUG_CONN1.1, L_3V3_OUT1.2, UC1MCU.VBAT, UC1MCU.VDDA, UC1PWR.VDD@1, UC1PWR.VDD@2, UC1PWR.VDD@3, UC1PWR.VDD@4
- removed net VREF: CDEC-VREF-4.+, U2.VREFABCD, U2.VREFEFGH, U3.VREFABCD, U3.VREFEFGH, VREF_DAC_2V5.VOUT
- new net 3V3: C_DEC_1.2, C_DEC_2.2, C_DEC_3.2, C_DEC_4.2, C_DEC_5.2, C_DEC_6.2, C_TLV_OUT.+, DEBUG_CONN.1, I2C_PU_SCL.2, I2C_PU_SDA.2, IC2.A1, IC2.A2, IC2.VCC, L_3V3.2, R_RST.1, R_SW1A.1, R_SW2A.1, U1.VBAT, U1.VDDA/VREF+, U1.VDD_1, U1.VDD_2, U1.VDD_3, U1.VDD_4
- new net CALIB_3340C: U1.PA2
- new net FEEDBACK_VCF: CRES_VCF.1, IC1.D1, IC1.D2
- new net JACK_SUM_STG: COUT_SUM_STG.-, JACK_SUM_STG.2
- new net OSC_IN: R_HSE.1, U1.PH0-OSC_IN
- new net OSC_OUT: C2_HSE.2, U1.PH1-OSC_OUT, XTAL_HSE.2
- new net OUT_SUM_STG: OPAMP_SUM_STG.OUT, ROUT_SUM_STG.2, SUM_STG_C.1, SUM_STG_R.1
- new net POT2_SUM_STG: COUT_SUM_STG.+, POT_SUM_STG.S
- new net POT3_SUM_STG: POT_SUM_STG.E, ROUT_SUM_STG.1
- net +15V: now also C+15V_SUM_STG.2, CONN_ALIM.7, CONN_ALIM.8, C_DEC_ALIM_+15V.+, IC1.VDD, OPAMP_SUM_STG.V+; no longer C+15VPOL_VCF.2, CDEC+15V6.1, CDEC+15V7.1, EXPCONV2.V+, VCF_ANALOG_SWP.V+, VCO2SUPPLY.V+
- net -15V: now also C-15V_SUM_STG.1, CONN_ALIM.5, CONN_ALIM.6, C_DEC_ALIM_-15V.+, IC1.VSS, OPAMP_SUM_STG.V-, RB2_VCF.1; no longer CDEC-15V6.2, CDEC-15V7.2, EXPCONV2.V-, RB2.1, RBIAS_EXPCONV2.1, RSQU_2.1, RTRI_2.1, VCF_ANALOG_SWP.V-, VCO2SUPPLY.V-
- net 411_IN_PULSE: now also U1.PC9
- net 411_IN_SAW: now also U1.PC7
- net 411_IN_SYNC: now also U1.PC6
- net 411_IN_TRI: now also U1.PC8
- net 5V: now also CONN_ALIM.3, CONN_ALIM.4, C_DEC_ALIM_5V.+, C_IN_ALIM_POL.+, IC1.VL, REG3V3.EN, REG3V3.IN; no longer C5VPOL_VCF.1, CDEC-VREF-1.2, CDEC-VREF-2.-, CDEC_5V1.1, CDEC_5V4.1, IC1B.K, IC1P.VDD, IC_EEPROM.A1, IC_EEPROM.A2, IC_EEPROM.VCC, R1_8.1, R3_EXPCONV2.2, R_SW1A.1, R_SW2A.1, U2.VDD, U3.VDD, VCF_ANALOG_SWVL.VL, VREF_DAC_2V5.+VIN
- net AGND: now also C+15V_SUM_STG.1, C-15V_SUM_STG.2, JACK_SUM_STG.1, OPAMP_SUM_STG.+IN, POT_SUM_STG.A; no longer C+15VPOL_VCF.1, C+15V_VCF.1, C-15VPOL_VCF.2, C-15V_VCF.2, C10.1, C3.1, C4.1, C5.1, C5VPOL_VCF.2, C5V_VCF.2, CDEC+15V6.2, CDEC+15V7.2, CDEC-15V6.1, CDEC-15V7.1, CDEC-VREF-1.1, CDEC-VREF-2.+, CDEC-VREF-3.2, CDEC-VREF-4.-, CDEC_5V1.2, CDEC_5V4.2, CF_2.1, CONN_UART_RPI.1, EXPCONV2.+IN, IC1A.CLK, IC1A.J, IC1A.K, IC1A.R, IC1A.S, IC1B.R, IC1B.S, IC1P.VSS, IC_EEPROM.A0, IC_EEPROM.GND, IC_EEPROM.WP, R1_VCF.2, R2_8.2, R2_EXPCONV2.2, R4_EXPCONV2.2, RA_2.1, RCAL_2.2, REE_2.2, RTEST_LOG2.2, R_PD_4TH_ORDER_VCF.1, U2.GND, U3.GND, VCFPOW$1.GND, VCF_ANALOG_SWP.GND, VCO2OTA1.IN_N, VREF_DAC_2V5.GND, VREF_DAC_2V5.TRIM
- net BOOT1: now also U1.BOOT0; no longer UC1MCU.BOOT0
- net CALIB_3340A: now also U1.PA0
- net CALIB_3340B: now also U1.PA1
- net CV_CUTOFF: now also TRIM_VCF_CUT.E; no longer R2_VCF.2, U2.VOUTG
- net CV_FREQ_3340A: no longer U2.VOUTD
- net CV_FREQ_3340B: no longer U2.VOUTA
- net CV_PWM_3340A: no longer U2.VOUTH
- net CV_PWM_3340B: no longer U2.VOUTB
- net CV_RES: now also TRIM_VCF_RES.E, TRIM_VCF_RES.S; no longer R_RES_VCF.2, U2.VOUTF
- net CV_VCA: no longer U2.VOUTE
- net FREQ_CV_VCF: now also TRIM_VCF_CUT.S; no longer R1_VCF.1, R2_VCF.1
- net GAIN1_A: no longer U3.VOUTA
- net GAIN1_B: no longer U3.VOUTE
- net GAIN2_A: no longer U3.VOUTB
- net GAIN2_B: no longer U3.VOUTF
- net GAIN3_A: no longer U3.VOUTC
- net GAIN3_B: no longer U3.VOUTG
- net GAIN4_A: no longer U3.VOUTD
- net GAIN4_B: no longer U3.VOUTH
- net GND: now also C+15V_VCF.1, C-15V_VCF.2, C10.1, C1_HSE.1, C2_HSE.1, C3.1, C4.1, C5.1, C5V_VCF.2, CONN_ALIM.1, CONN_ALIM.2, C_DEC_1.1, C_DEC_2.1, C_DEC_3.1, C_DEC_4.1, C_DEC_5.1, C_DEC_6.1, C_DEC_ALIM_+15V.-, C_DEC_ALIM_-15V.-, C_DEC_ALIM_5V.-, C_IN_ALIM_POL.-, C_NRST.1, C_TLV_OUT.-, C_VCAP.1, DEBUG_CONN.5, IC1.D3, IC1.D4, IC1.GND, IC1.IN3, IC1.IN4, IC1.S3, IC1.S4, IC2.A0, IC2.GND, IC2.WP, REG3V3.GND, R_PD_4TH_ORDER_VCF.1, SW_RST.P, SW_RST.P1, TRIM_VCF_CUT.A, U1.VSSA/VREF-, U1.VSS_1, U1.VSS_2, U1.VSS_3, U1.VSS_4, VCFPOW$1.GND; no longer BTN_RST1.1, C1_HSE1.1, C1_LSE1.1, C2_HSE1.1, C2_LSE1.1, C_DEC_10.1, C_DEC_11.1, C_DEC_12.1, C_DEC_13.1, C_DEC_14.1, C_DEC_8.1, C_DEC_9.1, C_DEC_POL3.-, C_DEC_POL4.-, C_IN_ALIM1.2, C_IN_ALIM_POL1.-, C_NRST1.1, C_VCAP1.1, DEBUG_CONN1.5, REGUL3V1.GND, UC1MCU.VSSA, UC1PWR.VSS@1, UC1PWR.VSS@2, V_CAP2.1
- net IN2_MIXERA: no longer JP_OUT_VCO3340A2.1
- net IN2_MIXERB: no longer JP8.2
- net IN3_MIXERB: no longer JP9.2
- net IN3_VCF: now also RB2_VCF.2, RC3_VCF.1, RF3_VCF.1; no longer RB3_VCF.2, RC3.1, RF3.1
- net IN4_MIXERB: no longer JP7.2
- net IN4_VCF: now also RB3_VCF.2, RC4_VCF.1, RF4_VCF.1; no longer RB2.2, RC4.1, RF4.1
- net INPUT_CURRENT_SUM_STG: now also OPAMP_SUM_STG.-IN, SUM_STG_C.2, SUM_STG_HEADER1.1, SUM_STG_HEADER1.2, SUM_STG_HEADER1.3, SUM_STG_HEADER1.4, SUM_STG_HEADER1.5, SUM_STG_HEADER1.6, SUM_STG_HEADER1.7, SUM_STG_HEADER1.8, SUM_STG_R.2
- net IN_VCF: now also C_IN_VCF.2; no longer C_IN2.2
- net IN_VCFORDER: now also IC1.IN1, IC1.IN2; no longer VCF_ANALOG_SWA.IN, VCF_ANALOG_SWB.IN
- net N$1: now also JP_MIXER_B.2, MIXER_BG$2.I_OUT; no longer JP_OUT_VCO3340A1.1
- net N$104: now also C1_HSE.2, R_HSE.2, XTAL_HSE.1; no longer C1_HSE1.2, R_HSE1.2, XTAL_HSE1.1
- net N$108: now also REG3V3.OUT, R_3V3.2; no longer REGUL3V1.VOUT, R_3V3_OUT1.2
- net N$109: now also L_3V3.1, R_3V3.1; no longer L_3V3_OUT1.1, R_3V3_OUT1.1
- net N$116: now also C_IN_VCF.1; no longer C_IN2.1
- net N$3: now also JP_OUT_VCO3340A2.1; no longer CDEC-VREF-3.1, VREF_DAC_2V5.TEMP
- net N$6: now also U1.PA15, U1.PA4, U1.PA5, U1.PA7, U1.PB10, U1.PB12, U1.PB13, U1.PB14, U1.PB15, U1.PB6, U1.PB7, U1.PC1, U1.PC10, U1.PC2; no longer IC1B.!Q, IC1B.J
- net NRST: now also C_NRST.2, DEBUG_CONN.3, R_RST.2, SW_RST.S, SW_RST.S1, U1.NRST; no longer BTN_RST1.2, C_NRST1.2, DEBUG_CONN1.3, UC1MCU.NRST
- net OUT2_VCF: now also IC1.S1, RC3_VCF.2; no longer RC3.2, VCF_ANALOG_SWB.D
- net OUT3_VCF: now also RC4_VCF.2, RF3_VCF.2; no longer RC4.2, RF3.2
- net OUT4_VCF: now also IC1.S2, RF4_VCF.2; no longer RF4.2, VCF_ANALOG_SWA.D
- net RES_CUR_VCF: now also TRIM_VCF_RES.A; no longer R_RES_VCF.1
- net SCL: now also I2C_PU_SCL.1, IC2.SCL, U1.PB8; no longer IC_EEPROM.SCL
- net SDA: now also I2C_PU_SDA.1, IC2.SDA, U1.PB9; no longer IC_EEPROM.SDA
- net SWCLK: now also DEBUG_CONN.4, U1.PA14; no longer DEBUG_CONN1.4, UC1MCU.PA14
- net SWDIO: now also DEBUG_CONN.2, U1.PA13; no longer DEBUG_CONN1.2, UC1MCU.PA13
- net VCAP1: now also C_VCAP.2, U1.VCAP_1; no longer C_VCAP1.2, UC1MCU.VCAP2
- net VEE_VCF: no longer C-15VPOL_VCF.1
Other:
- note added: "Cut off at 11Hz"
- note added: "Note: for a polyphonic synth, voice summing is performed here on the inverting input of the op amp."
- note added: "Output summing stage"
- note added: "POWER"
- note added: "Protection againt short circuits"
- note added: "STM32F446"
- note removed: "Le courant de polarisation vaut -15/RBIAS"
- note removed: "On doit avoir la même tension que de l'autre côté quand on met 2V en entrée (milieu de la gamme)"
- note removed: "Position du jumper: * 2-1 : tester le convertisseur exponentiel * 2-3 : connecter le convertisseur exp au VCO LM13700"
- note removed: "SD-ON connected to PA15 (JTDI) that is in pull-up after reset"
- note removed: "VCF : attention le GND est a gauche (sens opposé des autres connecteurs) !!!"
- note removed: "VCO 13700 (square, triangle, subbass outputs)"
- moved on the sheet: C_SW1, C_SW2, RB3_VCF, R_BOOT1, R_PD_4TH_ORDER_VCF, R_SW1A, R_SW1B, R_SW2A, R_SW2B, S1, S2

Commit message: PCB for F446
Parts:
- removed 3: ADG411R, analog-devices:ADG411R
- removed C+15V_SUM_STG, C-15V_SUM_STG: 100n, rcl:C-EU075-032X103
- removed C+15V_VCF, C-15V_VCF, C5V_VCF: 100n, rcl:C-EUC0805
- removed C1_1, C2_1, C3_1, CIN1_MIXERA, CIN2_MIXERA, CIN2_MIXERB, CIN3_MIXERA, CIN3_MIXERB, CIN4_MIXERA, CIN4_MIXERB, CIN4_MIXERB1: 470n, rcl:C-EUC0603
- removed C1_HSE, C2_HSE: 12pF, MyComponents:C-US0805
- removed C1_SYNC1, C1_SYNC3, C_1, C_3: 1n, rcl:C-EUC0603
- removed C1_VCA, C2_VCA: 4.7u, rcl:C-EUC0603
- removed C2_SYNC1, C2_SYNC3, CDEC+15VPOL_MIXERB, CDEC+15V_MIXERB, CDEC-15VPOL_MIXERB, CDEC-15V_MIXERB, CDEC_3340A2, CDEC_3340A6, CDEC_3340B2, CDEC_3340B6, CDEC_411B6: 100n, rcl:C-EUC0603
- removed C4_1, C4_3, C_CV_FREQ_STAB1, C_CV_FREQ_STAB3: 10n, rcl:C-EUC0603
- removed CDEC_3340A3, CDEC_3340A7, CDEC_3340B3, CDEC_3340B7, CDEC_411B7: 10u, rcl:C-EUC0603
- removed CONN_ALIM, JP_MIXER_A, JP_MIXER_B, SUM_STG_HEADER, SUM_STG_HEADER1: (no value), con-lstb:MA04-2
- removed CONV_ITOV_OUT: NE5534AD, linear:NE5534AD
- removed COUT_SUM_STG: 22u, resistor:CPOL-EUB45181A
- removed CRES_VCF: 1u, rcl:C-EUC0805
- removed CSTAB1_MIXERA, CSTAB2_MIXERA, CSTAB2_MIXERB, CSTAB3, CSTAB3_MIXERA, CSTAB3_MIXERB, CSTAB4_MIXERA, CSTAB8: 560p, rcl:C-EUC0603
- removed C_CONV_ITOV_OUT: 1p, rcl:C-EUC0603
- removed C_DEC_1, C_DEC_2, C_DEC_3, C_DEC_4, C_DEC_5, C_NRST: 0.1uF, MyComponents:C-US0805
- removed C_DEC_6: 1.0uF, MyComponents:C-US0805
- removed C_DEC_ALIM_+15V, C_DEC_ALIM_-15V, C_DEC_ALIM_5V, C_IN_ALIM_POL: 10u, MyComponents:CPOL-US2917
- removed C_IN_VCF: 470n, rcl:C-EUC0805
- removed C_SW1, C_SW2: 100n, 6P1_EVB:C-EUC0805
- removed C_TLV_OUT: 100 uF, MyComponents:CPOL-US2917
- removed C_VCAP: 2.2uF, MyComponents:C-US0805
- removed DEBUG_CONN: 75867-331LF, MyComponents:MA03-2
- removed I2C_PU_SCL, I2C_PU_SDA: 1k, 6P1_EVB:R-US_R0805
- removed IC1: ADG453BRZ, ADG453BRZ:ADG453BRZ
- removed IC2: 24C04AP, microchip:24C04AP
- removed JACK_SUM_STG: 1502_01, con-lumberg:1502_01
- removed JP1, JP_FMLIN_VCO3340B1, JP_OUT_VCO3340A, JP_OUT_VCO3340A2, JP_PULSEOUT_VCO3340B, JP_SAWOUT_VCO3340B, JP_SYNC_3340B_TO_A, JP_TRIOUT_VCO3340B: JUMPER, 6P1_EVB:JUMPER
- removed L_3V3: 1 uH, MyComponents:L-USL0805
- removed MIXER_A, MIXER_B: SSM2164_MULTI, analog-audio-chips:SSM2164_MULTI
- removed OPAMP_SUM_STG: NE5534AN, linear:NE5534AN
- removed POT_SUM_STG: 100kB, pot:3RP/1610N
- removed R10_1, R10_3, RSTAB1_MIXERA, RSTAB2_MIXERA, RSTAB2_MIXERB, RSTAB3_MIXERA, RSTAB3_MIXERB, RSTAB4_MIXERA, RSTAB4_MIXERB, RSTAB4_MIXERB2, R_CV_FREQ_STAB1, R_CV_FREQ_STAB3: 470, rcl:R-EU_R0603
- removed R11_1, R11_3: 1.8k, rcl:R-EU_R0603
- removed R1S_1, R2S_1, R3S_1: 1k, rcl:R-EU_R0603
- removed R1_3, R1_4: 30k, rcl:R-EU_R0603
- removed R1_7, R2_7, R3_4, R5_VCA, R_PD_411_IN_PULSE1, R_PD_411_IN_SAW1, R_PD_411_IN_SYNC1, R_PD_411_IN_TRI1: 100k, rcl:R-EU_R0603
- removed R1_PWM1, R1_PWM3, R_CV_FREQ1, R_CV_FREQ3: 68k, rcl:R-EU_R0603
- removed R1_VCA, R2_VCA, R3_VCA, R4_VCA, R5_1, R5_3: 10k, rcl:R-EU_R0603
- removed R2_3, R2_4, R7_1, R7_3: 5.6k, rcl:R-EU_R0603
- removed R2_PWM1, R2_PWM3: 330k, rcl:R-EU_R0603
- removed R3_1, R3_3: 820, rcl:R-EU_R0603
- removed R6_1, R6_3: 33k, rcl:R-EU_R0603
- removed R8_1, R8_3: 1.5M, rcl:R-EU_R0603
- removed RB1_VCF, RB2_VCF, RB3_VCF: 220k, rcl:R-EU_R0805
- removed RC1_VCF, RC2_VCF, RC3_VCF, RC4_VCF: 91k, rcl:R-EU_R0805
- removed REE_VCF: 1.5k, rcl:R-EU_R0805
- removed REG3V3: TLV75533PDBVR, TLV75533PDBVR:TLV75533PDBVR
- removed RF1_VCF, RF2_VCF, RF3_VCF, RF4_VCF, R_PD_4TH_ORDER_VCF: 100k, rcl:R-EU_R0805
- removed RIN1_MIXERA, RIN2_MIXERA, RIN2_MIXERB, RIN3_MIXERA, RIN3_MIXERB, RIN4_MIXERA, RIN4_MIXERB, RIN4_MIXERB1: 27k, rcl:R-EU_R0603
- removed RMODE_MIXERA, RMODE_MIXERB: 8.2k, rcl:R-EU_R0603
- removed ROUT_SUM_STG: 470, rcl:R-EU_0207/12
- removed RRI_VCF: 51k, rcl:R-EU_R0805
- removed R_3V3: 1, MyComponents:R-US0805
- removed R_BOOT1: 10K, MyComponents:R-US0805
- removed R_CONV_ITOV_OUT: 33K, rcl:R-EU_R0603
- removed R_CV_FREQ_BIAS1, R_CV_FREQ_BIAS3: 270k, rcl:R-EU_R0603
- removed R_GAIN_VCA: 47k, rcl:R-EU_R0603
- removed R_HSE: 100, MyComponents:R-US0805
- removed R_RST: 100k, MyComponents:R-US0805
- removed R_SW1A, R_SW1B, R_SW2A, R_SW2B: 10k, 6P1_EVB:R-US_R0805
- removed R_SYNC1, R_SYNC3: 470k, rcl:R-EU_R0603
- removed S1, S2, SW_RST: (no value), switch-omron:10-XX
- removed SUM_STG_C: 560p, rcl:C-EU075-032X103
- removed SUM_STG_R: 27k, rcl:R-EU_0207/10
- removed TP_PULSE1, TP_PULSE3, TP_SAW1, TP_SAW3, TP_TRI1, TP_TRI3: (no value), 6P1_EVB:TESTPOINT
- removed TRIM_VCF_CUT, TRIM_VCF_RES: 100k, adafruit:TRIM
- removed U1: STM32F446RCT7, STM32F446RCT7:STM32F446RCT7
- removed VCF: AS3320, analog-audio-chips:AS3320
- removed VCF_JUMPER: (no value), con-lstb:MA04-1
- removed XTAL_HSE: 16MHz, MyComponents:Q-HSEHC-46X
- added 0V/5V/-15V/+15V, SUM_CON: (no value), con-lstb:MA04-2
- added 2164A, 2164B: SSM2164, analog-audio-chips:SSM2164
- added 24C04: 24C04AP, microchip:24C04AP
- added A010/9/8/7/3/4/5/6: (no value), con-lstb:MA08-1
- added A02/1/12/11, ABCD: (no value), con-lstb:MA04-1
- added A1, A2, A3, A4, B1, B2, B3, B4, SUB2, SUB4, SUB_IN, TRI_A, TRI_B: T, 6P1_EVB:TESTPOINT
- added AD5644: ANALOG_DEVICES_AD5644RBRMZ-5ANALOG_DEVICES_AD5644RBRMZ-5_0_0, Analog Devices - AD5644RBRMZ-5:ANALOG_DEVICES_AD5644RBRMZ-5ANALOG_DEVICES_AD5644RBRMZ-5_0_0
- added ADG453: ADG453BRZ, ADG453BRZ:ADG453BRZ
- added BH2221: BH2221FV, BH2221FV:BH2221FV
- added C1, C11, C16, C2, C33, C34, C39, C40, C51, C6, C9: 100n, rcl:C-EUC0805
- added C12, C13, C14, C15: 10n, rcl:C-EUC0805
- added C17, C18, C19, C20, C21, C22, C23, C24, C41: 470n, rcl:C-EUC0805
- added C25, C26, C27, C28, C29, C30, C31, C32: 560p, rcl:C-EUC0805
- added C35: 1p, rcl:C-EUC0805
- added C36, C37, C38: 4.7u, rcl:C-EUC0805
- added C42, C44: 1u, rcl:C-EUC0805
- added C43, C45, C49, C52: 300p, rcl:C-EUC0805
- added C46: 100p, rcl:C-EUC0805
- added C47, C48, C61, C72: 100n, rcl:C-EUC1206
- added C50: 22u, resistor:CPOL-EUB45181A
- added C53, C54, C58, C59, C62, C73: 10u, MyComponents:CPOL-US2917
- added C55, C66, C67, C68, C69, C70: 0.1uF, MyComponents:C-US0805
- added C56, C57: 12pF, MyComponents:C-US0805
- added C60: 2.2uF, MyComponents:C-US0805
- added C63, C64: 100n, 6P1_EVB:C-EUC0805
- added C65: 100 uF, MyComponents:CPOL-US2917
- added C7, C8: 1n, rcl:C-EUC0805
- added C71: 1.0uF, MyComponents:C-US0805
- added CAL_A, SYNC_A, SYNC_B: SYNC_IN, 6P1_EVB:TESTPOINT
- added CAL_B: CALIB B, 6P1_EVB:TESTPOINT
- added CAL_IN_A, CAL_IN_B, CUTOFF, IN10, IN9, MIXOUT, Q, VCA_CV, VCA_IN, VCA_OUT, VCF_IN, VCF_OUT, XIN, XMOD: (no value), 6P1_EVB:TESTPOINT
- added CV_A, CV_B: CV, 6P1_EVB:TESTPOINT
- added CV_TM, HIGH_A, HIGH_B, LOW_A, LOW_B, Q_TM: 100k, adafruit:TRIM
- added F446: STM32F446RCT7, STM32F446RCT7:STM32F446RCT7
- added FM_B: FMLIN, 6P1_EVB:TESTPOINT
- added GAINS: GAIN_CTRL, con-lstb:MA08-1
- added IN34: IN34, stm32_pi_board:MA02-1
- added ITOV, SUM_OPAMP: NE5534AN, linear:NE5534AN
- added I_SUM: ITOV, con-lstb:MA08-2
- added JACK: 1502_01, con-lumberg:1502_01
- added L1: 1 uH, MyComponents:L-USL0805
- added MODRING: LM13700M, ota:LM13700M
- added Q1: 16MHz, MyComponents:Q-HSEHC-46X
- added R1, R3: 330k, rcl:R-EU_R0805
- added R10, R9: 820, rcl:R-EU_R0805
- added R11, R12: 24k, rcl:R-EU_R0805
- added R13, R27: 470k, rcl:R-EU_R0805
- added R14, R15, R16, R17: 5.6k, rcl:R-EU_R0805
- added R18, R19: 1.8k, rcl:R-EU_R0805
- added R2, R4: 68k, rcl:R-EU_R0805
- added R20, R22, R23, R24, R32, R37, R38, R39, R40, R41, R42, R43, R73: 470, rcl:R-EU_R0805
- added R21: 1M, rcl:R-EU_R0805
- added R25, R26: 1.5M, rcl:R-EU_R0805
- added R28, R29, R30, R31, R33, R34, R35, R36, R46, R47, R58: 27k, rcl:R-EU_R0805
- added R44, R45: 8.2k, rcl:R-EU_R0805
- added R48: 33K, rcl:R-EU_R0805
- added R49, R53, R62, R66, R67, R68, R72, R74, R78: 100k, rcl:R-EU_R0805
- added R5, R51, R52, R6, R63: 10k, rcl:R-EU_R0805
- added R50, R56: 1k, rcl:R-EU_R0805
- added R54: 1.5k, rcl:R-EU_R0805
- added R55: 51k, rcl:R-EU_R0805
- added R57: 4.7k, rcl:R-EU_R0805
- added R59, R64, R70, R76: 91k, rcl:R-EU_R0805
- added R60, R69: 47k, rcl:R-EU_R0805
- added R61: 22k, rcl:R-EU_R0805
- added R65, R71, R77: 220k, rcl:R-EU_R0805
- added R7, R8: 33k, rcl:R-EU_R0805
- added R75: 100kB, pot:3RP/1610N
- added R79: 100k, MyComponents:R-US0805
- added R80: 100, MyComponents:R-US0805
- added R81: 10K, MyComponents:R-US0805
- added R82, R83, R85, R86: 10k, 6P1_EVB:R-US_R0805
- added R84, R88: 1k, 6P1_EVB:R-US_R0805
- added R87: 1, MyComponents:R-US0805
- added RST, SW1, SW2: (no value), switch-omron:10-XX
- added SAW_A, SAW_B: S, 6P1_EVB:TESTPOINT
- added SD3: SD3, stm32_pi_board:MA02-1
- added SD4: SD4, stm32_pi_board:MA02-1
- added SQU_A, SQU_B: P, 6P1_EVB:TESTPOINT
- added STLINK: 75867-331LF, MyComponents:MA03-2
- added SUB: 4027D, 40xx:4027D
- added TEMCOA, TEMCOB: 10k, adafruit:TRIM
- added TLV75533: TLV75533PDBVR, TLV75533PDBVR:TLV75533PDBVR
- added VCF1: AS3320, analog-audio-chips:AS3320
- C10, C5: value 300p -> 100n
- C3, C4: value 300p -> 1n
Connections:
- removed net 2164_MODE_MIXA: MIXER_AG$1.MODE, RMODE_MIXERA.2
- removed net 411_IN_PULSE: 3D.IN, R_PD_411_IN_PULSE1.2, U1.PC9
- removed net 411_IN_SAW: 3C.IN, R_PD_411_IN_SAW1.1, U1.PC7
- removed net 411_IN_SYNC: 3B.IN, R_PD_411_IN_SYNC1.1, U1.PC6
- removed net 411_IN_TRI: 3A.IN, R_PD_411_IN_TRI1.1, U1.PC8
- removed net AGND: 3340A.GND, 3340B.GND, 3P.GND, C+15V_SUM_STG.1, C-15V_SUM_STG.2, C1_VCA.2, C2_SYNC1.1, C2_SYNC3.1, C4_1.2, C4_3.2, CDEC+15VPOL_MIXERB.1, CDEC+15V_MIXERB.1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
- removed net CALIB_3340C: U1.PA2
- removed net FREQ_CTRL_VCOA: 3340A.FREQ_CTRL, R_CV_FREQ3.1, R_CV_FREQ_BIAS3.1, R_CV_FREQ_STAB3.1
- removed net FREQ_CTRL_VCOB: 3340B.FREQ_CTRL, R_CV_FREQ1.1, R_CV_FREQ_BIAS1.1, R_CV_FREQ_STAB1.1
- removed net HARD_SYNC_VCOA: 3340A.HARD_SYNC, C1_SYNC3.2
- removed net HARD_SYNC_VCOB: 3340B.HARD_SYNC, C1_SYNC1.2
- removed net IN4_MIXERA: CIN4_MIXERA.1, JP_PULSEOUT_VCO3340B.2
- removed net INPUT_CURRENT_SUM_STG: JP1.1, JP1.2, OPAMP_SUM_STG.-IN, SUM_STG_C.2, SUM_STG_HEADER.2, SUM_STG_HEADER.4, SUM_STG_HEADER.6, SUM_STG_HEADER.8, SUM_STG_HEADER1.1, SUM_STG_HEADER1.2, SUM_STG_HEADER1.3, SUM_STG_HEADER1.4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
- removed net IN_VCA: R1_VCA.1, VCF_JUMPER.2
- removed net JACK_SUM_STG: COUT_SUM_STG.-, JACK_SUM_STG.2
- removed net LINEAR_CTRL_VCOA: 3340A.LINEAR_CTRL, R10_3.1, R8_3.1
- removed net LINEAR_CTRL_VCOB: 3340B.LINEAR_CTRL, R10_1.1, R8_1.1
- removed net MIXER_OUT1: CONV_ITOV_OUT.-IN, C_CONV_ITOV_OUT.1, JP_MIXER_A.1, JP_MIXER_A.3, JP_MIXER_A.5, JP_MIXER_A.7, JP_MIXER_B.1, JP_MIXER_B.3, JP_MIXER_B.5, JP_MIXER_B.7, R_CONV_ITOV_OUT.1
- removed net N$82: C_CV_FREQ_STAB1.2, R_CV_FREQ_STAB1.2
- removed net N$83: C4_1.1, R10_1.2
- removed net N$86: C_CV_FREQ_STAB3.2, R_CV_FREQ_STAB3.2
- removed net N$87: C4_3.1, R10_3.2
- removed net N$88: 3A.D, C1_1.2, R1_7.2
- removed net N$89: 3D.D, C2_1.2, R2_7.2
- removed net N$90: 3C.D, C3_1.2, R3_4.2
- removed net N$91: 3D.S, R2S_1.2
- removed net OUT_SUM_STG: OPAMP_SUM_STG.OUT, ROUT_SUM_STG.2, SUM_STG_C.1, SUM_STG_R.1
- removed net POT2_SUM_STG: COUT_SUM_STG.+, POT_SUM_STG.S
- removed net POT3_SUM_STG: POT_SUM_STG.E, ROUT_SUM_STG.1
- removed net PULSE_OUT_VCOA: 3C.S, R3S_1.2
- removed net PULSE_VCOA: 3340A.PULSE_OUT, C3_1.1, R6_3.2, TP_PULSE3.P$1
- removed net SAW_3340_VCOA: C2_1.1, R7_3.1, TP_SAW3.P$1
- removed net SAW_VCOA: 3340A.SAW_OUT, R7_3.2
- removed net SAW_VCOB: 3340B.SAW_OUT, R7_1.2
- removed net SCALE_VCOA: 3340A.SCALE, R11_3.1
- removed net SCALE_VCOB: 3340B.SCALE, R11_1.1
- removed net SOFT_SYNC_VCOA: 3340A.SOFT_SYNC, C2_SYNC3.2
- removed net SOFT_SYNC_VCOB: 3340B.SOFT_SYNC, C2_SYNC1.2
- removed net SYNC_3340_VCOA: 3B.D, C1_SYNC3.1, R_SYNC3.2
- removed net SYNC_3340_VCOB: C1_SYNC1.1, R_SYNC1.2
- removed net SYNC_IN_VCOA: 3B.S, JP_SYNC_3340B_TO_A.1
- removed net TEMPCO1_VCOA: 3340A.MUL_GAIN1, R1_4.1
- removed net TEMPCO1_VCOB: 3340B.MUL_GAIN1, R1_3.1
- removed net TIMING_CAP_VCOA: 3340A.TIMING_CAP, C_3.2
- removed net TIMING_CAP_VCOB: 3340B.TIMING_CAP, C_1.2
- removed net TRI_3340_VCOA: 3340A.TRI_OUT, C1_1.1, TP_TRI3.P$1
- removed net TRI_OUT_VCOA: 3A.S, R1S_1.1
- removed net VCO3340B_PULSE_OUT: 3340B.PULSE_OUT, JP_PULSEOUT_VCO3340B.1, R6_1.2, TP_PULSE1.P$1
- removed net VCO3340B_SAW_OUT: JP_SAWOUT_VCO3340B.1, JP_SYNC_3340B_TO_A.2, R7_1.1, TP_SAW1.P$1
- removed net VCO3340B_TRI_OUT: 3340B.TRI_OUT, JP_TRIOUT_VCO3340B.1, TP_TRI1.P$1
- removed net VCO440A_OUT: JP_OUT_VCO3340A.1, R1S_1.2, R2S_1.1, R3S_1.1
- new net AD5644_CLK: AD5644.SCLK, F446.PB10
- new net AD5644_DI: AD5644.DIN, F446.PC1
- new net AD5644_SYNC: AD5644.!SYNC!, F446.PB12
- new net BH2221_CLK: BH2221.CLK, F446.PA5
- new net BH2221_DI: BH2221.DI, F446.PA7
- new net BH2221_LD: BH2221.LD, F446.PA4
- new net CALIB_IN_3340A: CAL_IN_A.P$1, F446.PA0
- new net CALIB_IN_3340B: CAL_IN_B.P$1, F446.PA1
- new net FMLIN_3340B: C11.2, FM_B.P$1
- new net FREQ_CTRL_3340A: 3340A.FREQ_CTRL, HIGH_A.A, HIGH_A.S, LOW_A.A, LOW_A.S, R24.1
- new net FREQ_CTRL_3340B: 3340B.FREQ_CTRL, HIGH_B.A, HIGH_B.S, LOW_B.A, LOW_B.S, R23.1
- new net HEADIN_OPAMP_OUT: C46.2, R69.2, SUM_CON.1, SUM_CON.2, SUM_CON.3, SUM_CON.4, SUM_CON.5, SUM_CON.6, SUM_CON.7, SUM_CON.8, SUM_OPAMP.-IN
- new net IOUT_VCA: VCAOTA1.OUT, VCA_OUT.P$1
- new net ITOV_IN: C35.1, ITOV.-IN, I_SUM.1, I_SUM.11, I_SUM.13, I_SUM.15, I_SUM.3, I_SUM.5, I_SUM.7, I_SUM.9, R46.1, R47.1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
- new net LINEAR_CTRL_3340A: 3340A.LINEAR_CTRL, R22.1, R26.1
- new net LINEAR_CTRL_3340B: 3340B.LINEAR_CTRL, R20.1, R21.1, R25.1
- new net N$14: IN9.P$1, R46.2
- new net N$15: IN10.P$1, R47.2
- new net N$16: ADG453.D4, SD4.1
- new net N$171: C12.2, R23.2
- new net N$172: C14.1, R20.2
- new net N$173: 3340B.MUL_GAIN1, TEMCOB.A
- new net N$174: R11.1, TEMCOB.E, TEMCOB.S
- new net N$175: C11.1, R21.2
- new net N$176: 3340B.SAW_OUT, R14.2
- new net N$18: ADG453.S3, SD3.1
- new net N$19: A010/9/8/7/3/4/5/6.5, BH2221.AO3
- new net N$21: A010/9/8/7/3/4/5/6.6, BH2221.AO4
- new net N$23: A010/9/8/7/3/4/5/6.7, BH2221.AO5
- new net N$25: A010/9/8/7/3/4/5/6.8, BH2221.AO6
- new net N$26: A010/9/8/7/3/4/5/6.4, BH2221.AO7
- new net N$27: A010/9/8/7/3/4/5/6.3, BH2221.AO8
- new net N$28: A010/9/8/7/3/4/5/6.2, BH2221.AO9
- new net N$29: A010/9/8/7/3/4/5/6.1, BH2221.AO10
- new net N$30: A02/1/12/11.1, BH2221.AO2
- new net N$301: C13.2, R24.2
- new net N$302: C15.1, R22.2
- new net N$303: 3340A.MUL_GAIN1, TEMCOA.A
- new net N$304: R12.1, TEMCOA.E, TEMCOA.S
- new net N$306: 3340A.SAW_OUT, R15.2
- new net N$307: 3340A.HARD_SYNC, C4.2
- new net N$31: A02/1/12/11.2, BH2221.AO1
- new net N$32: A02/1/12/11.3, BH2221.AO12
- new net N$33: A02/1/12/11.4, BH2221.AO11
- new net N$34: ABCD.1, AD5644.VOUTA
- new net N$35: ABCD.2, AD5644.VOUTB
- new net N$36: ADG453.D3, SD3.2
- new net N$37: ADG453.IN3, IN34.1, R72.1
- new net N$38: 2164A.MODE, R45.2
- new net N$39: ABCD.3, AD5644.VOUTC
- new net N$40: ABCD.4, AD5644.VOUTD
- new net N$41: SUBA.!Q, SUBA.J
- new net N$42: C16.1, SUBA.K, SUBB.K, SUBP.VDD
- new net N$43: C38.1, R53.1
- new net N$44: MODRINGBUF2.E, R63.2
- new net N$45: C42.1, MODRINGOTA2.I_BIAS, R60.1
- new net N$46: C42.2, R57.1
- new net N$47: C36.1, R50.1, VCAOTA1.IN_P
- new net N$49: R57.2, XMOD.P$1
- new net N$50: C38.2, XIN.P$1
- new net N$51: MODRINGBUF2.B, MODRINGOTA2.OUT, R61.2
- new net N$8: C3.1, R13.2, SYNC_B.P$1
- new net N$9: ADG453.S4, SD4.2
- new net OUT_JACK: C50.-, JACK.2, JACK.3
- new net OUT_OPAMP: C46.1, R69.1, R73.2, SUM_OPAMP.OUT
- new net OUT_POT: C50.+, R73.1, R75.E, R75.S
- new net PULSE_3340A: 3340A.PULSE_OUT, R8.2, SQU_A.P$1
- new net PULSE_3340B: 3340B.PULSE_OUT, R7.2, SQU_B.P$1
- new net SAW_3340A: R15.1, SAW_A.P$1
- new net SAW_3340B: R14.1, SAW_B.P$1
- new net SCALE_3340A: 3340A.SCALE, R19.1
- new net SCALE_3340B: 3340B.SCALE, R18.1
- new net SOFT_SYNC_3340A: 3340A.SOFT_SYNC, C10.2
- new net SOFT_SYNC_3340B: 3340B.SOFT_SYNC, C9.2
- new net SUB_IN: SUBA.CLK, SUB_IN.P$1
- new net SUB_OUT2: SUB2.P$1, SUBA.Q, SUBB.CLK
- new net SUB_OUT4: SUB4.P$1, SUBB.Q
- new net SYNC_3340A: C4.1, R27.2, SYNC_A.P$1
- new net TIMING_CAP_3340A: 3340A.TIMING_CAP, C8.2
- new net TIMING_CAP_3340B: 3340B.TIMING_CAP, C7.2
- new net TRI_3340A: 3340A.TRI_OUT, TRI_A.P$1
- new net TRI_3340B: 3340B.TRI_OUT, TRI_B.P$1
- new net VCA_IN: R49.1, VCA_IN.P$1
- new net VCF_ANASW_IN4: ADG453.IN4, IN34.2, R66.2
- net +15V: now also 0V/5V/-15V/+15V.7, 0V/5V/-15V/+15V.8, 2164A.V+, 2164B.V+, ADG453.VDD, C33.2, C39.2, C47.2, C5.2, C53.+, C6.2, ITOV.V+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; no longer 3P.VDD, C+15V_SUM_STG.2, C+15V_VCF.2, CDEC+15VPOL_MIXERB.2, CDEC+15V_MIXERB.2, CDEC_3340A2.2, CDEC_3340A3.2, CDEC_3340A6.2, CDEC_3340A7.2, CONN_ALIM.7, CONN_ALIM.8, CONV_ITOV_OUT.V+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
- net -15V: now also 0V/5V/-15V/+15V.5, 0V/5V/-15V/+15V.6, 2164A.V-, 2164B.V-, ADG453.VSS, C34.1, C48.1, C54.+, ITOV.V-, MODRINGSUPPLY.V-, R10.1, R54.1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; no longer 3P.VSS, C-15V_SUM_STG.1, CDEC-15VPOL_MIXERB.1, CDEC-15V_MIXERB.1, CONN_ALIM.5, CONN_ALIM.6, CONV_ITOV_OUT.V-, C_DEC_ALIM_-15V.+, IC1.VSS, MIXER_AG$1.V-, MIXER_BG$1.V-, OPAMP_SUM_STG.V-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
- net 2164_IN1_MIXA: now also 2164A.I_IN1, R33.1, R40.1; no longer MIXER_AG$2.I_IN, RIN1_MIXERA.1, RSTAB1_MIXERA.1
- net 2164_IN2_MIXA: now also 2164A.I_IN2, R34.1, R41.1; no longer MIXER_AG$3.I_IN, RIN2_MIXERA.1, RSTAB2_MIXERA.1
- net 2164_IN2_MIXB: now also 2164B.I_IN2, R29.1, R37.1; no longer MIXER_BG$3.I_IN, RIN2_MIXERB.1, RSTAB2_MIXERB.1
- net 2164_IN3_MIXA: now also 2164A.I_IN3, R35.1, R42.1; no longer MIXER_AG$5.I_IN, RIN3_MIXERA.1, RSTAB3_MIXERA.1
- net 2164_IN3_MIXB: now also 2164B.I_IN3, R30.1, R38.1; no longer MIXER_BG$5.I_IN, RIN3_MIXERB.1, RSTAB3_MIXERB.1
- net 2164_IN4_MIXA: now also 2164A.I_IN4, R36.1, R43.1; no longer MIXER_AG$4.I_IN, RIN4_MIXERA.1, RSTAB4_MIXERA.1
- net 2164_IN4_MIXB: now also 2164B.I_IN4, R31.1, R39.1; no longer MIXER_BG$4.I_IN, RIN4_MIXERB.1, RSTAB4_MIXERB.1
- net 2164_IN4_MIXB1: now also 2164B.I_IN1, R28.1, R32.1; no longer MIXER_BG$2.I_IN, RIN4_MIXERB1.1, RSTAB4_MIXERB2.1
- net 2164_MODE_MIXB: now also 2164B.MODE, R44.2; no longer MIXER_BG$1.MODE, RMODE_MIXERB.2
- net 2164_OUT2_MIXA: now also 2164A.I_OUT2, I_SUM.4; no longer JP_MIXER_A.2, MIXER_AG$3.I_OUT
- net 2164_OUT2_MIXB: now also 2164B.I_OUT2, I_SUM.14; no longer JP_MIXER_B.4, MIXER_BG$3.I_OUT
- net 2164_OUT3_MIXA: now also 2164A.I_OUT3, I_SUM.8; no longer JP_MIXER_A.6, MIXER_AG$5.I_OUT
- net 2164_OUT3_MIXB: now also 2164B.I_OUT3, I_SUM.16; no longer JP_MIXER_B.8, MIXER_BG$5.I_OUT
- net 2164_OUT4_MIXA: now also 2164A.I_OUT4, I_SUM.6; no longer JP_MIXER_A.8, MIXER_AG$4.I_OUT
- net 2164_OUT4_MIXB: now also 2164B.I_OUT4, I_SUM.12; no longer JP_MIXER_B.6, MIXER_BG$4.I_OUT
- net 3V3: now also 24C04.A1, 24C04.A2, 24C04.VCC, C65.+, C66.2, C67.2, C68.2, C69.2, C70.2, C71.2, F446.VBAT, F446.VDDA/VREF+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; no longer C_DEC_1.2, C_DEC_2.2, C_DEC_3.2, C_DEC_4.2, C_DEC_5.2, C_DEC_6.2, C_TLV_OUT.+, DEBUG_CONN.1, I2C_PU_SCL.2, I2C_PU_SDA.2, IC2.A1, IC2.A2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
- net 5V: now also 0V/5V/-15V/+15V.3, 0V/5V/-15V/+15V.4, AD5644.VDD, ADG453.VL, BH2221.VCC, BH2221.VDD, C51.1, C58.+, C59.+, C61.2, C62.+, C72.2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; no longer 3P.VL, C5V_VCF.1, CDEC_411B6.1, CDEC_411B7.1, CONN_ALIM.3, CONN_ALIM.4, C_DEC_ALIM_5V.+, C_IN_ALIM_POL.+, IC1.VL, REG3V3.EN, REG3V3.IN, R_PD_411_IN_SAW1.2
- net BIAS_VCA: now also C37.1, R50.2, R51.2, R52.1, SUM_OPAMP.+IN, VCAOTA1.IN_N; no longer C1_VCA.1, C2_VCA.1, R3_VCA.1, R4_VCA.2, R5_VCA.1, VCAOTA1.IN_P
- net BOOT1: now also F446.BOOT0, R81.1; no longer R_BOOT1.1, U1.BOOT0
- net CALIB_3340A: now also CAL_A.P$1, R6.1, R8.1; no longer R5_3.1, R6_3.1, U1.PA0
- net CALIB_3340B: now also CAL_B.P$1, R5.1, R7.1; no longer R5_1.1, R6_1.1, U1.PA1
- net CAP1_VCF: now also C43.2, VCF1OTA$1.CAP; no longer C3.2, VCFOTA$1.CAP
- net CAP2_VCF: now also C45.2, VCF1OTA$2.CAP; no longer C5.2, VCFOTA$2.CAP
- net CAP3_VCF: now also C49.2, VCF1OTA$4.CAP; no longer C4.2, VCFOTA$4.CAP
- net CAP4_VCF: now also C52.2, VCF1OTA$3.CAP; no longer C10.2, VCFOTA$3.CAP
- net CV_CUTOFF: now also CUTOFF.P$1, CV_TM.E; no longer TRIM_VCF_CUT.E
- net CV_FREQ_3340A: now also CV_A.P$1, HIGH_A.E; no longer JP_FMLIN_VCO3340B1.1, R_CV_FREQ3.2
- net CV_FREQ_3340B: now also CV_B.P$1, HIGH_B.E; no longer R_CV_FREQ1.2
- net CV_PWM_3340A: now also R3.1, R4.1; no longer R1_PWM3.1, R2_PWM3.1
- net CV_PWM_3340B: now also R1.1, R2.1; no longer R1_PWM1.1, R2_PWM1.1
- net CV_RES: now also Q.P$1, Q_TM.E, Q_TM.S; no longer TRIM_VCF_RES.E, TRIM_VCF_RES.S
- net CV_VCA: now also R58.1, VCA_CV.P$1; no longer R_GAIN_VCA.1
- net FEEDBACK_VCF: now also ADG453.D1, ADG453.D2, C44.1; no longer CRES_VCF.1, IC1.D1, IC1.D2
- net FREQ_CV_VCF: now also CV_TM.S, VCF1POW$1.FREQ_CV; no longer TRIM_VCF_CUT.S, VCFPOW$1.FREQ_CV
- net GAIN1_A: now also 2164A.GAIN_VCA1, GAINS.8; no longer MIXER_AG$2.GAIN_VCA
- net GAIN1_B: now also 2164B.GAIN_VCA1, GAINS.4; no longer MIXER_BG$2.GAIN_VCA
- net GAIN2_A: now also 2164A.GAIN_VCA2, GAINS.5; no longer MIXER_AG$3.GAIN_VCA
- net GAIN2_B: now also 2164B.GAIN_VCA2, GAINS.1; no longer MIXER_BG$3.GAIN_VCA
- net GAIN3_A: now also 2164A.GAIN_VCA3, GAINS.6; no longer MIXER_AG$5.GAIN_VCA
- net GAIN3_B: now also 2164B.GAIN_VCA3, GAINS.2; no longer MIXER_BG$5.GAIN_VCA
- net GAIN4_A: now also 2164A.GAIN_VCA4, GAINS.7; no longer MIXER_AG$4.GAIN_VCA
- net GAIN4_B: now also 2164B.GAIN_VCA4, GAINS.3; no longer MIXER_BG$4.GAIN_VCA
- net GND: now also 0V/5V/-15V/+15V.1, 0V/5V/-15V/+15V.2, 2164A.GND, 2164B.GND, 24C04.A0, 24C04.GND, 24C04.WP, 3340A.GND, 3340B.GND, AD5644.GND, ADG453.GND, BH2221.GND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; no longer C+15V_VCF.1, C-15V_VCF.2, C1_HSE.1, C2_HSE.1, C3.1, C4.1, C5V_VCF.2, CONN_ALIM.1, CONN_ALIM.2, C_DEC_1.1, C_DEC_2.1, C_DEC_3.1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
- net IN1_MIXERA: now also A1.P$1, C18.1; no longer CIN1_MIXERA.1, JP_TRIOUT_VCO3340B.2
- net IN1_VCF: now also R59.2, R62.2, VCF1OTA$1.IN; no longer RC1_VCF.2, RF1_VCF.2, VCFOTA$1.IN
- net IN2_MIXERA: now also A2.P$1, C20.1; no longer CIN2_MIXERA.1, JP_OUT_VCO3340A.2
- net IN2_MIXERB: now also B2.P$1, C17.1; no longer CIN2_MIXERB.1
- net IN2_VCF: now also R64.1, R65.2, R67.1, VCF1OTA$2.IN; no longer RB1_VCF.2, RC2_VCF.1, RF2_VCF.1, VCFOTA$2.IN
- net IN3_MIXERA: now also A3.P$1, C23.1; no longer CIN3_MIXERA.1, JP_SAWOUT_VCO3340B.2
- net IN3_MIXERB: now also B3.P$1, C21.1; no longer CIN3_MIXERB.1
- net IN3_VCF: now also R70.1, R71.2, R74.1, VCF1OTA$4.IN; no longer RB2_VCF.2, RC3_VCF.1, RF3_VCF.1, VCFOTA$4.IN
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Other:
- note added: "Channels: A01-12 = 8 bits B01-04 = 14 bits - A01 à A08 : 2164D vca - A09 : VCF cutoff - A10 : VCF Q - A11 : PWM 3340A - A12 : PWM 3340B - B01 : CV 3340A - B02 : CV 3340B - B03 : noise / wave generator (VCO #3) - B04 : VCA LM13700"
- note added: "Connecté sur SPI1: - CLK=PA5 - MOSI=PA7 - NSS=PA4"
- note added: "Connecté sur SPI2: - CLK=PB10 - MOSI=PC1 - NSS=PB12"
- note added: "DAC (12 ch 8 bits + 4 ch 14 bits)"
- note added: "MOD RING"
- note added: "VCO3340B (multiwave output)"
- note removed: "C2_SYNC protège l'entrée soft sync contre le bruit"
- note removed: "Cut off at 11Hz"
- note removed: "FM lin non utilisée"
- note removed: "SAW is the only active output when nothing is plugged from the STM32."
- note removed: "VCO3340B (pulse, saw, triangle outputs)"
- note removed: "Values for R?S_411 depend on the level of the signal we wanna have at V2164's output."

Commit message: PCB update
Parts:
- added +15V, -15V, GREEN: (no value), Passives:LED-0805
- added 5V, RED1, RED2: (no value), Passives:LED-0603
- added I2C, MIDI: (no value), con-lstb:MA03-1
- added R89, R90, R91, R92, R93, R94: 330, MyComponents:R-US0805
Connections:
- new net LED1_PWM: F446.PA6, R90.1
- new net LED2_PWM: F446.PC7, R89.1
- new net LED3_PWM: F446.PB0, R91.1
- new net N$48: R89.2, RED1.A
- new net N$52: R91.2, RED2.A
- new net N$53: 5V.A, R92.2
- new net N$54: -15V.A, R93.2
- new net N$55: +15V.A, R94.2
- new net N$56: GREEN.A, R90.2
- new net USART1_RX: F446.PB7, MIDI.1
- new net USART1_TX: F446.PB6, MIDI.2
- net +15V: now also R94.1
- net -15V: now also R93.1
- net 5V: now also R92.1
- net GND: now also +15V.C, -15V.C, 5V.C, GREEN.C, I2C.3, MIDI.3, RED1.C, RED2.C
- net SCL: now also I2C.2
- net SDA: now also I2C.1
- net SW1: now also F446.PC9
- net SW2: now also F446.PC8

Commit message: Final PCB version sent to eurocircuits.com
Parts:
- removed C47, C48: 100n, rcl:C-EUC1206
- added 3V3: (no value), Passives:LED-0805
- added ANAIN: (no value), stm32_pi_board:MA02-1
- added C74, C75, C76, C77, C78, C79, C80, C81, C82, C83, C84, C85, C86, C87, C88: 1u, rcl:C-EUC1206
- added EXT: (no value), con-lstb:MA04-1
- added HOLE1, HOLE2, HOLE3, HOLE4: HOLES_MOUNT-PAD-ROUND-0.096-NS, 52101-101-REV-A:HOLES_MOUNT-PAD-ROUND-0.096-NS
- added R95: 330, MyComponents:R-US0805
Connections:
- new net EXT1: EXT.1, F446.PA15
- new net EXT2: EXT.2, F446.PC10
- new net EXT3: EXT.3, F446.PC11
- new net EXT4: EXT.4, F446.PC12
- new net N$57: 3V3.A, R95.2
- new net N$58: ANAIN.2, F446.PA2
- new net N$59: ANAIN.1, F446.PA3
- net +15V: now also C74.2, C77.2, C78.2, C79.2, C80.2, C81.2, C82.2, C83.2; no longer C47.2
- net -15V: now also C75.2, C84.2, C85.2, C86.2, C87.2, C88.2; no longer C48.1
- net 3V3: now also R95.1
- net 5V: now also C76.2
- net GND: now also 3V3.C, C74.1, C75.1, C76.1, C77.1, C78.1, C79.1, C80.1, C81.1, C82.1, C83.1, C84.1, C85.1, C86.1, C87.1, C88.1; no longer C47.1, C48.2
Other:
- moved on the sheet: C53
