File: eagle-schematics/themis-v2/Pysical_interface/shématic.sch (EAGLE design)
At the start: 35 parts, among them IC1 MCP23017SO, SW1 EC12E_SW, SW2 EC12E_SW, SW3 EC12E_SW, SW4 EC12E_SW

Commit message: Updated PCB
Parts:
- removed C1_E1, C1_E2, C1_E3, C1_E4, C1_E5, C1_E6, C1_E7, C1_E8, C2_E1, C2_E2, C2_E3, C2_E4: 100n, rcl:C-EU025-024X044
- removed NEOPIXEL1: NEOPIXEL12, Neopixel:NEOPIXEL12
- removed R1_E1, R1_E2, R1_E3, R1_E4, R1_E5, R1_E6, R1_E7, R1_E8, R2_E1, R2_E2, R2_E3, R2_E4: 100k, resistor:R-EU_0204/5
- removed RDIS1, RDIS2, RDIS3, RDIS4: 1k, resistor:R-EU_0204/5
- removed SW1: EC12E_SW, switch-alps:EC12E_SW
- added CA1, CA2, CA3, CA4, CA6, CA8, CB1, CB2, CB3, CB4, CB6, CB8, CC1, CC2, CC3, CC4, CC6, CC8: 100n, rcl:C-EUC1210
- added LED10, LED11, LED12, LED13, LED14, LED15, LED16, LED17, LED18, LED19, LED20, LED21, LED22, LED23, LED24, LED25, LED26, LED27, LED28, LED29, LED30, LED31, LED32, LED33, LED34, LED35, LED36, LED37, LED38, LED39, LED40, LED41, LED42, LED43, LED44, LED45, LED55, LED56, LED57, LED58, LED59, LED60, LED61, LED62, LED63, LED73, LED74, LED75, LED76, LED77, LED78, LED79, LED80, LED81: WS2812B5050, WS2812B:WS2812B5050
- added R_DISA1, R_DISA2, R_DISA3, R_DISA4, R_DISA6, R_DISA8, R_DISB1, R_DISB2, R_DISB3, R_DISB4, R_DISB6, R_DISB8: 1k, rcl:R-US_R1210
- added R_PDA1, R_PDA2, R_PDA3, R_PDA4, R_PDA6, R_PDA8, R_PUB1, R_PUB2, R_PUB3, R_PUB4, R_PUB6, R_PUB8, R_PUC1, R_PUC2, R_PUC3, R_PUC4, R_PUC6, R_PUC8: 100k, rcl:R-US_R1210
- added SW5, SW7, SW9: EC12E_SW, switch-alps:EC12E_SW
- added TP1, TP2, TP3, TP4: PTR1PAD1-13Y, testpad:PTR1PAD1-13Y
Connections:
- net INTA renamed INTROT_2
- net N$3 renamed INTROT1
- removed net BOUT_1: C1_E6.1, IC1.GPA0, R1_E6.2, SW3G$2.2
- removed net BOUT_2: C1_E2.1, IC1.GPA3, R1_E2.2, SW1G$2.2
- removed net BOUT_3: C1_E4.1, IC1.GPA6, R1_E4.2, SW2G$2.2
- removed net BOUT_4: C1_E8.1, IC1.GPB1, R1_E8.2, SW4G$2.2
- removed net DISCHARGE: RDIS1.1, RDIS2.1, RDIS3.1, RDIS4.1, SW1G$1.C, SW2G$1.C, SW3G$1.C, SW4G$1.C
- removed net EC1_1: C2_E3.1, IC1.GPA1, R2_E3.2, SW3G$1.A
- removed net EC1_2: C1_E5.1, IC1.GPA2, R1_E5.2, SW3G$1.B
- removed net EC2_1: C2_E1.1, IC1.GPA4, R2_E1.2, SW1G$1.A
- removed net EC2_2: C1_E1.1, IC1.GPA5, R1_E1.2, SW1G$1.B
- removed net EC3_1: C2_E2.1, IC1.GPA7, R2_E2.2, SW2G$1.A
- removed net EC3_2: C1_E3.1, IC1.GPB0, R1_E3.2, SW2G$1.B
- removed net EC4_1: C2_E4.1, IC1.GPB2, R2_E4.2, SW4G$1.A
- removed net EC4_2: C1_E7.1, IC1.GPB3, R1_E7.2, SW4G$1.B
- removed net INTB: IC1.INTB, U$2.A5
- removed net SPI1_DATA: NEOPIXEL1.P$IN, U$2.A6
- new net CLICK_1: CC1.2, IC1.GPA6, R_PUC1.1, SW2G$2.2
- new net CLICK_2: CC2.2, IC1.GPA7, R_PUC2.1, SW3G$2.2
- new net CLICK_3: CC3.2, IC1.GPB6, R_PUC3.1, SW4G$2.2
- new net CLICK_4: CC4.2, IC1.GPB7, R_PUC4.1, SW5G$2.2
- new net CLICK_5: CC6.2, R_PUC6.1, SW7G$2.2, U$2.A3
- new net CLICK_6: CC8.2, R_PUC8.1, SW9G$2.2, U$2.A2
- new net INTROT2: IC1.INTB
- new net INTROT_1: U$2.A5
- new net N$11: LED11.DO, LED12.DI
- new net N$12: LED12.DO, LED13.DI
- new net N$13: LED13.DO, LED14.DI
- new net N$16: R_DISB1.1, SW2G$1.A
- new net N$17: R_DISA1.1, SW2G$1.B
- new net N$18: LED17.DO, LED18.DI
- new net N$19: LED16.DO, LED17.DI
- new net N$20: LED15.DO, LED16.DI
- new net N$21: LED14.DO, LED15.DI
- new net N$22: LED19.DO, LED20.DI
- new net N$23: LED20.DO, LED21.DI
- new net N$24: LED21.DO, LED22.DI
- new net N$25: LED22.DO, LED23.DI
- new net N$26: R_DISB2.1, SW3G$1.A
- new net N$27: R_DISA2.1, SW3G$1.B
- new net N$28: LED26.DO, LED27.DI
- new net N$29: LED25.DO, LED26.DI
- new net N$3: U$2.A1
- new net N$30: LED24.DO, LED25.DI
- new net N$31: LED23.DO, LED24.DI
- new net N$32: LED28.DO, LED29.DI
- new net N$33: LED29.DO, LED30.DI
- new net N$34: LED30.DO, LED31.DI
- new net N$35: LED31.DO, LED32.DI
- new net N$36: R_DISB3.1, SW4G$1.A
- new net N$37: R_DISA3.1, SW4G$1.B
- new net N$38: LED35.DO, LED36.DI
- new net N$39: LED34.DO, LED35.DI
- new net N$40: LED33.DO, LED34.DI
- new net N$41: LED32.DO, LED33.DI
- new net N$42: LED37.DO, LED38.DI
- new net N$43: LED38.DO, LED39.DI
- new net N$44: LED39.DO, LED40.DI
- new net N$45: LED40.DO, LED41.DI
- new net N$46: R_DISB4.1, SW5G$1.A
- new net N$47: R_DISA4.1, SW5G$1.B
- new net N$48: LED44.DO, LED45.DI
- new net N$49: LED43.DO, LED44.DI
- new net N$50: LED42.DO, LED43.DI
- new net N$51: LED41.DO, LED42.DI
- new net N$6: LED10.DO, LED11.DI
- new net N$62: LED55.DO, LED56.DI
- new net N$63: LED56.DO, LED57.DI
- new net N$64: LED57.DO, LED58.DI
- new net N$65: LED58.DO, LED59.DI
- new net N$66: R_DISB6.1, SW7G$1.A
- new net N$67: R_DISA6.1, SW7G$1.B
- new net N$68: LED62.DO, LED63.DI
- new net N$69: LED61.DO, LED62.DI
- new net N$70: LED60.DO, LED61.DI
- new net N$71: LED59.DO, LED60.DI
- new net N$82: LED73.DO, LED74.DI
- new net N$83: LED74.DO, LED75.DI
- new net N$84: LED75.DO, LED76.DI
- new net N$85: LED76.DO, LED77.DI
- new net N$86: R_DISB8.1, SW9G$1.A
- new net N$87: R_DISA8.1, SW9G$1.B
- new net N$88: LED80.DO, LED81.DI
- new net N$89: LED79.DO, LED80.DI
- new net N$90: LED78.DO, LED79.DI
- new net N$91: LED77.DO, LED78.DI
- new net NEOPIXEL_IN: LED10.DI, U$2.D6
- new net PIXEL_1: LED18.DO, LED19.DI
- new net PIXEL_2: LED27.DO, LED28.DI
- new net PIXEL_3: LED36.DO, LED37.DI
- new net PIXEL_4: LED45.DO, LED55.DI
- new net PIXEL_5: LED63.DO, LED73.DI
- new net PIXEL_OUT: LED81.DO
- new net ROT1_1: CA1.1, IC1.GPA0, R_DISA1.2, R_PDA1.1
- new net ROT1_2: CA2.1, IC1.GPB0, R_DISA2.2, R_PDA2.1
- new net ROT1_3: CA3.1, R_DISA3.2, R_PDA3.1
- new net ROT1_4: CA4.1, R_DISA4.2, R_PDA4.1
- new net ROT1_5: CA6.1, R_DISA6.2, R_PDA6.1
- new net ROT1_6: CA8.1, R_DISA8.2, R_PDA8.1
- new net ROT2_1: CB1.1, IC1.GPA1, R_DISB1.2, R_PUB1.1
- new net ROT2_2: CB2.1, IC1.GPB1, R_DISB2.2, R_PUB2.1
- new net ROT2_3: CB3.1, R_DISB3.2, R_PUB3.1
- new net ROT2_4: CB4.1, R_DISB4.2, R_PUB4.1
- new net ROT2_5: CB6.1, R_DISB6.2, R_PUB6.1
- new net ROT2_6: CB8.1, R_DISB8.2, R_PUB8.1
- new net ROT3_1: IC1.GPA2
- new net ROT3_2: IC1.GPB2
- new net ROT4_1: IC1.GPA3
- new net ROT4_2: IC1.GPB3
- new net ROT5_1: IC1.GPA4
- new net ROT5_2: IC1.GPB4
- new net ROT6_1: IC1.GPA5
- new net ROT6_2: IC1.GPB5
- net GND: now also CA1.2, CA2.2, CA3.2, CA4.2, CA6.2, CA8.2, CB1.2, CB2.2, CB3.2, CB4.2, CB6.2, CB8.2, CC1.1, CC2.1, CC3.1, CC4.1, CC6.1, CC8.1, LED10.GND, LED11.GND, LED12.GND, LED13.GND, LED14.GND, LED15.GND, LED16.GND, LED17.GND, LED18.GND, LED19.GND, LED20.GND, LED21.GND, LED22.GND, LED23.GND, LED24.GND, LED25.GND, LED26.GND, LED27.GND, LED28.GND, LED29.GND, LED30.GND, LED31.GND, LED32.GND, LED33.GND, LED34.GND, LED35.GND, LED36.GND, LED37.GND, LED38.GND, LED39.GND, LED40.GND, LED41.GND, LED42.GND, LED43.GND, LED44.GND, LED45.GND, LED55.GND, LED56.GND, LED57.GND, LED58.GND, LED59.GND, LED60.GND, LED61.GND, LED62.GND, LED63.GND, LED73.GND, LED74.GND, LED75.GND, LED76.GND, LED77.GND, LED78.GND, LED79.GND, LED80.GND, LED81.GND, SW2G$1.C, SW3G$1.C, SW4G$1.C, SW5G$1.C, SW5G$2.1, SW7G$1.C, SW7G$2.1, SW9G$1.C, SW9G$2.1, TP4.TP; no longer C1_E1.2, C1_E2.2, C1_E3.2, C1_E4.2, C1_E5.2, C1_E6.2, C1_E7.2, C1_E8.2, C2_E1.2, C2_E2.2, C2_E3.2, C2_E4.2, RDIS1.2, RDIS2.2, RDIS3.2, RDIS4.2, SW1G$2.1
- net I2C_CLK: now also TP1.TP
- net I2C_DATA: now also TP2.TP
- net VCC: now also LED10.VDD, LED11.VDD, LED12.VDD, LED13.VDD, LED14.VDD, LED15.VDD, LED16.VDD, LED17.VDD, LED18.VDD, LED19.VDD, LED20.VDD, LED21.VDD, LED22.VDD, LED23.VDD, LED24.VDD, LED25.VDD, LED26.VDD, LED27.VDD, LED28.VDD, LED29.VDD, LED30.VDD, LED31.VDD, LED32.VDD, LED33.VDD, LED34.VDD, LED35.VDD, LED36.VDD, LED37.VDD, LED38.VDD, LED39.VDD, LED40.VDD, LED41.VDD, LED42.VDD, LED43.VDD, LED44.VDD, LED45.VDD, LED55.VDD, LED56.VDD, LED57.VDD, LED58.VDD, LED59.VDD, LED60.VDD, LED61.VDD, LED62.VDD, LED63.VDD, LED73.VDD, LED74.VDD, LED75.VDD, LED76.VDD, LED77.VDD, LED78.VDD, LED79.VDD, LED80.VDD, LED81.VDD, R_PDA1.2, R_PDA2.2, R_PDA3.2, R_PDA4.2, R_PDA6.2, R_PDA8.2, R_PUB1.2, R_PUB2.2, R_PUB3.2, R_PUB4.2, R_PUB6.2, R_PUB8.2, R_PUC1.2, R_PUC2.2, R_PUC3.2, R_PUC4.2, R_PUC6.2, R_PUC8.2, TP3.TP; no longer NEOPIXEL1.P$5V, R1_E1.1, R1_E2.1, R1_E3.1, R1_E4.1, R1_E5.1, R1_E6.1, R1_E7.1, R1_E8.1, R2_E1.1, R2_E2.1, R2_E3.1, R2_E4.1
Other:
- note removed: "ENCODEUR 1"
- moved on the sheet: SW2, SW3, SW4
