File: eagle-schematics/themis-v1/DAC STM32 Board/DAC STM32 Board v4.1 - AD5391.sch (EAGLE design)
At the start: 36 parts, among them IC1 MCP23017SO, U1 ANALOG_DEVICES_AD5391BSTZ-3AN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

Commit message: Added new schematic for HP-LP-BP filter
Parts:
- added D1: (no value), SparkFun-LED:LED-3MM-NO_SILK
- added R_LED: 330, 6P1_EVB:R-US_0204/7
- added R_SCL_PU, R_SDA_PU: 1k, 6P1_EVB:R-US_0207/10
- added TP_DAC_BUSY, TP_DAC_SDO: PAD-TESTPOINT, ee2parts:PAD-TESTPOINT
Connections:
- removed net DAC_BUSY: A1B.PA4, U1A.!BUSY!
- new net LED: A1A.PB1, R_LED.2
- new net N$1: TP_DAC_BUSY.P, U1A.!BUSY!
- new net N$4: D1.A, R_LED.1
- net 3V3: now also R_SCL_PU.2, R_SDA_PU.2, R_SW1A.1, R_SW2A.1
- net 5V: no longer R_SW1A.1, R_SW2A.1
- net GND: now also D1.C
- net SCL: now also R_SCL_PU.1
- net SDA: now also R_SDA_PU.1
- net SPI_MISO: now also TP_DAC_SDO.P; no longer A1B.PA6
