File: front-pane/eagle-schematics/v3/STM32F446 front pane - v3.brd (EAGLE design)
At the start: 218.4 x 232.2 mm, 11 parts

Commit message: Updated front pane
Parts:
- removed C1, C2, C3: 10n, stock-perso:0805-CAP
- removed PIXEL0: NEOPIXEL-TLC59731DR, stock-perso:SOIC127P600X175-8N
- added 0V/5V: (no value), stock-perso:MA04-1
- added 3V3, GREEN: (no value), Passives:0805-LED
- added 5V: (no value), Passives:0603-LED
- added C10, C11, C12, C16, C17, C18, C22, C23, C24, C28, C29, C30, C34, C35, C36, C4, C40, C41, C42, C46, C47, C48, C5, C6, C7, C8, C9, CB1, CB10, CB100, CB104, CB105, CB106, CB11, CB110, CB111, CB112, CB116, CB117, CB118, CB12, CB13, CB14, CB15, CB16, CB17, CB18, CB19, CB2, CB20, CB21, CB22, CB23, CB24, CB25, CB26, CB27, CB28, CB29, CB3, CB30, CB31, CB32, CB33, CB34, CB35, CB36, CB37, CB38, CB39, CB4, CB40, CB41, CB42, CB43, CB44, CB45, CB47, CB48, CB49, CB5, CB50, CB51, CB52, CB53, CB54, CB55, CB56, CB57, CB58, CB59, CB6, CB60, CB61, CB62, CB63, CB64, CB65, CB66, CB67, CB68, CB70, CB71, CB72, CB73, CB74, CB75, CB76, CB77, CB78, CB79, CB8, CB80, CB81, CB82, CB83, CB84, CB85, CB89, CB9, CB90, CB91, CB92, CB93, CB94, CB98, CB99: 10n, stock-perso:0805-CAP
- added C55, C66, C67, C68, C69, C70: 0.1uF, MyComponents:C0805
- added C60: 2.2uF, MyComponents:C0805
- added C62: 10u, MyComponents:CPOL2917
- added C65: 100 uF, MyComponents:CPOL2917
- added C71: 1.0uF, MyComponents:C0805
- added C76: 1u, rcl:C1206
- added CDEC1, CDEC10, CDEC11, CDEC12, CDEC14, CDEC15, CDEC16, CDEC17, CDEC18, CDEC19, CDEC2, CDEC20, CDEC22, CDEC23, CDEC24, CDEC25, CDEC26, CDEC28, CDEC29, CDEC3, CDEC31, CDEC33, CDEC35, CDEC37, CDEC4, CDEC5, CDEC6, CDEC7, CDEC8, CDEC9, CDEC_11A, CDEC_12A, CDEC_2A1, CDEC_2A2, CDEC_2A3, CPOL13, CPOL21, CPOL30, CPOL32, CPOL36, CPOL39: 10u, stock-perso:CPOL2917
- added CDEC13, CDEC21, CDEC30, CDEC32, CDEC36, CDEC39, CDEC_11B, CDEC_12B, CDEC_2B1, CDEC_2B2, CDEC_2B3, CPOL1, CPOL10, CPOL11, CPOL12, CPOL14, CPOL15, CPOL16, CPOL17, CPOL18, CPOL19, CPOL2, CPOL20, CPOL22, CPOL23, CPOL24, CPOL25, CPOL26, CPOL28, CPOL29, CPOL3, CPOL31, CPOL33, CPOL35, CPOL37, CPOL4, CPOL5, CPOL6, CPOL7, CPOL8, CPOL9: 100n, stock-perso:0805-CAP
- added CDEC_1, CDEC_10, CDEC_11, CDEC_12, CDEC_13, CDEC_2, CDEC_3, CDEC_4, CDEC_5, CDEC_6, CDEC_7, CDEC_8, CDEC_9: 100n, stock-perso:1206
- added ENC_01, ENC_02, ENC_11, ENC_13, ENC_14, ENC_21, ENC_23, ENC_3, ENC_41, ENC_44, ENC_45, ENC_48, ENC_51, ENC_53, ENC_54, ENC_55, ENC_56, ENC_57, ENC_61, ENC_62, ENC_63, ENC_64, ENC_71, ENC_72, ENC_73, ENC_74, ENC_75, ENC_81, ENC_82, ENC_83, ENC_84, ENC_85, ENC_86, ENC_87, ENC_88, S24, S31, S34, S35: (no value), stock-perso:ENCODER_LED_3
- added F446: STM32F446RCT7, STM32F446RCT7:QFP50P1200X1200X160-64N
- added I2C1, MIDI: (no value), con-lstb:MA03-1
- added L1: 1 uH, MyComponents:L0805
- added LED1, LED2, LED22, LED4, LED6, LED7, LED_42, LED_43, LED_46, LED_47: CZXR-80RGB03-A, OPL_Optoelectronics:LED4-2.0-D8.0MM
- added MCP_11, MCP_12, MCP_2, MCP_31, MCP_32: MCP23017, a_ranger_work:SOIC-28
- added PIXEL_01, PIXEL_02, PIXEL_03, PIXEL_11, PIXEL_12, PIXEL_13, PIXEL_14, PIXEL_21, PIXEL_22, PIXEL_23, PIXEL_24, PIXEL_31, PIXEL_32, PIXEL_33, PIXEL_34, PIXEL_35, PIXEL_41, PIXEL_42, PIXEL_43, PIXEL_44, PIXEL_45, PIXEL_46, PIXEL_47, PIXEL_48, PIXEL_51, PIXEL_52, PIXEL_53, PIXEL_54, PIXEL_55, PIXEL_56, PIXEL_57, PIXEL_61, PIXEL_62, PIXEL_63, PIXEL_64, PIXEL_65, PIXEL_71, PIXEL_72, PIXEL_73, PIXEL_74, PIXEL_75, PIXEL_81, PIXEL_83, PIXEL_84, PIXEL_85, PIXEL_86, PIXEL_87, PIXEL_88, PIXE_82: NEOPIXEL-TLC59731DR, stock-perso:SOIC127P600X175-8N
- added R10, R100, R101, R102, R103, R104, R109, R11, R110, R111, R112, R113, R114, R115, R116, R117, R118, R12, R123, R124, R125, R126, R127, R128, R129, R130, R131, R132, R133, R134, R135, R136, R137, R138, R139, R140, R141, R142, R143, R144, R145, R146, R147, R148, R150, R151, R152, R153, R154, R155, R156, R157, R158, R159, R160, R161, R162, R163, R164, R167, R168, R169, R17, R170, R171, R172, R173, R174, R175, R176, R177, R178, R179, R18, R180, R181, R183, R184, R185, R188, R189, R19, R190, R191, R192, R193, R195, R196, R197, R200, R201, R202, R24, R25, R26, R31, R32, R33, R34, R35, R36, R37, R38, R39, R40, R45, R46, R47, R48, R49, R50, R51, R52, R53, R54, R59, R60, R61, R62, R63, R64, R65, R66, R67, R68, R73, R74, R75, R76, R77, R78, R80, R82, R83, R84, R85, R86, R94, R96, R97, R98, R99: 100, stock-perso:1206
- added R105, R119, R13, R20, R27, R41, R55, R69, R88, RPD1, RPD10, RPD11, RPD12, RPD14, RPD15, RPD16, RPD17, RPD18, RPD19, RPD2, RPD20, RPD22, RPD23, RPD24, RPD25, RPD26, RPD28, RPD29, RPD3, RPD31, RPD33, RPD35, RPD37, RPD4, RPD5, RPD6, RPD7, RPD8, RPD9: 10k, stock-perso:1206
- added R106, R107, R108, R120, R121, R122, R14, R15, R16, R21, R22, R23, R28, R29, R30, R42, R43, R44, R56, R57, R58, R70, R71, R72, R89, R91, R93, RB1, RB10, RB100, RB104, RB105, RB106, RB11, RB110, RB111, RB112, RB116, RB117, RB118, RB12, RB13, RB14, RB15, RB16, RB17, RB18, RB19, RB2, RB20, RB21, RB22, RB23, RB24, RB25, RB26, RB27, RB28, RB29, RB3, RB30, RB31, RB32, RB33, RB34, RB35, RB36, RB37, RB38, RB39, RB4, RB40, RB41, RB42, RB43, RB44, RB45, RB47, RB48, RB49, RB5, RB50, RB51, RB52, RB53, RB54, RB55, RB56, RB57, RB58, RB59, RB6, RB60, RB61, RB62, RB63, RB64, RB65, RB66, RB67, RB68, RB70, RB71, RB72, RB73, RB74, RB75, RB76, RB77, RB78, RB79, RB8, RB80, RB81, RB82, RB83, RB84, RB85, RB89, RB9, RB90, RB91, RB92, RB93, RB94, RB98, RB99: 470, stock-perso:1206
- added R149, R165, R166, R182, R186, R187, R4, R5: 1k, 6P1_EVB:R0805
- added R79: 100k, MyComponents:R0805
- added R81: 10K, MyComponents:R0805
- added R87: 1, MyComponents:R0805
- added R90, R95: 1k, MyComponents:R0805
- added R92: 470, MyComponents:R0805
- added S2: SWITCH-SKRKAEE020, stock-perso:SKRKAEE020
- added S3: JOYSTICK_THUMB, stock-perso:JOYSTICK
- added S32, S33, SW_42, SW_43, SW_46, SW_47, SW_52, SW_65, S_12, S_22: B3F-1000, Switch:B3F-1000
- added STLINK: 75867-331LF, MyComponents:MA03-2
- added TLV75533: TLV75533PDBVR, TLV75533PDBVR:SOT95P280X145-5N
- R1, R2: value 100 -> 1k; device stock-perso:1206 -> 6P1_EVB:R0805
- R6: value 10k -> 100
- R7, R8, R9: value 470 -> 100
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Connections:
- removed net GPA0_0: R7.1
- removed net GPA1_0: R8.1
- removed net GPA2_0: R6.1, R9.1
- removed net N$1: R1.2
- removed net N$10: C1.2, R7.2
- removed net N$11: C2.2, R8.2
- removed net N$2: R2.2
- removed net N$3: R3.2
- removed net N$4: PIXEL0.1, R1.1
- removed net N$5: PIXEL0.2, R2.1
- removed net N$6: PIXEL0.3, R3.1
- removed net N$8: C3.1, R9.2
- removed net SDO_PIXEL0: PIXEL0.5
- new net 5V: 0V/5V.3, 0V/5V.4, C62.+, C76.2, R92.1, TLV75533.1, TLV75533.3
- new net ADC1_IN1: F446.15
- new net ADC1_IN10: F446.8
- new net ADC1_IN4: F446.20
- new net BOOT1: F446.60, R81.1
- new net DATA_PIXEL11: PIXEL_11.5, PIXEL_21.6
- new net DATA_PIXEL12: PIXEL_11.6, PIXEL_12.5
- new net DATA_PIXEL13: PIXEL_12.6, PIXEL_13.5
- new net DATA_PIXEL14: PIXEL_13.6, PIXEL_14.5
- new net DATA_PIXEL21: PIXEL_21.5, PIXEL_22.6
- new net DATA_PIXEL22: PIXEL_22.5, PIXEL_23.6
- new net DATA_PIXEL23: PIXEL_23.5, PIXEL_24.6
- new net DATA_PIXEL24: PIXEL_24.5, PIXEL_35.6
- new net DATA_PIXEL31: PIXEL_31.5
- new net DATA_PIXEL32: PIXEL_31.6, PIXEL_32.5
- new net DATA_PIXEL33: PIXEL_32.6, PIXEL_33.5
- new net DATA_PIXEL34: PIXEL_33.6, PIXEL_34.5
- new net DATA_PIXEL35: PIXEL_34.6, PIXEL_35.5
- new net GP: ENC_01.3, ENC_02.3, ENC_3.3, ENC_54.3, ENC_61.3, ENC_62.3, ENC_63.3, ENC_64.3, ENC_71.3, ENC_72.3, ENC_73.3, ENC_74.3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
- new net GPA: ENC_01.A, ENC_02.A, ENC_3.A, ENC_54.A, ENC_61.A, ENC_62.A, ENC_63.A, ENC_64.A, ENC_71.A, ENC_72.A, ENC_73.A, ENC_74.A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
- new net GPA0_11: MCP_11.21, R71.1, S24.B
- new net GPA0_12: MCP_12.21, R121.1, S35.B
- new net GPA0_2: MCP_2.21, RB70.1, SW_47.3, SW_47.4
- new net GPA0_31: ENC_51.A, MCP_31.21, RB8.1
- new net GPA0_32: MCP_32.21
- new net GPA1_11: MCP_11.22, R70.1, S24.A
- new net GPA1_12: MCP_12.22, R119.1, R122.1, S35.3
- new net GPA1_2: ENC_45.A, MCP_2.22, RB23.1
- new net GPA1_31: ENC_51.B, MCP_31.22, RB9.1
- new net GPA1_32: MCP_32.22
- new net GPA2_11: MCP_11.23, R69.1, R72.1, S24.3
- new net GPA2_12: MCP_12.23, R120.1, S35.A
- new net GPA2_2: ENC_45.B, MCP_2.23, RB24.1
- new net GPA2_31: ENC_51.3, MCP_31.23, RB10.1, RPD1.1
- new net GPA2_32: MCP_32.23
- new net GPA3_11: ENC_23.A, MCP_11.24, R56.1
- new net GPA3_12: MCP_12.24, R107.1, S34.B
- new net GPA3_2: ENC_45.3, MCP_2.24, RB25.1, RPD6.1
- new net GPA3_31: MCP_31.24, RB5.1, SW_52.3, SW_52.4
- new net GPA3_32: MCP_32.24
- new net GPA4_11: ENC_23.B, MCP_11.25, R57.1
- new net GPA4_12: MCP_12.25, R106.1, S34.A
- new net GPA4_2: MCP_2.25, RB68.1, SW_46.3, SW_46.4
- new net GPA4_31: ENC_53.3, MCP_31.25, RB16.1, RPD3.1
- new net GPA4_32: MCP_32.25
- new net GPA5_11: ENC_23.3, MCP_11.26, R55.1, R58.1
- new net GPA5_12: MCP_12.26, R105.1, R108.1, S34.3
- new net GPA5_2: ENC_48.A, MCP_2.26, RB29.1
- new net GPA5_31: ENC_53.A, MCP_31.26, RB14.1
- new net GPA5_32: MCP_32.26
- new net GPA6_11: ENC_11.3, MCP_11.27, R13.1, R16.1
- new net GPA6_12: MCP_12.27, RB6.1, S33.3, S33.4
- new net GPA6_2: ENC_48.3, MCP_2.27, RB31.1, RPD8.1
- new net GPA6_31: ENC_53.B, MCP_31.27, RB15.1
- new net GPA6_32: MCP_32.27
- new net GPA7_11: MCP_11.28, RB2.1, S_12.3, S_12.4
- new net GPA7_12: MCP_12.28, RB1.1, S32.3, S32.4
- new net GPA7_2: ENC_48.B, MCP_2.28, RB30.1
- new net GPA7_31: ENC_57.3, MCP_31.28, RB49.1, RPD14.1
- new net GPA7_32: MCP_32.28
- new net GPB: ENC_01.B, ENC_02.B, ENC_3.B, ENC_54.B, ENC_61.B, ENC_62.B, ENC_63.B, ENC_64.B, ENC_71.B, ENC_72.B, ENC_73.B, ENC_74.B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
- new net GPB0_11: ENC_11.A, MCP_11.1, R14.1
- new net GPB0_12: MCP_12.1
- new net GPB0_2: MCP_2.1, RB3.1, SW_42.3, SW_42.4
- new net GPB0_31: ENC_57.B, MCP_31.1, RB48.1
- new net GPB0_32: MCP_32.1
- new net GPB1_11: ENC_11.B, MCP_11.2, R15.1
- new net GPB1_12: MCP_12.2, R91.1, S31.B
- new net GPB1_2: ENC_44.A, MCP_2.2, RB17.1
- new net GPB1_31: ENC_57.A, MCP_31.2, RB47.1
- new net GPB1_32: MCP_32.2
- new net GPB2_11: ENC_13.A, MCP_11.3, R21.1
- new net GPB2_12: MCP_12.3, R88.1, R93.1, S31.3
- new net GPB2_2: ENC_44.B, MCP_2.3, RB18.1
- new net GPB2_31: ENC_56.3, MCP_31.3, RB43.1, RPD12.1
- new net GPB2_32: MCP_32.3
- new net GPB3_11: ENC_13.B, MCP_11.4, R22.1
- new net GPB3_12: MCP_12.4, R89.1, S31.A
- new net GPB3_2: ENC_44.3, MCP_2.4, RB19.1, RPD4.1
- new net GPB3_31: ENC_56.B, MCP_31.4, RB42.1
- new net GPB3_32: MCP_32.4
- new net GPB4_11: ENC_13.3, MCP_11.5, R20.1, R23.1
- new net GPB4_12: ENC_21.3, MCP_12.5, R41.1, R44.1
- new net GPB4_2: ENC_41.A, MCP_2.5, RB11.1
- new net GPB4_31: ENC_56.A, MCP_31.5, RB41.1
- new net GPB4_32: MCP_32.5
- new net GPB5_11: ENC_14.3, MCP_11.6, R27.1, R30.1
- new net GPB5_12: ENC_21.A, MCP_12.6, R42.1
- new net GPB5_2: ENC_41.B, MCP_2.6, RB12.1
- new net GPB5_31: ENC_55.A, MCP_31.6, RB35.1
- new net GPB5_32: MCP_32.6
- new net GPB6_11: ENC_14.A, MCP_11.7, R28.1
- new net GPB6_12: ENC_21.B, MCP_12.7, R43.1
- new net GPB6_2: ENC_41.3, MCP_2.7, RB13.1, RPD2.1
- new net GPB6_31: ENC_55.B, MCP_31.7, RB36.1
- new net GPB6_32: MCP_32.7
- new net GPB7_11: ENC_14.B, MCP_11.8, R29.1
- new net GPB7_12: MCP_12.8, RB4.1, S_22.3, S_22.4
- new net GPB7_2: MCP_2.8, RB45.1, SW_43.3, SW_43.4
- new net GPB7_31: ENC_55.3, MCP_31.8, RB37.1, RPD10.1
- new net GPB7_32: MCP_32.8
- new net GPIO_EXTI1: F446.27
- new net GPIO_EXTI10: F446.43
- new net GPIO_EXTI11: F446.44
- new net GPIO_EXTI12: F446.45
- new net GPIO_EXTI14: F446.35
- new net GPIO_EXTI15: F446.36
- new net GPIO_EXTI2: F446.10
- new net GPIO_EXTI3: F446.11
- new net GPIO_EXTI4: F446.24
- new net GPIO_EXTI5: F446.25
- new net GPIO_EXTI6: F446.37
- new net GPIO_EXTI7: F446.38
- new net GPIO_EXTI8: F446.39
- new net GPIO_EXTI9: F446.42
- new net I2C1_SCL: F446.61, I2C1.2, MCP_11.12, MCP_12.12, R186.1, R4.1
- new net I2C1_SDA: F446.62, I2C1.1, MCP_11.13, MCP_12.13, R187.1, R5.1
- new net I2C2_SCL: F446.29, MCP_2.12, MCP_31.12, MCP_32.12, R1.1, R149.1, R166.1
- new net I2C2_SDA: F446.53, MCP_2.13, MCP_31.13, MCP_32.13, R165.1, R182.1, R2.1
- new net I2C3_SCL: F446.41
- new net I2C3_SDA: F446.40
- new net INTA_11: MCP_11.20
- new net INTA_12: MCP_12.20
- new net INTA_2: MCP_2.20
- new net INTA_31: MCP_31.20
- new net INTA_32: MCP_32.20
- new net INTB_11: MCP_11.19
- new net INTB_12: MCP_12.19
- new net INTB_2: MCP_2.19
- new net INTB_31: MCP_31.19
- new net INTB_32: MCP_32.19
- new net N$10160: PIXEL_46.1, R188.1
- new net N$10161: PIXEL_46.2, R192.1
- new net N$10162: PIXEL_46.3, R193.1
- new net N$10163: CB68.2, RB68.2
- new net N$10164: LED_46.1, R193.2
- new net N$10165: LED_46.4, R192.2
- new net N$10166: LED_46.3, R188.2
- new net N$10174: ENC_02.1, R189.2
- new net N$10175: ENC_02.2, R190.2
- new net N$10176: ENC_02.4, R191.2
- new net N$10177: PIXEL_02.1, R189.1
- new net N$10178: PIXEL_02.2, R190.1
- new net N$10179: PIXEL_02.3, R191.1
- new net N$10180: CB110.2, RB110.2
- new net N$10181: CB111.2, RB111.2
- new net N$10182: CB112.1, RB112.2
- new net N$10540: ENC_3.1, R195.2
- new net N$10541: ENC_3.2, R196.2
- new net N$10542: ENC_3.4, R197.2
- new net N$10543: PIXEL_03.1, R195.1
- new net N$10544: PIXEL_03.2, R196.1
- new net N$10545: PIXEL_03.3, R197.1
- new net N$10546: CB116.2, RB116.2
- new net N$10547: CB117.2, RB117.2
- new net N$10548: CB118.1, RB118.2
- new net N$1069: ENC_13.1, R17.2
- new net N$1070: ENC_13.2, R18.2
- new net N$1071: ENC_13.4, R19.2
- new net N$1072: PIXEL_13.1, R17.1
- new net N$1073: PIXEL_13.2, R18.1
- new net N$1074: PIXEL_13.3, R19.1
- new net N$1075: C7.2, R21.2
- new net N$1076: C8.2, R22.2
- new net N$1077: C9.1, R23.2
- new net N$108: R87.2, TLV75533.5
- new net N$10888: PIXEL_47.1, R200.1
- new net N$10889: PIXEL_47.2, R201.1
- new net N$10890: PIXEL_47.3, R202.1
- new net N$10891: CB70.2, RB70.2
- new net N$10892: LED_47.1, R202.2
- new net N$10893: LED_47.4, R201.2
- new net N$10894: LED_47.3, R200.2
- new net N$109: L1.1, R87.1
- new net N$1252: ENC_14.1, R24.2
- new net N$1253: ENC_14.2, R25.2
- new net N$1254: ENC_14.4, R26.2
- new net N$1255: PIXEL_14.1, R24.1
- new net N$1256: PIXEL_14.2, R25.1
- new net N$1257: PIXEL_14.3, R26.1
- new net N$1258: C10.2, R28.2
- new net N$1259: C11.2, R29.2
- new net N$1260: C12.1, R30.2
- new net N$1435: PIXEL_32.3, R7.1
- new net N$1436: CB1.2, RB1.2
- new net N$1437: LED1.1, R7.2
- new net N$1438: LED1.4, R6.2
- new net N$1439: LED1.3, R3.2
- new net N$1614: PIXEL_12.1, R8.1
- new net N$1615: PIXEL_12.2, R9.1
- new net N$1616: PIXEL_12.3, R31.1
- new net N$1617: CB2.2, RB2.2
- new net N$1618: ENC_21.1, R38.2
- new net N$1619: ENC_21.2, R39.2
- new net N$1620: ENC_21.4, R40.2
- new net N$1621: PIXEL_21.1, R38.1
- new net N$1622: PIXEL_21.2, R39.1
- new net N$1623: PIXEL_21.3, R40.1
- new net N$1624: C16.2, R42.2
- new net N$1625: C17.2, R43.2
- new net N$1626: C18.1, R44.2
- new net N$1801: LED2.1, R31.2
- new net N$1802: LED2.4, R9.2
- new net N$1803: LED2.3, R8.2
- new net N$1978: PIXEL_42.2, R123.1
- new net N$1979: ENC_51.1, R33.2
- new net N$1980: ENC_51.2, R34.2
- new net N$1981: ENC_51.4, R45.2
- new net N$1982: PIXEL_51.1, R33.1
- new net N$1983: PIXEL_51.2, R34.1
- new net N$1984: ENC_23.1, R52.2
- new net N$1985: ENC_23.2, R53.2
- new net N$1986: ENC_23.4, R54.2
- new net N$1987: PIXEL_23.1, R52.1
- new net N$1988: PIXEL_23.2, R53.1
- new net N$1989: PIXEL_23.3, R54.1
- new net N$1990: C22.2, R56.2
- new net N$1991: C23.2, R57.2
- new net N$1992: C24.1, R58.2
- new net N$2167: PIXEL_51.3, R45.1
- new net N$2168: CB8.2, RB8.2
- new net N$2169: CB9.2, RB9.2
- new net N$2170: CB10.1, RB10.2
- new net N$2342: PIXEL_22.1, R35.1
- new net N$2343: PIXEL_22.2, R36.1
- new net N$2344: PIXEL_22.3, R37.1
- new net N$2345: CB4.2, RB4.2
- new net N$2346: LED22.1, R37.2
- new net N$2347: LED22.4, R36.2
- new net N$2348: LED22.3, R35.2
- new net N$2350: R66.2, S24.1
- new net N$2351: R67.2, S24.2
- new net N$2352: R68.2, S24.4
- new net N$2353: PIXEL_24.1, R66.1
- new net N$2354: PIXEL_24.2, R67.1
- new net N$2355: PIXEL_24.3, R68.1
- new net N$2356: C28.2, R70.2
- new net N$2357: C29.2, R71.2
- new net N$2358: C30.1, R72.2
- new net N$2709: ENC_41.1, R46.2
- new net N$2710: ENC_41.2, R47.2
- new net N$2711: ENC_41.4, R51.2
- new net N$2712: PIXEL_41.1, R46.1
- new net N$2713: PIXEL_41.2, R47.1
- new net N$2714: PIXEL_41.3, R51.1
- new net N$2715: CB11.2, RB11.2
- new net N$2716: R82.2, S31.1
- new net N$2717: R84.2, S31.2
- new net N$2718: R85.2, S31.4
- new net N$2719: PIXEL_31.1, R82.1
- new net N$2720: PIXEL_31.2, R84.1
- new net N$2721: PIXEL_31.3, R85.1
- new net N$2722: C34.2, R89.2
- new net N$2723: C35.2, R91.2
- new net N$2724: C36.1, R93.2
- new net N$2899: CB12.2, RB12.2
- new net N$2900: CB13.1, RB13.2
- new net N$3070: PIXEL_33.1, R48.1
- new net N$3071: PIXEL_33.2, R49.1
- new net N$3072: PIXEL_33.3, R50.1
- new net N$3073: CB6.2, RB6.2
- new net N$3074: LED6.1, R50.2
- new net N$3075: LED6.4, R49.2
- new net N$3076: LED6.3, R48.2
- new net N$3082: R102.2, S34.1
- new net N$3083: R103.2, S34.2
- new net N$3084: R104.2, S34.4
- new net N$3085: PIXEL_34.1, R102.1
- new net N$3086: PIXEL_34.2, R103.1
- new net N$3087: PIXEL_34.3, R104.1
- new net N$3088: C40.2, R106.2
- new net N$3089: C41.2, R107.2
- new net N$3090: C42.1, R108.2
- new net N$3439: ENC_53.1, R59.2
- new net N$3440: ENC_53.2, R60.2
- new net N$3441: ENC_53.4, R61.2
- new net N$3442: PIXEL_53.1, R59.1
- new net N$3443: PIXEL_53.2, R60.1
- new net N$3444: PIXEL_53.3, R61.1
- new net N$3445: CB14.2, RB14.2
- new net N$3446: CB15.2, RB15.2
- new net N$3447: CB16.1, RB16.2
- new net N$3448: R116.2, S35.1
- new net N$3449: R117.2, S35.2
- new net N$3450: R118.2, S35.4
- new net N$3451: PIXEL_35.1, R116.1
- new net N$3452: PIXEL_35.2, R117.1
- new net N$3453: PIXEL_35.3, R118.1
- new net N$3454: C46.2, R120.2
- new net N$3455: C47.2, R121.2
- new net N$3456: C48.1, R122.2
- new net N$3814: ENC_44.1, R62.2
- new net N$3815: ENC_44.2, R63.2
- new net N$3816: ENC_44.4, R64.2
- new net N$3817: PIXEL_44.1, R62.1
- new net N$3818: PIXEL_44.2, R63.1
- new net N$3819: PIXEL_44.3, R64.1
- new net N$3820: CB17.2, RB17.2
- new net N$3821: CB18.2, RB18.2
- new net N$3822: CB19.1, RB19.2
- new net N$4510: ENC_82.1, R65.2
- new net N$4511: ENC_82.2, R73.2
- new net N$4512: ENC_82.4, R74.2
- new net N$4513: PIXE_82.1, R65.1
- new net N$4514: PIXE_82.2, R73.1
- new net N$4515: PIXE_82.3, R74.1
- new net N$4516: CB20.2, RB20.2
- new net N$4517: CB21.2, RB21.2
- new net N$4518: CB22.1, RB22.2
- new net N$4867: ENC_45.1, R75.2
- new net N$4868: ENC_45.2, R76.2
- new net N$4869: ENC_45.4, R77.2
- new net N$4870: PIXEL_45.1, R75.1
- new net N$4871: PIXEL_45.2, R76.1
- new net N$4872: PIXEL_45.3, R77.1
- new net N$4873: CB23.2, RB23.2
- new net N$4874: CB24.2, RB24.2
- new net N$4875: CB25.1, RB25.2
- new net N$5050: ENC_54.1, R78.2
- new net N$5051: ENC_54.2, R80.2
- new net N$5052: ENC_54.4, R83.2
- new net N$5053: PIXEL_54.1, R78.1
- new net N$5054: PIXEL_54.2, R80.1
- new net N$5055: PIXEL_54.3, R83.1
- new net N$5056: CB26.2, RB26.2
- new net N$5057: CB27.2, RB27.2
- new net N$5058: CB28.1, RB28.2
- new net N$5233: ENC_48.1, R86.2
- new net N$5234: ENC_48.2, R94.2
- new net N$5235: ENC_48.4, R96.2
- new net N$5236: PIXEL_48.1, R86.1
- new net N$5237: PIXEL_48.2, R94.1
- new net N$5238: PIXEL_48.3, R96.1
- new net N$5239: CB29.2, RB29.2
- new net N$5240: CB30.2, RB30.2
- new net N$5241: CB31.1, RB31.2
- new net N$53: 5V.A, R92.2
- new net N$5416: ENC_71.1, R97.2
- new net N$5417: ENC_71.2, R98.2
- new net N$5418: ENC_71.4, R99.2
- new net N$5419: PIXEL_71.1, R97.1
- new net N$5420: PIXEL_71.2, R98.1
- new net N$5421: PIXEL_71.3, R99.1
- new net N$5422: CB32.2, RB32.2
- new net N$5423: CB33.2, RB33.2
- new net N$5424: CB34.1, RB34.2
- new net N$5599: ENC_55.1, R100.2
- new net N$56: GREEN.A, R90.2
- new net N$5600: ENC_55.2, R101.2
- new net N$5601: ENC_55.4, R109.2
- new net N$5602: PIXEL_55.1, R100.1
- new net N$5603: PIXEL_55.2, R101.1
- new net N$5604: PIXEL_55.3, R109.1
- new net N$5605: CB35.2, RB35.2
- new net N$5606: CB36.2, RB36.2
- new net N$5607: CB37.1, RB37.2
- new net N$57: 3V3.A, R95.2
- new net N$5782: ENC_83.1, R110.2
- new net N$5783: ENC_83.2, R111.2
- new net N$5784: ENC_83.4, R112.2
- new net N$5785: PIXEL_83.1, R110.1
- new net N$5786: PIXEL_83.2, R111.1
- new net N$5787: PIXEL_83.3, R112.1
- new net N$5788: CB38.2, RB38.2
- new net N$5789: CB39.2, RB39.2
- new net N$5790: CB40.1, RB40.2
- new net N$5965: ENC_56.1, R113.2
- new net N$5966: ENC_56.2, R114.2
- new net N$5967: ENC_56.4, R115.2
- new net N$5968: PIXEL_56.1, R113.1
- new net N$5969: PIXEL_56.2, R114.1
- new net N$5970: PIXEL_56.3, R115.1
- new net N$5971: CB41.2, RB41.2
- new net N$5972: CB42.2, RB42.2
- new net N$5973: CB43.1, RB43.2
- new net N$6148: PIXEL_42.3, R124.1
- new net N$6149: CB3.2, RB3.2
- new net N$6150: LED_42.1, R124.2
- new net N$6151: LED_42.4, R123.2
- new net N$6152: LED_42.3, R32.2
- new net N$6327: PIXEL_52.1, R125.1
- new net N$6328: PIXEL_52.2, R147.1
- new net N$6329: PIXEL_52.3, R148.1
- new net N$6330: CB5.2, RB5.2
- new net N$6331: ENC_57.1, R126.2
- new net N$6332: ENC_57.2, R127.2
- new net N$6333: ENC_57.4, R128.2
- new net N$6334: PIXEL_57.1, R126.1
- new net N$6335: PIXEL_57.2, R127.1
- new net N$6336: PIXEL_57.3, R128.1
- new net N$6337: CB47.2, RB47.2
- new net N$6338: CB48.2, RB48.2
- new net N$6339: CB49.1, RB49.2
- new net N$6514: ENC_84.1, R129.2
- new net N$6515: ENC_84.2, R130.2
- new net N$6516: ENC_84.4, R131.2
- new net N$6517: PIXEL_84.1, R129.1
- new net N$6518: PIXEL_84.2, R130.1
- new net N$6519: PIXEL_84.3, R131.1
- new net N$6520: CB50.2, RB50.2
- new net N$6521: CB51.2, RB51.2
- new net N$6522: CB52.1, RB52.2
- new net N$6697: ENC_61.1, R132.2
- new net N$6698: ENC_61.2, R133.2
- new net N$6699: ENC_61.4, R134.2
- new net N$6700: PIXEL_61.1, R132.1
- new net N$6701: PIXEL_61.2, R133.1
- new net N$6702: PIXEL_61.3, R134.1
- new net N$6703: CB53.2, RB53.2
- new net N$6704: CB54.2, RB54.2
- new net N$6705: CB55.1, RB55.2
- new net N$6880: ENC_72.1, R135.2
- new net N$6881: ENC_72.2, R136.2
- new net N$6882: ENC_72.4, R137.2
- new net N$6883: PIXEL_72.1, R135.1
- new net N$6884: PIXEL_72.2, R136.1
- new net N$6885: PIXEL_72.3, R137.1
- new net N$6886: CB56.2, RB56.2
- new net N$6887: CB57.2, RB57.2
- new net N$6888: CB58.1, RB58.2
- new net N$7063: ENC_62.1, R138.2
- new net N$7064: ENC_62.2, R139.2
- new net N$7065: ENC_62.4, R140.2
- new net N$7066: PIXEL_62.1, R138.1
- new net N$7067: PIXEL_62.2, R139.1
- new net N$7068: PIXEL_62.3, R140.1
- new net N$7069: CB59.2, RB59.2
- new net N$7070: CB60.2, RB60.2
- new net N$7071: CB61.1, RB61.2
- new net N$709: PIXEL_42.1, R32.1
- new net N$710: PIXEL_32.1, R3.1
- new net N$711: PIXEL_32.2, R6.1
- new net N$712: ENC_11.1, R10.2
- new net N$713: ENC_11.2, R11.2
- new net N$714: ENC_11.4, R12.2
- new net N$715: PIXEL_11.1, R10.1
- new net N$716: PIXEL_11.2, R11.1
- new net N$717: PIXEL_11.3, R12.1
- new net N$718: C4.2, R14.2
- new net N$719: C5.2, R15.2
- new net N$720: C6.1, R16.2
- new net N$7246: ENC_85.1, R141.2
- new net N$7247: ENC_85.2, R142.2
- new net N$7248: ENC_85.4, R143.2
- new net N$7249: PIXEL_85.1, R141.1
- new net N$7250: PIXEL_85.2, R142.1
- new net N$7251: PIXEL_85.3, R143.1
- new net N$7252: CB62.2, RB62.2
- new net N$7253: CB63.2, RB63.2
- new net N$7254: CB64.1, RB64.2
- new net N$7429: ENC_63.1, R144.2
- new net N$7430: ENC_63.2, R145.2
- new net N$7431: ENC_63.4, R146.2
- new net N$7432: PIXEL_63.1, R144.1
- new net N$7433: PIXEL_63.2, R145.1
- new net N$7434: PIXEL_63.3, R146.1
- new net N$7435: CB65.2, RB65.2
- new net N$7436: CB66.2, RB66.2
- new net N$7437: CB67.1, RB67.2
- new net N$7612: LED4.1, R148.2
- new net N$7613: LED4.4, R147.2
- new net N$7614: LED4.3, R125.2
- new net N$7795: ENC_64.1, R150.2
- new net N$7796: ENC_64.2, R151.2
- new net N$7797: ENC_64.4, R152.2
- new net N$7798: PIXEL_64.1, R150.1
- new net N$7799: PIXEL_64.2, R151.1
- new net N$7800: PIXEL_64.3, R152.1
- new net N$7801: CB71.2, RB71.2
- new net N$7802: CB72.2, RB72.2
- new net N$7803: CB73.1, RB73.2
- new net N$7978: ENC_86.1, R153.2
- new net N$7979: ENC_86.2, R154.2
- new net N$7980: ENC_86.4, R155.2
- new net N$7981: PIXEL_86.1, R153.1
- new net N$7982: PIXEL_86.2, R154.1
- new net N$7983: PIXEL_86.3, R155.1
- new net N$7984: CB74.2, RB74.2
- new net N$7985: CB75.2, RB75.2
- new net N$7986: CB76.1, RB76.2
- new net N$8161: ENC_81.1, R156.2
- new net N$8162: ENC_81.2, R157.2
- new net N$8163: ENC_81.4, R158.2
- new net N$8164: PIXEL_81.1, R156.1
- new net N$8165: PIXEL_81.2, R157.1
- new net N$8166: PIXEL_81.3, R158.1
- new net N$8167: CB77.2, RB77.2
- new net N$8168: CB78.2, RB78.2
- new net N$8169: CB79.1, RB79.2
- new net N$8344: ENC_73.1, R159.2
- new net N$8345: ENC_73.2, R160.2
- new net N$8346: ENC_73.4, R161.2
- new net N$8347: PIXEL_73.1, R159.1
- new net N$8348: PIXEL_73.2, R160.1
- new net N$8349: PIXEL_73.3, R161.1
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Routing:
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Other:
- board size 218.4 x 232.2 mm -> 450 x 300 mm
- board text added: "2nd/4th"
- board text added: "AMP EG"
- board text added: "AMP/EG3"
- board text added: "ANALOG OSC 1"
- board text added: "ANALOG OSC 2"
- board text added: "Amount"
- board text added: "Amount/Dest"
- board text added: "Attack"
- board text added: "Back-Forth"
- board text added: "Chorus"
- board text added: "Cutoff/Reso"
- board text added: "DIG OSC"
- board text added: "Decay"
- board text added: "Delay"
- board text added: "Detune"
- board text added: "Drive"
- board text added: "EFFECTS"
- board text added: "EG Amount/Kbd Tracking"
- board text added: "FILTER"
- board text added: "FILTER EG"
- board text added: "Human"
- board text added: "Joystick"
- board text added: "LFO 1"
- board text added: "LFO 2"
- board text added: "Latch"
- board text added: "MIDI Sync"
- board text added: "ON/OFF"
- board text added: "Octave"
- board text added: "Output Jack"
- board text added: "PORTA"
- board text added: "PRESETS/ARP"
- board text added: "Param1"
- board text added: "Param2"
- board text added: "Param3"
- board text added: "Pattern"
- board text added: "RAINBOW by SYD X. REY & MARION MUCCIANTE (c) 2021"
- board text added: "Range"
- board text added: "Rate"
- board text added: "Rate/Wave"
- board text added: "Release"
- board text added: "Reverb"
- board text added: "Sustain"
- board text added: "Sync"
- board text added: "Time/ON-OFF"
- board text added: "Volume"
- board text added: "Wave"
- board text added: "Wave/PWM"
- board text added: "Wave/PWM/Sub"
- board text removed: "SYD.X.REY INSTR. 2020"

Commit message: Front pane update
Parts:
- removed I2C1, MIDI: (no value), con-lstb:MA03-1
- removed S3: JOYSTICK_THUMB, stock-perso:JOYSTICK
- added CDEC_41A, CDEC_42A, CDEC_5A: 10u, stock-perso:CPOL2917
- added CDEC_41B, CDEC_42B, CDEC_5B: 100n, stock-perso:0805-CAP
- added JOYSTICK: (no value), MyComponents:MA05-1
- added MCP_41, MCP_42, MCP_5: MCP23017, a_ranger_work:SOIC-28
- added R194, R198, R199, R203, R204, R205: 1k, 6P1_EVB:R0805
- added TFT_EXT, TFT_EXT_2: (no value), con-lstb:MA06-2
- moved 3V3 13.0 mm to (225.2, 224.3)
- moved C66 13.0 mm to (235.8, 207.5)
- moved C70 13.0 mm to (228.7, 221.9)
- moved C76 13.0 mm to (235.7, 235.7)
- moved STLINK 13.0 mm to (225.0, 208.6)
- moved 0V/5V 13.0 mm to (246.0, 231.8)
- moved 5V 13.0 mm to (249.0, 229.5)
- moved C55 13.0 mm to (237.0, 225.9)
- moved C62 13.0 mm to (236.9, 231.7)
- moved C65 13.0 mm to (226.0, 228.1)
- moved C69 13.0 mm to (247.4, 219.0)
- moved C71 13.0 mm to (234.1, 225.9)
- moved GREEN 13.0 mm to (247.9, 224.2)
- moved R79 13.0 mm to (240.7, 227.1)
- moved R95 13.0 mm to (225.2, 222.0)
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Connections:
- new net ENC_01_A: ENC_01.A, RB104.1, TFT_EXT_2.3
- new net ENC_01_B: ENC_01.B, RB105.1, TFT_EXT_2.5
- new net ENC_01_SW: ENC_01.3, RB106.1, RPD33.1, TFT_EXT_2.6
- new net ENC_02_A: ENC_02.A, RB110.1, TFT_EXT_2.11
- new net ENC_02_B: ENC_02.B, RB111.1, TFT_EXT_2.12
- new net ENC_02_SW: ENC_02.3, RB112.1, RPD35.1, TFT_EXT_2.4
- new net ENC_03_A: ENC_3.A, RB116.1, TFT_EXT_2.10
- new net ENC_03_B: ENC_3.B, RB117.1, TFT_EXT_2.8
- new net ENC_03_SW: ENC_3.3, RB118.1, RPD37.1, TFT_EXT_2.2
- new net GPA0_41: MCP_41.21
- new net GPA0_42: ENC_83.A, MCP_42.21, RB38.1
- new net GPA0_5: ENC_74.3, MCP_5.21, RB94.1, RPD29.1
- new net GPA1_41: MCP_41.22
- new net GPA1_42: ENC_83.B, MCP_42.22, RB39.1
- new net GPA1_5: ENC_74.B, MCP_5.22, RB93.1
- new net GPA2_41: MCP_41.23
- new net GPA2_42: ENC_84.A, MCP_42.23, RB50.1
- new net GPA2_5: ENC_74.A, MCP_5.23, RB92.1
- new net GPA3_41: MCP_41.24
- new net GPA3_42: ENC_84.B, MCP_42.24, RB51.1
- new net GPA3_5: ENC_73.3, MCP_5.24, RB82.1, RPD25.1
- new net GPA4_41: MCP_41.25
- new net GPA4_42: ENC_84.3, MCP_42.25, RB52.1, RPD15.1
- new net GPA4_5: ENC_86.A, MCP_5.25, RB74.1
- new net GPA5_41: MCP_41.26
- new net GPA5_42: ENC_85.A, MCP_42.26, RB62.1
- new net GPA5_5: ENC_86.B, MCP_5.26, RB75.1
- new net GPA6_41: MCP_41.27
- new net GPA6_42: ENC_85.B, MCP_42.27, RB63.1
- new net GPA6_5: ENC_86.3, MCP_5.27, RB76.1, RPD23.1
- new net GPA7_41: MCP_41.28
- new net GPA7_42: ENC_85.3, MCP_42.28, RB64.1, RPD19.1
- new net GPA7_5: ENC_87.3, MCP_5.28, RB85.1, RPD26.1
- new net GPB0_41: MCP_41.1
- new net GPB0_42: ENC_73.B, MCP_42.1, RB81.1
- new net GPB0_5: ENC_87.B, MCP_5.1, RB84.1
- new net GPB1_41: MCP_41.2
- new net GPB1_42: ENC_73.A, MCP_42.2, RB80.1
- new net GPB1_5: ENC_87.A, MCP_5.2, RB83.1
- new net GPB2_41: MCP_41.3
- new net GPB2_42: ENC_72.B, MCP_42.3, RB57.1
- new net GPB2_5: ENC_88.3, MCP_5.3, RB91.1, RPD28.1
- new net GPB3_41: MCP_41.4
- new net GPB3_42: ENC_72.A, MCP_42.4, RB56.1
- new net GPB3_5: ENC_88.A, MCP_5.4, RB89.1
- new net GPB4_41: MCP_41.5
- new net GPB4_42: ENC_72.3, MCP_42.5, RB58.1, RPD17.1
- new net GPB4_5: ENC_88.B, MCP_5.5, RB90.1
- new net GPB5_41: MCP_41.6
- new net GPB5_42: ENC_71.B, MCP_42.6, RB33.1
- new net GPB5_5: ENC_75.3, MCP_5.6, RB100.1, RPD31.1
- new net GPB6_41: MCP_41.7
- new net GPB6_42: ENC_71.A, MCP_42.7, RB32.1
- new net GPB6_5: ENC_75.A, MCP_5.7, RB98.1
- new net GPB7_41: MCP_41.8
- new net GPB7_42: ENC_71.3, MCP_42.8, RB34.1, RPD9.1
- new net GPB7_5: ENC_75.B, MCP_5.8, RB99.1
- new net INTA_41: MCP_41.20
- new net INTA_42: MCP_42.20
- new net INTA_5: MCP_5.20
- new net INTB_41: MCP_41.19
- new net INTB_42: MCP_42.19
- new net INTB_5: MCP_5.19
- new net JOY_SEL: JOYSTICK.2
- new net JOY_XOUT: JOYSTICK.4
- new net JOY_YOUT: JOYSTICK.3
- new net N$1: TFT_EXT.10, TFT_EXT.11, TFT_EXT.12, TFT_EXT.2, TFT_EXT.3, TFT_EXT.4, TFT_EXT.5, TFT_EXT.6, TFT_EXT.8
- new net PIXEL_IN: PIXEL_03.6, TFT_EXT_2.9
- net 3V3: now also CDEC_41A.+, CDEC_41B.1, CDEC_42A.+, CDEC_42B.1, CDEC_5A.+, CDEC_5B.1, JOYSTICK.5, MCP_31.15, MCP_32.17, MCP_41.15, MCP_41.17, MCP_41.9, MCP_42.16, MCP_42.17, MCP_42.9, MCP_5.16, MCP_5.17, MCP_5.9, R194.2, R198.2, R199.2, R203.2, R204.2, R205.2, TFT_EXT.1, TFT_EXT_2.1; no longer MCP_32.16
- net GND: now also CDEC_41A.-, CDEC_41B.2, CDEC_42A.-, CDEC_42B.2, CDEC_5A.-, CDEC_5B.2, JOYSTICK.1, MCP_32.16, MCP_41.10, MCP_41.16, MCP_42.10, MCP_42.15, MCP_5.10, MCP_5.15, TFT_EXT.7, TFT_EXT_2.7; no longer I2C1.3, MCP_31.15, MCP_32.17, MIDI.3
- net GP: no longer ENC_01.3, ENC_02.3, ENC_3.3, ENC_71.3, ENC_72.3, ENC_73.3, ENC_74.3, ENC_75.3, ENC_84.3, ENC_85.3, ENC_86.3, ENC_87.3, ENC_88.3, RB100.1, RB106.1, RB112.1, RB118.1, RB34.1, RB52.1, RB58.1, RB64.1, RB76.1, RB82.1, RB85.1, RB91.1, RB94.1, RPD15.1, RPD17.1, RPD19.1, RPD23.1, RPD25.1, RPD26.1, RPD28.1, RPD29.1, RPD31.1, RPD33.1, RPD35.1, RPD37.1, RPD9.1
- net GPA: no longer ENC_01.A, ENC_02.A, ENC_3.A, ENC_71.A, ENC_72.A, ENC_73.A, ENC_74.A, ENC_75.A, ENC_83.A, ENC_84.A, ENC_85.A, ENC_86.A, ENC_87.A, ENC_88.A, RB104.1, RB110.1, RB116.1, RB32.1, RB38.1, RB50.1, RB56.1, RB62.1, RB74.1, RB80.1, RB83.1, RB89.1, RB92.1, RB98.1
- net GPB: no longer ENC_01.B, ENC_02.B, ENC_3.B, ENC_71.B, ENC_72.B, ENC_73.B, ENC_74.B, ENC_75.B, ENC_83.B, ENC_84.B, ENC_85.B, ENC_86.B, ENC_87.B, ENC_88.B, RB105.1, RB111.1, RB117.1, RB33.1, RB39.1, RB51.1, RB57.1, RB63.1, RB75.1, RB81.1, RB84.1, RB90.1, RB93.1, RB99.1
- net I2C1_SCL: no longer I2C1.2
- net I2C1_SDA: no longer I2C1.1
- net I2C3_SCL: now also MCP_41.12, MCP_42.12, MCP_5.12, R194.1, R199.1, R204.1
- net I2C3_SDA: now also MCP_41.13, MCP_42.13, MCP_5.13, R198.1, R203.1, R205.1
- net PIXEL_81: now also TFT_EXT.9; no longer PIXEL_03.6
- net RST: now also MCP_41.18, MCP_42.18, MCP_5.18
- net USART1_RX: no longer MIDI.1
- net USART1_TX: no longer MIDI.2
Routing:
- net GND: track 4357.0 -> 4191.6 mm, vias 19 -> 18
- net I2C3_SDA: track 0.00 -> 132.6 mm, vias 0 -> 3
- net I2C3_SCL: track 0.00 -> 125.6 mm, vias 0 -> 3
- net GP: track 190.8 -> 72.7 mm
- net 3V3: track 3463.5 -> 3581.1 mm, vias 21 -> 27
- net ENC_01_SW: track 0.00 -> 101.7 mm
- net ENC_01_A: track 0.00 -> 89.7 mm
- net ENC_01_B: track 0.00 -> 86.6 mm
- net PIXEL_81: track 90.6 -> 12.1 mm, vias 2 -> 1
- net GPA7_42: track 0.00 -> 70.1 mm, vias 0 -> 1
- net GPA3_5: track 0.00 -> 67.4 mm
- net ENC_02_SW: track 0.00 -> 66.4 mm
- net GPA2_5: track 0.00 -> 65.5 mm, vias 0 -> 2
- net GPB2_5: track 0.00 -> 57.8 mm, vias 0 -> 1
- net GPB7_5: track 0.00 -> 57.7 mm, vias 0 -> 1
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Other:
- board text added: "AMPLITUDE ENVELOPE GENERATOR"
- board text added: "FILTER ENVELOPE GENERATOR"
- board text added: "MODULATION 1"
- board text added: "MODULATION 2"
- board text removed: "AMP EG"
- board text removed: "FILTER EG"
- board text removed: "Joystick"
- board text removed: "LFO 1"
- board text removed: "LFO 2"

Commit message: Finished front pane and sent to production
Parts:
- removed 3V3: (no value), Passives:0805-LED
- removed 5V: (no value), Passives:0603-LED
- removed JOYSTICK: (no value), MyComponents:MA05-1
- added ANALOG_IN: (no value), con-lstb:MA04-1
- added CONN_STH_BRD_1, CONN_STH_BRD_2: (no value), MyComponents:MA10-2
- added LED_3V3: (no value), Passives:0805-LED
- added LED_5V: (no value), Passives:0603-LED
- added UART_ANALOG, UART_DISCO, UART_MIDI: (no value), con-lstb:MA03-1
- moved C9 7.23 mm to (110.6, 161.7), turned to 90 degrees
- moved R148 6.69 mm to (307.7, 159.5), turned to 90 degrees
- moved R81 6.10 mm to (225.1, 220.5)
- moved C12 5.30 mm to (143.0, 161.3), turned to 90 degrees
- moved C66 5.22 mm to (234.2, 212.5)
- moved 0V/5V 5.03 mm to (245.1, 236.8)
- moved C55 5.03 mm to (236.1, 230.9)
- moved C62 5.03 mm to (236.1, 236.7)
- moved C65 5.03 mm to (225.1, 233.0)
- moved C69 5.03 mm to (246.6, 224.0)
- moved C70 5.03 mm to (227.8, 226.9)
- moved C71 5.03 mm to (233.2, 230.8)
- moved GREEN 5.03 mm to (247.0, 229.1)
- moved L1 5.03 mm to (229.6, 237.9)
- moved R79 5.03 mm to (239.8, 232.1)
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- renumbered MCP_11 to MCP_000, MCP_12 to MCP_001, MCP_2 to MCP_010, MCP_31 to MCP_011, MCP_32 to MCP_100, MCP_41 to MCP_101, MCP_42 to MCP_110, MCP_5 to MCP_111
Connections:
- removed net DATA_PIXEL31: PIXEL_31.5
- removed net GP: ENC_54.3, ENC_61.3, ENC_62.3, ENC_63.3, ENC_64.3, ENC_81.3, ENC_82.3, ENC_83.3, RB22.1, RB28.1, RB40.1, RB55.1, RB61.1, RB67.1, RB73.1, RB79.1, RPD11.1, RPD16.1, RPD18.1, RPD20.1, RPD22.1, RPD24.1, RPD5.1, RPD7.1
- removed net GPA: ENC_54.A, ENC_61.A, ENC_62.A, ENC_63.A, ENC_64.A, ENC_81.A, ENC_82.A, RB20.1, RB26.1, RB44.1, RB53.1, RB59.1, RB65.1, RB71.1, RB77.1, SW_65.3, SW_65.4
- removed net GPB: ENC_54.B, ENC_61.B, ENC_62.B, ENC_63.B, ENC_64.B, ENC_81.B, ENC_82.B, RB21.1, RB27.1, RB54.1, RB60.1, RB66.1, RB72.1, RB78.1
- removed net GPB0_12: MCP_001.1
- removed net INTA_41: MCP_101.20
- removed net INTA_42: MCP_110.20
- removed net INTA_5: MCP_111.20
- removed net INTB_41: MCP_101.19
- removed net INTB_42: MCP_110.19
- removed net INTB_5: MCP_111.19
- removed net JOY_SEL: JOYSTICK.2
- removed net JOY_XOUT: JOYSTICK.4
- removed net JOY_YOUT: JOYSTICK.3
- removed net N$1: TFT_EXT.10, TFT_EXT.11, TFT_EXT.12, TFT_EXT.2, TFT_EXT.3, TFT_EXT.4, TFT_EXT.5, TFT_EXT.6, TFT_EXT.8
- removed net PIXEL_01: PIXEL_01.5
- removed net PIXEL_65: PIXEL_65.5
- removed net SPI1_SCK: F446.21
- removed net SPI2_SCK: F446.34
- removed net SPI3_SCK: F446.51
- new net GPIO_EXTI0: F446.5, MCP_101.19
- new net GPIO_EXTI13: F446.2, MCP_101.20
- net 3V3: now also CONN_STH_BRD_1.2, CONN_STH_BRD_1.4, CONN_STH_BRD_2.2, CONN_STH_BRD_2.4, MCP_111.15; no longer JOYSTICK.5
- net ADC1_IN1: now also ANALOG_IN.4
- net ADC1_IN10: now also ANALOG_IN.2
- net ADC1_IN4: now also ANALOG_IN.3
- net GND: now also ANALOG_IN.1, CONN_STH_BRD_1.1, CONN_STH_BRD_2.1, LED_3V3.C, LED_5V.C, UART_ANALOG.1, UART_DISCO.1, UART_MIDI.1; no longer 3V3.C, 5V.C, JOYSTICK.1, MCP_111.15
- net GPA0_32: now also RB44.1, SW_65.3, SW_65.4
- net GPA0_41: now also ENC_81.3, RB79.1, RPD24.1
- net GPA1_32: now also ENC_64.3, RB73.1, RPD22.1
- net GPA1_41: now also ENC_82.3, RB22.1, RPD5.1
- net GPA2_32: now also ENC_64.B, RB72.1
- net GPA2_41: now also ENC_82.A, RB20.1
- net GPA3_32: now also ENC_64.A, RB71.1
- net GPA3_41: now also ENC_82.B, RB21.1
- net GPA4_32: now also ENC_63.3, RB67.1, RPD20.1
- net GPA4_41: now also ENC_83.3, RB40.1, RPD11.1
- net GPA5_32: now also ENC_63.B, RB66.1
- net GPA5_41: now also TFT_EXT.5
- net GPA6_32: now also ENC_63.A, RB65.1
- net GPA6_41: now also TFT_EXT.3
- net GPA7_32: now also ENC_62.3, RB61.1, RPD18.1
- net GPA7_41: now also TFT_EXT.2
- net GPB0_32: now also ENC_62.B, RB60.1
- net GPB0_41: now also TFT_EXT.11
- net GPB1_32: now also ENC_62.A, RB59.1
- net GPB1_41: now also TFT_EXT.12
- net GPB2_32: now also ENC_61.B, RB54.1
- net GPB2_41: now also TFT_EXT.10
- net GPB3_32: now also ENC_61.A, RB53.1
- net GPB3_41: now also TFT_EXT.8
- net GPB4_32: now also ENC_61.3, RB55.1, RPD16.1
- net GPB4_41: now also TFT_EXT.6
- net GPB5_32: now also ENC_54.A, RB26.1
- net GPB5_41: now also TFT_EXT.4
- net GPB6_32: now also ENC_54.B, RB27.1
- net GPB6_41: now also ENC_81.A, RB77.1
- net GPB7_32: now also ENC_54.3, RB28.1, RPD7.1
- net GPB7_41: now also ENC_81.B, RB78.1
- net GPIO_EXTI1: now also CONN_STH_BRD_1.17
- net GPIO_EXTI10: now also CONN_STH_BRD_1.10
- net GPIO_EXTI11: now also CONN_STH_BRD_1.7
- net GPIO_EXTI12: now also CONN_STH_BRD_1.8
- net GPIO_EXTI14: now also CONN_STH_BRD_1.18
- net GPIO_EXTI15: now also CONN_STH_BRD_1.15
- net GPIO_EXTI2: now also MCP_110.19
- net GPIO_EXTI3: now also MCP_110.20
- net GPIO_EXTI4: now also MCP_111.20
- net GPIO_EXTI5: now also MCP_111.19
- net GPIO_EXTI6: now also CONN_STH_BRD_1.16
- net GPIO_EXTI7: now also CONN_STH_BRD_1.13
- net GPIO_EXTI8: now also CONN_STH_BRD_1.14
- net GPIO_EXTI9: now also CONN_STH_BRD_1.9
- net I2C1_SCL: now also MCP_101.12, MCP_110.12, MCP_111.12, R194.1, R199.1, R204.1; no longer MCP_000.12, MCP_001.12, R186.1, R4.1
- net I2C1_SDA: now also MCP_101.13, MCP_110.13, MCP_111.13, R198.1, R203.1, R205.1; no longer MCP_000.13, MCP_001.13, R187.1, R5.1
- net I2C2_SCL: now also CONN_STH_BRD_1.20, CONN_STH_BRD_2.20
- net I2C2_SDA: now also CONN_STH_BRD_1.5, CONN_STH_BRD_2.5
- net I2C3_SCL: now also CONN_STH_BRD_1.12, CONN_STH_BRD_2.12, MCP_000.12, MCP_001.12, R186.1, R4.1; no longer MCP_101.12, MCP_110.12, MCP_111.12, R194.1, R199.1, R204.1
- net I2C3_SDA: now also CONN_STH_BRD_1.11, CONN_STH_BRD_2.11, MCP_000.13, MCP_001.13, R187.1, R5.1; no longer MCP_101.13, MCP_110.13, MCP_111.13, R198.1, R203.1, R205.1
- net INTA_11: now also CONN_STH_BRD_2.8
- net INTA_12: now also CONN_STH_BRD_2.9
- net INTA_2: now also CONN_STH_BRD_2.13
- net INTA_31: now also CONN_STH_BRD_2.18
- net INTA_32: now also CONN_STH_BRD_2.15
- net INTB_11: now also CONN_STH_BRD_2.7
- net INTB_12: now also CONN_STH_BRD_2.10
- net INTB_2: now also CONN_STH_BRD_2.14
- net INTB_31: now also CONN_STH_BRD_2.17
- net INTB_32: now also CONN_STH_BRD_2.16
- net N$53: now also LED_5V.A; no longer 5V.A
- net N$57: now also LED_3V3.A; no longer 3V3.A
- net RST: now also CONN_STH_BRD_1.3, CONN_STH_BRD_2.3
- net SPI1_MOSI: now also CONN_STH_BRD_1.6, CONN_STH_BRD_2.6
- net SPI2_MOSI: now also PIXEL_71.6; no longer PIXEL_51.6
- net SPI3_MOSI: now also CONN_STH_BRD_1.19, CONN_STH_BRD_2.19, PIXEL_51.6; no longer PIXEL_71.6
- net UART4_RX: now also UART_ANALOG.2
- net UART4_TX: now also UART_ANALOG.3
- net USART1_RX: now also UART_DISCO.2
- net USART1_TX: now also UART_DISCO.3
- net USART2_RX: now also UART_MIDI.2
- net USART2_TX: now also UART_MIDI.3
Routing:
- net 3V3: track 3581.1 -> 3921.5 mm, vias 27 -> 36
- net RST: track 431.6 -> 624.2 mm, vias 12 -> 18
- net GPIO_EXTI4: track 0.00 -> 142.0 mm, vias 0 -> 2
- net GPIO_EXTI5: track 0.00 -> 142.0 mm, vias 0 -> 2
- net INTB_32: track 0.00 -> 126.1 mm, vias 0 -> 4
- net INTA_32: track 0.00 -> 125.5 mm, vias 0 -> 4
- net INTB_11: track 0.00 -> 120.2 mm, vias 0 -> 1
- net INTA_12: track 100.4 -> 205.7 mm, vias 2 -> 3
- net INTB_12: track 97.9 -> 203.1 mm, vias 2 -> 3
- net I2C3_SCL: track 125.6 -> 224.2 mm, vias 3 -> 4
- net I2C3_SDA: track 132.6 -> 229.2 mm, vias 3 -> 4
- net GPA4_41: track 0.00 -> 89.4 mm, vias 0 -> 1
- net GPA0_32: track 0.00 -> 87.2 mm, vias 0 -> 1
- net INTA_11: track 35.7 -> 121.4 mm, vias 2 -> 1
- net INTA_31: track 0.00 -> 74.7 mm, vias 0 -> 2
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- added copper zone on layer 1, net GND
- added copper zone on layer 16, net GND
Other:
- board text added: "RAINBOW by SYD X. REY (c) 2021"
- board text removed: "RAINBOW by SYD X. REY & MARION MUCCIANTE (c) 2021"
