File: front-pane/eagle-schematics/v3/STM32F446 front pane - v3.sch (EAGLE design)
At the start: 11 parts

Commit message: Updated front pane
Parts:
- removed C1, C2, C3: 10n, stock-perso:PASSIF-CAP-0805
- removed PIXEL0: NEOPIXEL-TLC59731DR, stock-perso:NEOPIXEL-TLC59731DR
- added 0V/5V: (no value), stock-perso:PINHEADER-M04PL
- added 3V3, GREEN: (no value), Passives:LED-0805
- added 5V: (no value), Passives:LED-0603
- added C10, C11, C12, C16, C17, C18, C22, C23, C24, C28, C29, C30, C34, C35, C36, C4, C40, C41, C42, C46, C47, C48, C5, C6, C7, C8, C9, CB1, CB10, CB100, CB104, CB105, CB106, CB11, CB110, CB111, CB112, CB116, CB117, CB118, CB12, CB13, CB14, CB15, CB16, CB17, CB18, CB19, CB2, CB20, CB21, CB22, CB23, CB24, CB25, CB26, CB27, CB28, CB29, CB3, CB30, CB31, CB32, CB33, CB34, CB35, CB36, CB37, CB38, CB39, CB4, CB40, CB41, CB42, CB43, CB44, CB45, CB47, CB48, CB49, CB5, CB50, CB51, CB52, CB53, CB54, CB55, CB56, CB57, CB58, CB59, CB6, CB60, CB61, CB62, CB63, CB64, CB65, CB66, CB67, CB68, CB70, CB71, CB72, CB73, CB74, CB75, CB76, CB77, CB78, CB79, CB8, CB80, CB81, CB82, CB83, CB84, CB85, CB89, CB9, CB90, CB91, CB92, CB93, CB94, CB98, CB99: 10n, stock-perso:PASSIF-CAP-0805
- added C55, C66, C67, C68, C69, C70: 0.1uF, MyComponents:C-US0805
- added C60: 2.2uF, MyComponents:C-US0805
- added C62: 10u, MyComponents:CPOL-US2917
- added C65: 100 uF, MyComponents:CPOL-US2917
- added C71: 1.0uF, MyComponents:C-US0805
- added C76: 1u, rcl:C-EUC1206
- added CDEC1, CDEC10, CDEC11, CDEC12, CDEC14, CDEC15, CDEC16, CDEC17, CDEC18, CDEC19, CDEC2, CDEC20, CDEC22, CDEC23, CDEC24, CDEC25, CDEC26, CDEC28, CDEC29, CDEC3, CDEC31, CDEC33, CDEC35, CDEC37, CDEC4, CDEC5, CDEC6, CDEC7, CDEC8, CDEC9, CDEC_11A, CDEC_12A, CDEC_2A1, CDEC_2A2, CDEC_2A3, CPOL13, CPOL21, CPOL30, CPOL32, CPOL36, CPOL39: 10u, stock-perso:PASSIF-CPOL-US2917
- added CDEC13, CDEC21, CDEC30, CDEC32, CDEC36, CDEC39, CDEC_11B, CDEC_12B, CDEC_2B1, CDEC_2B2, CDEC_2B3, CPOL1, CPOL10, CPOL11, CPOL12, CPOL14, CPOL15, CPOL16, CPOL17, CPOL18, CPOL19, CPOL2, CPOL20, CPOL22, CPOL23, CPOL24, CPOL25, CPOL26, CPOL28, CPOL29, CPOL3, CPOL31, CPOL33, CPOL35, CPOL37, CPOL4, CPOL5, CPOL6, CPOL7, CPOL8, CPOL9: 100n, stock-perso:PASSIF-CAP-0805
- added CDEC_1, CDEC_10, CDEC_11, CDEC_12, CDEC_13, CDEC_2, CDEC_3, CDEC_4, CDEC_5, CDEC_6, CDEC_7, CDEC_8, CDEC_9: 100n, stock-perso:PASSIF-CAP-1206
- added ENC_01, ENC_02, ENC_11, ENC_13, ENC_14, ENC_21, ENC_23, ENC_3, ENC_41, ENC_44, ENC_45, ENC_48, ENC_51, ENC_53, ENC_54, ENC_55, ENC_56, ENC_57, ENC_61, ENC_62, ENC_63, ENC_64, ENC_71, ENC_72, ENC_73, ENC_74, ENC_75, ENC_81, ENC_82, ENC_83, ENC_84, ENC_85, ENC_86, ENC_87, ENC_88, S24, S31, S34, S35: (no value), stock-perso:ENCODER-RGB-SWITCH-NO_NUT
- added F446: STM32F446RCT7, STM32F446RCT7:STM32F446RCT7
- added I2C1, MIDI: (no value), con-lstb:MA03-1
- added L1: 1 uH, MyComponents:L-USL0805
- added LED1, LED2, LED22, LED4, LED6, LED7, LED_42, LED_43, LED_46, LED_47: CZXR-80RGB03-A, OPL_Optoelectronics:DIP-LED-RGB-COMMON-ANODE(4P-D8MM)
- added MCP_11, MCP_12, MCP_2, MCP_31, MCP_32: MCP23017, a_ranger_work:MCP23017
- added PIXEL_01, PIXEL_02, PIXEL_03, PIXEL_11, PIXEL_12, PIXEL_13, PIXEL_14, PIXEL_21, PIXEL_22, PIXEL_23, PIXEL_24, PIXEL_31, PIXEL_32, PIXEL_33, PIXEL_34, PIXEL_35, PIXEL_41, PIXEL_42, PIXEL_43, PIXEL_44, PIXEL_45, PIXEL_46, PIXEL_47, PIXEL_48, PIXEL_51, PIXEL_52, PIXEL_53, PIXEL_54, PIXEL_55, PIXEL_56, PIXEL_57, PIXEL_61, PIXEL_62, PIXEL_63, PIXEL_64, PIXEL_65, PIXEL_71, PIXEL_72, PIXEL_73, PIXEL_74, PIXEL_75, PIXEL_81, PIXEL_83, PIXEL_84, PIXEL_85, PIXEL_86, PIXEL_87, PIXEL_88, PIXE_82: NEOPIXEL-TLC59731DR, stock-perso:NEOPIXEL-TLC59731DR
- added R10, R100, R101, R102, R103, R104, R109, R11, R110, R111, R112, R113, R114, R115, R116, R117, R118, R12, R123, R124, R125, R126, R127, R128, R129, R130, R131, R132, R133, R134, R135, R136, R137, R138, R139, R140, R141, R142, R143, R144, R145, R146, R147, R148, R150, R151, R152, R153, R154, R155, R156, R157, R158, R159, R160, R161, R162, R163, R164, R167, R168, R169, R17, R170, R171, R172, R173, R174, R175, R176, R177, R178, R179, R18, R180, R181, R183, R184, R185, R188, R189, R19, R190, R191, R192, R193, R195, R196, R197, R200, R201, R202, R24, R25, R26, R31, R32, R33, R34, R35, R36, R37, R38, R39, R40, R45, R46, R47, R48, R49, R50, R51, R52, R53, R54, R59, R60, R61, R62, R63, R64, R65, R66, R67, R68, R73, R74, R75, R76, R77, R78, R80, R82, R83, R84, R85, R86, R94, R96, R97, R98, R99: 100, stock-perso:PASSIF-RESISTOR-1206
- added R105, R119, R13, R20, R27, R41, R55, R69, R88, RPD1, RPD10, RPD11, RPD12, RPD14, RPD15, RPD16, RPD17, RPD18, RPD19, RPD2, RPD20, RPD22, RPD23, RPD24, RPD25, RPD26, RPD28, RPD29, RPD3, RPD31, RPD33, RPD35, RPD37, RPD4, RPD5, RPD6, RPD7, RPD8, RPD9: 10k, stock-perso:PASSIF-RESISTOR-1206
- added R106, R107, R108, R120, R121, R122, R14, R15, R16, R21, R22, R23, R28, R29, R30, R42, R43, R44, R56, R57, R58, R70, R71, R72, R89, R91, R93, RB1, RB10, RB100, RB104, RB105, RB106, RB11, RB110, RB111, RB112, RB116, RB117, RB118, RB12, RB13, RB14, RB15, RB16, RB17, RB18, RB19, RB2, RB20, RB21, RB22, RB23, RB24, RB25, RB26, RB27, RB28, RB29, RB3, RB30, RB31, RB32, RB33, RB34, RB35, RB36, RB37, RB38, RB39, RB4, RB40, RB41, RB42, RB43, RB44, RB45, RB47, RB48, RB49, RB5, RB50, RB51, RB52, RB53, RB54, RB55, RB56, RB57, RB58, RB59, RB6, RB60, RB61, RB62, RB63, RB64, RB65, RB66, RB67, RB68, RB70, RB71, RB72, RB73, RB74, RB75, RB76, RB77, RB78, RB79, RB8, RB80, RB81, RB82, RB83, RB84, RB85, RB89, RB9, RB90, RB91, RB92, RB93, RB94, RB98, RB99: 470, stock-perso:PASSIF-RESISTOR-1206
- added R149, R165, R166, R182, R186, R187, R4, R5: 1k, 6P1_EVB:R-US_R0805
- added R79: 100k, MyComponents:R-US0805
- added R81: 10K, MyComponents:R-US0805
- added R87: 1, MyComponents:R-US0805
- added R90, R95: 1k, MyComponents:R-US0805
- added R92: 470, MyComponents:R-US0805
- added S2: SWITCH-SKRKAEE020, stock-perso:SWITCH-SKRKAEE020
- added S3: JOYSTICK_THUMB, stock-perso:JOYSTICK_THUMB
- added S32, S33, SW_42, SW_43, SW_46, SW_47, SW_52, SW_65, S_12, S_22: B3F-1000, Switch:B3F-1000
- added STLINK: 75867-331LF, MyComponents:MA03-2
- added TLV75533: TLV75533PDBVR, TLV75533PDBVR:TLV75533PDBVR
- R1, R2: value 100 -> 1k; device stock-perso:PASSIF-RESISTOR-1206 -> 6P1_EVB:R-US_R0805
- R6: value 10k -> 100
- R7, R8, R9: value 470 -> 100
Connections:
- removed net GPA0_0: R7.1
- removed net GPA1_0: R8.1
- removed net GPA2_0: R6.1, R9.1
- removed net N$1: R1.2
- removed net N$10: C1.2, R7.2
- removed net N$11: C2.2, R8.2
- removed net N$2: R2.2
- removed net N$3: R3.2
- removed net N$4: PIXEL0.OUT0, R1.1
- removed net N$5: PIXEL0.OUT1, R2.1
- removed net N$6: PIXEL0.OUT2, R3.1
- removed net N$8: C3.1, R9.2
- removed net SDO_PIXEL0: PIXEL0.SDO
- new net 5V: 0V/5V.3, 0V/5V.4, C62.+, C76.2, R92.1, TLV75533.EN, TLV75533.IN
- new net ADC1_IN1: F446.PA1
- new net ADC1_IN10: F446.PC0
- new net ADC1_IN4: F446.PA4
- new net BOOT1: F446.BOOT0, R81.1
- new net DATA_PIXEL11: PIXEL_11.SDO, PIXEL_21.SDI
- new net DATA_PIXEL12: PIXEL_11.SDI, PIXEL_12.SDO
- new net DATA_PIXEL13: PIXEL_12.SDI, PIXEL_13.SDO
- new net DATA_PIXEL14: PIXEL_13.SDI, PIXEL_14.SDO
- new net DATA_PIXEL21: PIXEL_21.SDO, PIXEL_22.SDI
- new net DATA_PIXEL22: PIXEL_22.SDO, PIXEL_23.SDI
- new net DATA_PIXEL23: PIXEL_23.SDO, PIXEL_24.SDI
- new net DATA_PIXEL24: PIXEL_24.SDO, PIXEL_35.SDI
- new net DATA_PIXEL31: PIXEL_31.SDO
- new net DATA_PIXEL32: PIXEL_31.SDI, PIXEL_32.SDO
- new net DATA_PIXEL33: PIXEL_32.SDI, PIXEL_33.SDO
- new net DATA_PIXEL34: PIXEL_33.SDI, PIXEL_34.SDO
- new net DATA_PIXEL35: PIXEL_34.SDI, PIXEL_35.SDO
- new net GP: ENC_01.SW, ENC_02.SW, ENC_3.SW, ENC_54.SW, ENC_61.SW, ENC_62.SW, ENC_63.SW, ENC_64.SW, ENC_71.SW, ENC_72.SW, ENC_73.SW, ENC_74.SW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
- new net GPA: ENC_01.A, ENC_02.A, ENC_3.A, ENC_54.A, ENC_61.A, ENC_62.A, ENC_63.A, ENC_64.A, ENC_71.A, ENC_72.A, ENC_73.A, ENC_74.A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
- new net GPA0_11: MCP_11.GPA0, R71.1, S24.B
- new net GPA0_12: MCP_12.GPA0, R121.1, S35.B
- new net GPA0_2: MCP_2.GPA0, RB70.1, SW_47.3, SW_47.4
- new net GPA0_31: ENC_51.A, MCP_31.GPA0, RB8.1
- new net GPA0_32: MCP_32.GPA0
- new net GPA1_11: MCP_11.GPA1, R70.1, S24.A
- new net GPA1_12: MCP_12.GPA1, R119.1, R122.1, S35.SW
- new net GPA1_2: ENC_45.A, MCP_2.GPA1, RB23.1
- new net GPA1_31: ENC_51.B, MCP_31.GPA1, RB9.1
- new net GPA1_32: MCP_32.GPA1
- new net GPA2_11: MCP_11.GPA2, R69.1, R72.1, S24.SW
- new net GPA2_12: MCP_12.GPA2, R120.1, S35.A
- new net GPA2_2: ENC_45.B, MCP_2.GPA2, RB24.1
- new net GPA2_31: ENC_51.SW, MCP_31.GPA2, RB10.1, RPD1.1
- new net GPA2_32: MCP_32.GPA2
- new net GPA3_11: ENC_23.A, MCP_11.GPA3, R56.1
- new net GPA3_12: MCP_12.GPA3, R107.1, S34.B
- new net GPA3_2: ENC_45.SW, MCP_2.GPA3, RB25.1, RPD6.1
- new net GPA3_31: MCP_31.GPA3, RB5.1, SW_52.3, SW_52.4
- new net GPA3_32: MCP_32.GPA3
- new net GPA4_11: ENC_23.B, MCP_11.GPA4, R57.1
- new net GPA4_12: MCP_12.GPA4, R106.1, S34.A
- new net GPA4_2: MCP_2.GPA4, RB68.1, SW_46.3, SW_46.4
- new net GPA4_31: ENC_53.SW, MCP_31.GPA4, RB16.1, RPD3.1
- new net GPA4_32: MCP_32.GPA4
- new net GPA5_11: ENC_23.SW, MCP_11.GPA5, R55.1, R58.1
- new net GPA5_12: MCP_12.GPA5, R105.1, R108.1, S34.SW
- new net GPA5_2: ENC_48.A, MCP_2.GPA5, RB29.1
- new net GPA5_31: ENC_53.A, MCP_31.GPA5, RB14.1
- new net GPA5_32: MCP_32.GPA5
- new net GPA6_11: ENC_11.SW, MCP_11.GPA6, R13.1, R16.1
- new net GPA6_12: MCP_12.GPA6, RB6.1, S33.3, S33.4
- new net GPA6_2: ENC_48.SW, MCP_2.GPA6, RB31.1, RPD8.1
- new net GPA6_31: ENC_53.B, MCP_31.GPA6, RB15.1
- new net GPA6_32: MCP_32.GPA6
- new net GPA7_11: MCP_11.GPA7, RB2.1, S_12.3, S_12.4
- new net GPA7_12: MCP_12.GPA7, RB1.1, S32.3, S32.4
- new net GPA7_2: ENC_48.B, MCP_2.GPA7, RB30.1
- new net GPA7_31: ENC_57.SW, MCP_31.GPA7, RB49.1, RPD14.1
- new net GPA7_32: MCP_32.GPA7
- new net GPB: ENC_01.B, ENC_02.B, ENC_3.B, ENC_54.B, ENC_61.B, ENC_62.B, ENC_63.B, ENC_64.B, ENC_71.B, ENC_72.B, ENC_73.B, ENC_74.B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
- new net GPB0_11: ENC_11.A, MCP_11.GPB0, R14.1
- new net GPB0_12: MCP_12.GPB0
- new net GPB0_2: MCP_2.GPB0, RB3.1, SW_42.3, SW_42.4
- new net GPB0_31: ENC_57.B, MCP_31.GPB0, RB48.1
- new net GPB0_32: MCP_32.GPB0
- new net GPB1_11: ENC_11.B, MCP_11.GPB1, R15.1
- new net GPB1_12: MCP_12.GPB1, R91.1, S31.B
- new net GPB1_2: ENC_44.A, MCP_2.GPB1, RB17.1
- new net GPB1_31: ENC_57.A, MCP_31.GPB1, RB47.1
- new net GPB1_32: MCP_32.GPB1
- new net GPB2_11: ENC_13.A, MCP_11.GPB2, R21.1
- new net GPB2_12: MCP_12.GPB2, R88.1, R93.1, S31.SW
- new net GPB2_2: ENC_44.B, MCP_2.GPB2, RB18.1
- new net GPB2_31: ENC_56.SW, MCP_31.GPB2, RB43.1, RPD12.1
- new net GPB2_32: MCP_32.GPB2
- new net GPB3_11: ENC_13.B, MCP_11.GPB3, R22.1
- new net GPB3_12: MCP_12.GPB3, R89.1, S31.A
- new net GPB3_2: ENC_44.SW, MCP_2.GPB3, RB19.1, RPD4.1
- new net GPB3_31: ENC_56.B, MCP_31.GPB3, RB42.1
- new net GPB3_32: MCP_32.GPB3
- new net GPB4_11: ENC_13.SW, MCP_11.GPB4, R20.1, R23.1
- new net GPB4_12: ENC_21.SW, MCP_12.GPB4, R41.1, R44.1
- new net GPB4_2: ENC_41.A, MCP_2.GPB4, RB11.1
- new net GPB4_31: ENC_56.A, MCP_31.GPB4, RB41.1
- new net GPB4_32: MCP_32.GPB4
- new net GPB5_11: ENC_14.SW, MCP_11.GPB5, R27.1, R30.1
- new net GPB5_12: ENC_21.A, MCP_12.GPB5, R42.1
- new net GPB5_2: ENC_41.B, MCP_2.GPB5, RB12.1
- new net GPB5_31: ENC_55.A, MCP_31.GPB5, RB35.1
- new net GPB5_32: MCP_32.GPB5
- new net GPB6_11: ENC_14.A, MCP_11.GPB6, R28.1
- new net GPB6_12: ENC_21.B, MCP_12.GPB6, R43.1
- new net GPB6_2: ENC_41.SW, MCP_2.GPB6, RB13.1, RPD2.1
- new net GPB6_31: ENC_55.B, MCP_31.GPB6, RB36.1
- new net GPB6_32: MCP_32.GPB6
- new net GPB7_11: ENC_14.B, MCP_11.GPB7, R29.1
- new net GPB7_12: MCP_12.GPB7, RB4.1, S_22.3, S_22.4
- new net GPB7_2: MCP_2.GPB7, RB45.1, SW_43.3, SW_43.4
- new net GPB7_31: ENC_55.SW, MCP_31.GPB7, RB37.1, RPD10.1
- new net GPB7_32: MCP_32.GPB7
- new net GPIO_EXTI1: F446.PB1
- new net GPIO_EXTI10: F446.PA10
- new net GPIO_EXTI11: F446.PA11
- new net GPIO_EXTI12: F446.PA12
- new net GPIO_EXTI14: F446.PB14
- new net GPIO_EXTI15: F446.PB15
- new net GPIO_EXTI2: F446.PC2
- new net GPIO_EXTI3: F446.PC3
- new net GPIO_EXTI4: F446.PC4
- new net GPIO_EXTI5: F446.PC5
- new net GPIO_EXTI6: F446.PC6
- new net GPIO_EXTI7: F446.PC7
- new net GPIO_EXTI8: F446.PC8
- new net GPIO_EXTI9: F446.PA9
- new net I2C1_SCL: F446.PB8, I2C1.2, MCP_11.SCL, MCP_12.SCL, R186.1, R4.1
- new net I2C1_SDA: F446.PB9, I2C1.1, MCP_11.SDA, MCP_12.SDA, R187.1, R5.1
- new net I2C2_SCL: F446.PB10, MCP_2.SCL, MCP_31.SCL, MCP_32.SCL, R1.1, R149.1, R166.1
- new net I2C2_SDA: F446.PC12, MCP_2.SDA, MCP_31.SDA, MCP_32.SDA, R165.1, R182.1, R2.1
- new net I2C3_SCL: F446.PA8
- new net I2C3_SDA: F446.PC9
- new net INTA_11: MCP_11.INTA
- new net INTA_12: MCP_12.INTA
- new net INTA_2: MCP_2.INTA
- new net INTA_31: MCP_31.INTA
- new net INTA_32: MCP_32.INTA
- new net INTB_11: MCP_11.INTB
- new net INTB_12: MCP_12.INTB
- new net INTB_2: MCP_2.INTB
- new net INTB_31: MCP_31.INTB
- new net INTB_32: MCP_32.INTB
- new net N$10160: PIXEL_46.OUT0, R188.1
- new net N$10161: PIXEL_46.OUT1, R192.1
- new net N$10162: PIXEL_46.OUT2, R193.1
- new net N$10163: CB68.2, RB68.2
- new net N$10164: LED_46.R, R193.2
- new net N$10165: LED_46.B, R192.2
- new net N$10166: LED_46.G, R188.2
- new net N$10174: ENC_02.-R, R189.2
- new net N$10175: ENC_02.-G, R190.2
- new net N$10176: ENC_02.-B, R191.2
- new net N$10177: PIXEL_02.OUT0, R189.1
- new net N$10178: PIXEL_02.OUT1, R190.1
- new net N$10179: PIXEL_02.OUT2, R191.1
- new net N$10180: CB110.2, RB110.2
- new net N$10181: CB111.2, RB111.2
- new net N$10182: CB112.1, RB112.2
- new net N$10540: ENC_3.-R, R195.2
- new net N$10541: ENC_3.-G, R196.2
- new net N$10542: ENC_3.-B, R197.2
- new net N$10543: PIXEL_03.OUT0, R195.1
- new net N$10544: PIXEL_03.OUT1, R196.1
- new net N$10545: PIXEL_03.OUT2, R197.1
- new net N$10546: CB116.2, RB116.2
- new net N$10547: CB117.2, RB117.2
- new net N$10548: CB118.1, RB118.2
- new net N$1069: ENC_13.-R, R17.2
- new net N$1070: ENC_13.-G, R18.2
- new net N$1071: ENC_13.-B, R19.2
- new net N$1072: PIXEL_13.OUT0, R17.1
- new net N$1073: PIXEL_13.OUT1, R18.1
- new net N$1074: PIXEL_13.OUT2, R19.1
- new net N$1075: C7.2, R21.2
- new net N$1076: C8.2, R22.2
- new net N$1077: C9.1, R23.2
- new net N$108: R87.2, TLV75533.OUT
- new net N$10888: PIXEL_47.OUT0, R200.1
- new net N$10889: PIXEL_47.OUT1, R201.1
- new net N$10890: PIXEL_47.OUT2, R202.1
- new net N$10891: CB70.2, RB70.2
- new net N$10892: LED_47.R, R202.2
- new net N$10893: LED_47.B, R201.2
- new net N$10894: LED_47.G, R200.2
- new net N$109: L1.1, R87.1
- new net N$1252: ENC_14.-R, R24.2
- new net N$1253: ENC_14.-G, R25.2
- new net N$1254: ENC_14.-B, R26.2
- new net N$1255: PIXEL_14.OUT0, R24.1
- new net N$1256: PIXEL_14.OUT1, R25.1
- new net N$1257: PIXEL_14.OUT2, R26.1
- new net N$1258: C10.2, R28.2
- new net N$1259: C11.2, R29.2
- new net N$1260: C12.1, R30.2
- new net N$1435: PIXEL_32.OUT2, R7.1
- new net N$1436: CB1.2, RB1.2
- new net N$1437: LED1.R, R7.2
- new net N$1438: LED1.B, R6.2
- new net N$1439: LED1.G, R3.2
- new net N$1614: PIXEL_12.OUT0, R8.1
- new net N$1615: PIXEL_12.OUT1, R9.1
- new net N$1616: PIXEL_12.OUT2, R31.1
- new net N$1617: CB2.2, RB2.2
- new net N$1618: ENC_21.-R, R38.2
- new net N$1619: ENC_21.-G, R39.2
- new net N$1620: ENC_21.-B, R40.2
- new net N$1621: PIXEL_21.OUT0, R38.1
- new net N$1622: PIXEL_21.OUT1, R39.1
- new net N$1623: PIXEL_21.OUT2, R40.1
- new net N$1624: C16.2, R42.2
- new net N$1625: C17.2, R43.2
- new net N$1626: C18.1, R44.2
- new net N$1801: LED2.R, R31.2
- new net N$1802: LED2.B, R9.2
- new net N$1803: LED2.G, R8.2
- new net N$1978: PIXEL_42.OUT1, R123.1
- new net N$1979: ENC_51.-R, R33.2
- new net N$1980: ENC_51.-G, R34.2
- new net N$1981: ENC_51.-B, R45.2
- new net N$1982: PIXEL_51.OUT0, R33.1
- new net N$1983: PIXEL_51.OUT1, R34.1
- new net N$1984: ENC_23.-R, R52.2
- new net N$1985: ENC_23.-G, R53.2
- new net N$1986: ENC_23.-B, R54.2
- new net N$1987: PIXEL_23.OUT0, R52.1
- new net N$1988: PIXEL_23.OUT1, R53.1
- new net N$1989: PIXEL_23.OUT2, R54.1
- new net N$1990: C22.2, R56.2
- new net N$1991: C23.2, R57.2
- new net N$1992: C24.1, R58.2
- new net N$2167: PIXEL_51.OUT2, R45.1
- new net N$2168: CB8.2, RB8.2
- new net N$2169: CB9.2, RB9.2
- new net N$2170: CB10.1, RB10.2
- new net N$2342: PIXEL_22.OUT0, R35.1
- new net N$2343: PIXEL_22.OUT1, R36.1
- new net N$2344: PIXEL_22.OUT2, R37.1
- new net N$2345: CB4.2, RB4.2
- new net N$2346: LED22.R, R37.2
- new net N$2347: LED22.B, R36.2
- new net N$2348: LED22.G, R35.2
- new net N$2350: R66.2, S24.-R
- new net N$2351: R67.2, S24.-G
- new net N$2352: R68.2, S24.-B
- new net N$2353: PIXEL_24.OUT0, R66.1
- new net N$2354: PIXEL_24.OUT1, R67.1
- new net N$2355: PIXEL_24.OUT2, R68.1
- new net N$2356: C28.2, R70.2
- new net N$2357: C29.2, R71.2
- new net N$2358: C30.1, R72.2
- new net N$2709: ENC_41.-R, R46.2
- new net N$2710: ENC_41.-G, R47.2
- new net N$2711: ENC_41.-B, R51.2
- new net N$2712: PIXEL_41.OUT0, R46.1
- new net N$2713: PIXEL_41.OUT1, R47.1
- new net N$2714: PIXEL_41.OUT2, R51.1
- new net N$2715: CB11.2, RB11.2
- new net N$2716: R82.2, S31.-R
- new net N$2717: R84.2, S31.-G
- new net N$2718: R85.2, S31.-B
- new net N$2719: PIXEL_31.OUT0, R82.1
- new net N$2720: PIXEL_31.OUT1, R84.1
- new net N$2721: PIXEL_31.OUT2, R85.1
- new net N$2722: C34.2, R89.2
- new net N$2723: C35.2, R91.2
- new net N$2724: C36.1, R93.2
- new net N$2899: CB12.2, RB12.2
- new net N$2900: CB13.1, RB13.2
- new net N$3070: PIXEL_33.OUT0, R48.1
- new net N$3071: PIXEL_33.OUT1, R49.1
- new net N$3072: PIXEL_33.OUT2, R50.1
- new net N$3073: CB6.2, RB6.2
- new net N$3074: LED6.R, R50.2
- new net N$3075: LED6.B, R49.2
- new net N$3076: LED6.G, R48.2
- new net N$3082: R102.2, S34.-R
- new net N$3083: R103.2, S34.-G
- new net N$3084: R104.2, S34.-B
- new net N$3085: PIXEL_34.OUT0, R102.1
- new net N$3086: PIXEL_34.OUT1, R103.1
- new net N$3087: PIXEL_34.OUT2, R104.1
- new net N$3088: C40.2, R106.2
- new net N$3089: C41.2, R107.2
- new net N$3090: C42.1, R108.2
- new net N$3439: ENC_53.-R, R59.2
- new net N$3440: ENC_53.-G, R60.2
- new net N$3441: ENC_53.-B, R61.2
- new net N$3442: PIXEL_53.OUT0, R59.1
- new net N$3443: PIXEL_53.OUT1, R60.1
- new net N$3444: PIXEL_53.OUT2, R61.1
- new net N$3445: CB14.2, RB14.2
- new net N$3446: CB15.2, RB15.2
- new net N$3447: CB16.1, RB16.2
- new net N$3448: R116.2, S35.-R
- new net N$3449: R117.2, S35.-G
- new net N$3450: R118.2, S35.-B
- new net N$3451: PIXEL_35.OUT0, R116.1
- new net N$3452: PIXEL_35.OUT1, R117.1
- new net N$3453: PIXEL_35.OUT2, R118.1
- new net N$3454: C46.2, R120.2
- new net N$3455: C47.2, R121.2
- new net N$3456: C48.1, R122.2
- new net N$3814: ENC_44.-R, R62.2
- new net N$3815: ENC_44.-G, R63.2
- new net N$3816: ENC_44.-B, R64.2
- new net N$3817: PIXEL_44.OUT0, R62.1
- new net N$3818: PIXEL_44.OUT1, R63.1
- new net N$3819: PIXEL_44.OUT2, R64.1
- new net N$3820: CB17.2, RB17.2
- new net N$3821: CB18.2, RB18.2
- new net N$3822: CB19.1, RB19.2
- new net N$4510: ENC_82.-R, R65.2
- new net N$4511: ENC_82.-G, R73.2
- new net N$4512: ENC_82.-B, R74.2
- new net N$4513: PIXE_82.OUT0, R65.1
- new net N$4514: PIXE_82.OUT1, R73.1
- new net N$4515: PIXE_82.OUT2, R74.1
- new net N$4516: CB20.2, RB20.2
- new net N$4517: CB21.2, RB21.2
- new net N$4518: CB22.1, RB22.2
- new net N$4867: ENC_45.-R, R75.2
- new net N$4868: ENC_45.-G, R76.2
- new net N$4869: ENC_45.-B, R77.2
- new net N$4870: PIXEL_45.OUT0, R75.1
- new net N$4871: PIXEL_45.OUT1, R76.1
- new net N$4872: PIXEL_45.OUT2, R77.1
- new net N$4873: CB23.2, RB23.2
- new net N$4874: CB24.2, RB24.2
- new net N$4875: CB25.1, RB25.2
- new net N$5050: ENC_54.-R, R78.2
- new net N$5051: ENC_54.-G, R80.2
- new net N$5052: ENC_54.-B, R83.2
- new net N$5053: PIXEL_54.OUT0, R78.1
- new net N$5054: PIXEL_54.OUT1, R80.1
- new net N$5055: PIXEL_54.OUT2, R83.1
- new net N$5056: CB26.2, RB26.2
- new net N$5057: CB27.2, RB27.2
- new net N$5058: CB28.1, RB28.2
- new net N$5233: ENC_48.-R, R86.2
- new net N$5234: ENC_48.-G, R94.2
- new net N$5235: ENC_48.-B, R96.2
- new net N$5236: PIXEL_48.OUT0, R86.1
- new net N$5237: PIXEL_48.OUT1, R94.1
- new net N$5238: PIXEL_48.OUT2, R96.1
- new net N$5239: CB29.2, RB29.2
- new net N$5240: CB30.2, RB30.2
- new net N$5241: CB31.1, RB31.2
- new net N$53: 5V.A, R92.2
- new net N$5416: ENC_71.-R, R97.2
- new net N$5417: ENC_71.-G, R98.2
- new net N$5418: ENC_71.-B, R99.2
- new net N$5419: PIXEL_71.OUT0, R97.1
- new net N$5420: PIXEL_71.OUT1, R98.1
- new net N$5421: PIXEL_71.OUT2, R99.1
- new net N$5422: CB32.2, RB32.2
- new net N$5423: CB33.2, RB33.2
- new net N$5424: CB34.1, RB34.2
- new net N$5599: ENC_55.-R, R100.2
- new net N$56: GREEN.A, R90.2
- new net N$5600: ENC_55.-G, R101.2
- new net N$5601: ENC_55.-B, R109.2
- new net N$5602: PIXEL_55.OUT0, R100.1
- new net N$5603: PIXEL_55.OUT1, R101.1
- new net N$5604: PIXEL_55.OUT2, R109.1
- new net N$5605: CB35.2, RB35.2
- new net N$5606: CB36.2, RB36.2
- new net N$5607: CB37.1, RB37.2
- new net N$57: 3V3.A, R95.2
- new net N$5782: ENC_83.-R, R110.2
- new net N$5783: ENC_83.-G, R111.2
- new net N$5784: ENC_83.-B, R112.2
- new net N$5785: PIXEL_83.OUT0, R110.1
- new net N$5786: PIXEL_83.OUT1, R111.1
- new net N$5787: PIXEL_83.OUT2, R112.1
- new net N$5788: CB38.2, RB38.2
- new net N$5789: CB39.2, RB39.2
- new net N$5790: CB40.1, RB40.2
- new net N$5965: ENC_56.-R, R113.2
- new net N$5966: ENC_56.-G, R114.2
- new net N$5967: ENC_56.-B, R115.2
- new net N$5968: PIXEL_56.OUT0, R113.1
- new net N$5969: PIXEL_56.OUT1, R114.1
- new net N$5970: PIXEL_56.OUT2, R115.1
- new net N$5971: CB41.2, RB41.2
- new net N$5972: CB42.2, RB42.2
- new net N$5973: CB43.1, RB43.2
- new net N$6148: PIXEL_42.OUT2, R124.1
- new net N$6149: CB3.2, RB3.2
- new net N$6150: LED_42.R, R124.2
- new net N$6151: LED_42.B, R123.2
- new net N$6152: LED_42.G, R32.2
- new net N$6327: PIXEL_52.OUT0, R125.1
- new net N$6328: PIXEL_52.OUT1, R147.1
- new net N$6329: PIXEL_52.OUT2, R148.1
- new net N$6330: CB5.2, RB5.2
- new net N$6331: ENC_57.-R, R126.2
- new net N$6332: ENC_57.-G, R127.2
- new net N$6333: ENC_57.-B, R128.2
- new net N$6334: PIXEL_57.OUT0, R126.1
- new net N$6335: PIXEL_57.OUT1, R127.1
- new net N$6336: PIXEL_57.OUT2, R128.1
- new net N$6337: CB47.2, RB47.2
- new net N$6338: CB48.2, RB48.2
- new net N$6339: CB49.1, RB49.2
- new net N$6514: ENC_84.-R, R129.2
- new net N$6515: ENC_84.-G, R130.2
- new net N$6516: ENC_84.-B, R131.2
- new net N$6517: PIXEL_84.OUT0, R129.1
- new net N$6518: PIXEL_84.OUT1, R130.1
- new net N$6519: PIXEL_84.OUT2, R131.1
- new net N$6520: CB50.2, RB50.2
- new net N$6521: CB51.2, RB51.2
- new net N$6522: CB52.1, RB52.2
- new net N$6697: ENC_61.-R, R132.2
- new net N$6698: ENC_61.-G, R133.2
- new net N$6699: ENC_61.-B, R134.2
- new net N$6700: PIXEL_61.OUT0, R132.1
- new net N$6701: PIXEL_61.OUT1, R133.1
- new net N$6702: PIXEL_61.OUT2, R134.1
- new net N$6703: CB53.2, RB53.2
- new net N$6704: CB54.2, RB54.2
- new net N$6705: CB55.1, RB55.2
- new net N$6880: ENC_72.-R, R135.2
- new net N$6881: ENC_72.-G, R136.2
- new net N$6882: ENC_72.-B, R137.2
- new net N$6883: PIXEL_72.OUT0, R135.1
- new net N$6884: PIXEL_72.OUT1, R136.1
- new net N$6885: PIXEL_72.OUT2, R137.1
- new net N$6886: CB56.2, RB56.2
- new net N$6887: CB57.2, RB57.2
- new net N$6888: CB58.1, RB58.2
- new net N$7063: ENC_62.-R, R138.2
- new net N$7064: ENC_62.-G, R139.2
- new net N$7065: ENC_62.-B, R140.2
- new net N$7066: PIXEL_62.OUT0, R138.1
- new net N$7067: PIXEL_62.OUT1, R139.1
- new net N$7068: PIXEL_62.OUT2, R140.1
- new net N$7069: CB59.2, RB59.2
- new net N$7070: CB60.2, RB60.2
- new net N$7071: CB61.1, RB61.2
- new net N$709: PIXEL_42.OUT0, R32.1
- new net N$710: PIXEL_32.OUT0, R3.1
- new net N$711: PIXEL_32.OUT1, R6.1
- new net N$712: ENC_11.-R, R10.2
- new net N$713: ENC_11.-G, R11.2
- new net N$714: ENC_11.-B, R12.2
- new net N$715: PIXEL_11.OUT0, R10.1
- new net N$716: PIXEL_11.OUT1, R11.1
- new net N$717: PIXEL_11.OUT2, R12.1
- new net N$718: C4.2, R14.2
- new net N$719: C5.2, R15.2
- new net N$720: C6.1, R16.2
- new net N$7246: ENC_85.-R, R141.2
- new net N$7247: ENC_85.-G, R142.2
- new net N$7248: ENC_85.-B, R143.2
- new net N$7249: PIXEL_85.OUT0, R141.1
- new net N$7250: PIXEL_85.OUT1, R142.1
- new net N$7251: PIXEL_85.OUT2, R143.1
- new net N$7252: CB62.2, RB62.2
- new net N$7253: CB63.2, RB63.2
- new net N$7254: CB64.1, RB64.2
- new net N$7429: ENC_63.-R, R144.2
- new net N$7430: ENC_63.-G, R145.2
- new net N$7431: ENC_63.-B, R146.2
- new net N$7432: PIXEL_63.OUT0, R144.1
- new net N$7433: PIXEL_63.OUT1, R145.1
- new net N$7434: PIXEL_63.OUT2, R146.1
- new net N$7435: CB65.2, RB65.2
- new net N$7436: CB66.2, RB66.2
- new net N$7437: CB67.1, RB67.2
- new net N$7612: LED4.R, R148.2
- new net N$7613: LED4.B, R147.2
- new net N$7614: LED4.G, R125.2
- new net N$7795: ENC_64.-R, R150.2
- new net N$7796: ENC_64.-G, R151.2
- new net N$7797: ENC_64.-B, R152.2
- new net N$7798: PIXEL_64.OUT0, R150.1
- new net N$7799: PIXEL_64.OUT1, R151.1
- new net N$7800: PIXEL_64.OUT2, R152.1
- new net N$7801: CB71.2, RB71.2
- new net N$7802: CB72.2, RB72.2
- new net N$7803: CB73.1, RB73.2
- new net N$7978: ENC_86.-R, R153.2
- new net N$7979: ENC_86.-G, R154.2
- new net N$7980: ENC_86.-B, R155.2
- new net N$7981: PIXEL_86.OUT0, R153.1
- new net N$7982: PIXEL_86.OUT1, R154.1
- new net N$7983: PIXEL_86.OUT2, R155.1
- new net N$7984: CB74.2, RB74.2
- new net N$7985: CB75.2, RB75.2
- new net N$7986: CB76.1, RB76.2
- new net N$8161: ENC_81.-R, R156.2
- new net N$8162: ENC_81.-G, R157.2
- new net N$8163: ENC_81.-B, R158.2
- new net N$8164: PIXEL_81.OUT0, R156.1
- new net N$8165: PIXEL_81.OUT1, R157.1
- new net N$8166: PIXEL_81.OUT2, R158.1
- new net N$8167: CB77.2, RB77.2
- new net N$8168: CB78.2, RB78.2
- new net N$8169: CB79.1, RB79.2
- new net N$8344: ENC_73.-R, R159.2
- new net N$8345: ENC_73.-G, R160.2
- new net N$8346: ENC_73.-B, R161.2
- new net N$8347: PIXEL_73.OUT0, R159.1
- new net N$8348: PIXEL_73.OUT1, R160.1
- new net N$8349: PIXEL_73.OUT2, R161.1
- new net N$8350: CB80.2, RB80.2
- new net N$8351: CB81.2, RB81.2
- new net N$8352: CB82.1, RB82.2
- new net N$8527: ENC_87.-R, R162.2
- new net N$8528: ENC_87.-G, R163.2
- new net N$8529: ENC_87.-B, R164.2
- new net N$8530: PIXEL_87.OUT0, R162.1
- new net N$8531: PIXEL_87.OUT1, R163.1
- new net N$8532: PIXEL_87.OUT2, R164.1
- new net N$8533: CB83.2, RB83.2
- new net N$8534: CB84.2, RB84.2
- new net N$8535: CB85.1, RB85.2
- new net N$8885: PIXEL_65.OUT0, R167.1
- new net N$8886: PIXEL_65.OUT1, R174.1
- new net N$8887: PIXEL_65.OUT2, R175.1
- new net N$8888: CB44.2, RB44.2
- new net N$8889: LED7.R, R175.2
- new net N$8890: LED7.B, R174.2
- new net N$8891: LED7.G, R167.2
- new net N$8893: ENC_88.-R, R168.2
- new net N$8894: ENC_88.-G, R169.2
- new net N$8895: ENC_88.-B, R170.2
- new net N$8896: PIXEL_88.OUT0, R168.1
- new net N$8897: PIXEL_88.OUT1, R169.1
- new net N$8898: PIXEL_88.OUT2, R170.1
- new net N$8899: CB89.2, RB89.2
- new net N$8900: CB90.2, RB90.2
- new net N$8901: CB91.1, RB91.2
- new net N$9076: ENC_74.-R, R171.2
- new net N$9077: ENC_74.-G, R172.2
- new net N$9078: ENC_74.-B, R173.2
- new net N$9079: PIXEL_74.OUT0, R171.1
- new net N$9080: PIXEL_74.OUT1, R172.1
- new net N$9081: PIXEL_74.OUT2, R173.1
- new net N$9082: CB92.2, RB92.2
- new net N$9083: CB93.2, RB93.2
- new net N$9084: CB94.1, RB94.2
- new net N$9432: PIXEL_43.OUT0, R176.1
- new net N$9433: PIXEL_43.OUT1, R180.1
- new net N$9434: PIXEL_43.OUT2, R181.1
- new net N$9435: CB45.2, RB45.2
- new net N$9436: LED_43.R, R181.2
- new net N$9437: LED_43.B, R180.2
- new net N$9438: LED_43.G, R176.2
- new net N$9442: ENC_75.-R, R177.2
- new net N$9443: ENC_75.-G, R178.2
- new net N$9444: ENC_75.-B, R179.2
- new net N$9445: PIXEL_75.OUT0, R177.1
- new net N$9446: PIXEL_75.OUT1, R178.1
- new net N$9447: PIXEL_75.OUT2, R179.1
- new net N$9448: CB98.2, RB98.2
- new net N$9449: CB99.2, RB99.2
- new net N$9450: CB100.1, RB100.2
- new net N$9808: ENC_01.-R, R183.2
- new net N$9809: ENC_01.-G, R184.2
- new net N$9810: ENC_01.-B, R185.2
- new net N$9811: PIXEL_01.OUT0, R183.1
- new net N$9812: PIXEL_01.OUT1, R184.1
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Other:
- note added: "ARP"
- note added: "EFFECTS"
- note added: "EG"
- note added: "LFO"
- note added: "MCP 11 & 12"
- note added: "OSCILLATORS"
- note added: "RGB ENCODER"
- note added: "RGB ENCODER 11"
- note added: "RGB ENCODER 13"
- note added: "RGB ENCODER 14"
- note added: "RGB ENCODER 21"
- note added: "RGB ENCODER 23"
- note added: "RGB ENCODER 24"
- note added: "RGB ENCODER 31"
- note added: "RGB ENCODER 34"
- note added: "RGB ENCODER 35"
- note added: "RGB ENCODER 41"
- note added: "RGB ENCODER 44"
- note added: "RGB ENCODER 45"
- note added: "RGB ENCODER 48"
- note added: "RGB ENCODER 51"
- note added: "RGB ENCODER 53"
- note added: "RGB ENCODER 54"
- note added: "RGB ENCODER 55"
- note added: "RGB ENCODER 56"
- note added: "RGB ENCODER 57"
- note added: "RGB ENCODER 61"
- note added: "RGB ENCODER 62"
- note added: "RGB ENCODER 63"
- note added: "RGB ENCODER 64"
- note added: "RGB ENCODER 71"
- note added: "RGB ENCODER 72"
- note added: "RGB ENCODER 73"
- note added: "RGB ENCODER 74"
- note added: "RGB ENCODER 75"
- note added: "RGB ENCODER 81"
- note added: "RGB ENCODER 82"
- note added: "RGB ENCODER 83"
- note added: "RGB ENCODER 84"
- note added: "RGB ENCODER 85"
- note added: "RGB ENCODER 86"
- note added: "RGB ENCODER 87"
- note added: "RGB ENCODER 88"
- note added: "STM32"
- note added: "STM32F446"
- note added: "SWITCH RGB 12"
- note added: "SWITCH RGB 22"
- note added: "SWITCH RGB 32"
- note added: "SWITCH RGB 33"
- note added: "SWITCH RGB 42"
- note added: "SWITCH RGB 43"
- note added: "SWITCH RGB 46"
- note added: "SWITCH RGB 47"
- note added: "SWITCH RGB 52"
- note added: "SWITCH RGB 65"

Commit message: Front pane update
Parts:
- removed I2C1, MIDI: (no value), con-lstb:MA03-1
- removed S3: JOYSTICK_THUMB, stock-perso:JOYSTICK_THUMB
- added CDEC_41A, CDEC_42A, CDEC_5A: 10u, stock-perso:PASSIF-CPOL-US2917
- added CDEC_41B, CDEC_42B, CDEC_5B: 100n, stock-perso:PASSIF-CAP-0805
- added JOYSTICK: (no value), MyComponents:MA05-1PL
- added MCP_41, MCP_42, MCP_5: MCP23017, a_ranger_work:MCP23017
- added R194, R198, R199, R203, R204, R205: 1k, 6P1_EVB:R-US_R0805
- added TFT_EXT, TFT_EXT_2: (no value), con-lstb:MA06-2
Connections:
- new net ENC_01_A: ENC_01.A, RB104.1, TFT_EXT_2.3
- new net ENC_01_B: ENC_01.B, RB105.1, TFT_EXT_2.5
- new net ENC_01_SW: ENC_01.SW, RB106.1, RPD33.1, TFT_EXT_2.6
- new net ENC_02_A: ENC_02.A, RB110.1, TFT_EXT_2.11
- new net ENC_02_B: ENC_02.B, RB111.1, TFT_EXT_2.12
- new net ENC_02_SW: ENC_02.SW, RB112.1, RPD35.1, TFT_EXT_2.4
- new net ENC_03_A: ENC_3.A, RB116.1, TFT_EXT_2.10
- new net ENC_03_B: ENC_3.B, RB117.1, TFT_EXT_2.8
- new net ENC_03_SW: ENC_3.SW, RB118.1, RPD37.1, TFT_EXT_2.2
- new net GPA0_41: MCP_41.GPA0
- new net GPA0_42: ENC_83.A, MCP_42.GPA0, RB38.1
- new net GPA0_5: ENC_74.SW, MCP_5.GPA0, RB94.1, RPD29.1
- new net GPA1_41: MCP_41.GPA1
- new net GPA1_42: ENC_83.B, MCP_42.GPA1, RB39.1
- new net GPA1_5: ENC_74.B, MCP_5.GPA1, RB93.1
- new net GPA2_41: MCP_41.GPA2
- new net GPA2_42: ENC_84.A, MCP_42.GPA2, RB50.1
- new net GPA2_5: ENC_74.A, MCP_5.GPA2, RB92.1
- new net GPA3_41: MCP_41.GPA3
- new net GPA3_42: ENC_84.B, MCP_42.GPA3, RB51.1
- new net GPA3_5: ENC_73.SW, MCP_5.GPA3, RB82.1, RPD25.1
- new net GPA4_41: MCP_41.GPA4
- new net GPA4_42: ENC_84.SW, MCP_42.GPA4, RB52.1, RPD15.1
- new net GPA4_5: ENC_86.A, MCP_5.GPA4, RB74.1
- new net GPA5_41: MCP_41.GPA5
- new net GPA5_42: ENC_85.A, MCP_42.GPA5, RB62.1
- new net GPA5_5: ENC_86.B, MCP_5.GPA5, RB75.1
- new net GPA6_41: MCP_41.GPA6
- new net GPA6_42: ENC_85.B, MCP_42.GPA6, RB63.1
- new net GPA6_5: ENC_86.SW, MCP_5.GPA6, RB76.1, RPD23.1
- new net GPA7_41: MCP_41.GPA7
- new net GPA7_42: ENC_85.SW, MCP_42.GPA7, RB64.1, RPD19.1
- new net GPA7_5: ENC_87.SW, MCP_5.GPA7, RB85.1, RPD26.1
- new net GPB0_41: MCP_41.GPB0
- new net GPB0_42: ENC_73.B, MCP_42.GPB0, RB81.1
- new net GPB0_5: ENC_87.B, MCP_5.GPB0, RB84.1
- new net GPB1_41: MCP_41.GPB1
- new net GPB1_42: ENC_73.A, MCP_42.GPB1, RB80.1
- new net GPB1_5: ENC_87.A, MCP_5.GPB1, RB83.1
- new net GPB2_41: MCP_41.GPB2
- new net GPB2_42: ENC_72.B, MCP_42.GPB2, RB57.1
- new net GPB2_5: ENC_88.SW, MCP_5.GPB2, RB91.1, RPD28.1
- new net GPB3_41: MCP_41.GPB3
- new net GPB3_42: ENC_72.A, MCP_42.GPB3, RB56.1
- new net GPB3_5: ENC_88.A, MCP_5.GPB3, RB89.1
- new net GPB4_41: MCP_41.GPB4
- new net GPB4_42: ENC_72.SW, MCP_42.GPB4, RB58.1, RPD17.1
- new net GPB4_5: ENC_88.B, MCP_5.GPB4, RB90.1
- new net GPB5_41: MCP_41.GPB5
- new net GPB5_42: ENC_71.B, MCP_42.GPB5, RB33.1
- new net GPB5_5: ENC_75.SW, MCP_5.GPB5, RB100.1, RPD31.1
- new net GPB6_41: MCP_41.GPB6
- new net GPB6_42: ENC_71.A, MCP_42.GPB6, RB32.1
- new net GPB6_5: ENC_75.A, MCP_5.GPB6, RB98.1
- new net GPB7_41: MCP_41.GPB7
- new net GPB7_42: ENC_71.SW, MCP_42.GPB7, RB34.1, RPD9.1
- new net GPB7_5: ENC_75.B, MCP_5.GPB7, RB99.1
- new net INTA_41: MCP_41.INTA
- new net INTA_42: MCP_42.INTA
- new net INTA_5: MCP_5.INTA
- new net INTB_41: MCP_41.INTB
- new net INTB_42: MCP_42.INTB
- new net INTB_5: MCP_5.INTB
- new net JOY_SEL: JOYSTICK.2
- new net JOY_XOUT: JOYSTICK.4
- new net JOY_YOUT: JOYSTICK.3
- new net N$1: TFT_EXT.10, TFT_EXT.11, TFT_EXT.12, TFT_EXT.2, TFT_EXT.3, TFT_EXT.4, TFT_EXT.5, TFT_EXT.6, TFT_EXT.8
- new net PIXEL_IN: PIXEL_03.SDI, TFT_EXT_2.9
- net 3V3: now also CDEC_41A.+, CDEC_41B.1, CDEC_42A.+, CDEC_42B.1, CDEC_5A.+, CDEC_5B.1, JOYSTICK.5, MCP_31.A0, MCP_32.A2, MCP_41.A0, MCP_41.A2, MCP_41.VDD, MCP_42.A1, MCP_42.A2, MCP_42.VDD, MCP_5.A1, MCP_5.A2, MCP_5.VDD, R194.2, R198.2, R199.2, R203.2, R204.2, R205.2, TFT_EXT.1, TFT_EXT_2.1; no longer MCP_32.A1
- net GND: now also CDEC_41A.-, CDEC_41B.2, CDEC_42A.-, CDEC_42B.2, CDEC_5A.-, CDEC_5B.2, JOYSTICK.1, MCP_32.A1, MCP_41.A1, MCP_41.VSS, MCP_42.A0, MCP_42.VSS, MCP_5.A0, MCP_5.VSS, TFT_EXT.7, TFT_EXT_2.7; no longer I2C1.3, MCP_31.A0, MCP_32.A2, MIDI.3
- net GP: no longer ENC_01.SW, ENC_02.SW, ENC_3.SW, ENC_71.SW, ENC_72.SW, ENC_73.SW, ENC_74.SW, ENC_75.SW, ENC_84.SW, ENC_85.SW, ENC_86.SW, ENC_87.SW, ENC_88.SW, RB100.1, RB106.1, RB112.1, RB118.1, RB34.1, RB52.1, RB58.1, RB64.1, RB76.1, RB82.1, RB85.1, RB91.1, RB94.1, RPD15.1, RPD17.1, RPD19.1, RPD23.1, RPD25.1, RPD26.1, RPD28.1, RPD29.1, RPD31.1, RPD33.1, RPD35.1, RPD37.1, RPD9.1
- net GPA: no longer ENC_01.A, ENC_02.A, ENC_3.A, ENC_71.A, ENC_72.A, ENC_73.A, ENC_74.A, ENC_75.A, ENC_83.A, ENC_84.A, ENC_85.A, ENC_86.A, ENC_87.A, ENC_88.A, RB104.1, RB110.1, RB116.1, RB32.1, RB38.1, RB50.1, RB56.1, RB62.1, RB74.1, RB80.1, RB83.1, RB89.1, RB92.1, RB98.1
- net GPB: no longer ENC_01.B, ENC_02.B, ENC_3.B, ENC_71.B, ENC_72.B, ENC_73.B, ENC_74.B, ENC_75.B, ENC_83.B, ENC_84.B, ENC_85.B, ENC_86.B, ENC_87.B, ENC_88.B, RB105.1, RB111.1, RB117.1, RB33.1, RB39.1, RB51.1, RB57.1, RB63.1, RB75.1, RB81.1, RB84.1, RB90.1, RB93.1, RB99.1
- net I2C1_SCL: no longer I2C1.2
- net I2C1_SDA: no longer I2C1.1
- net I2C3_SCL: now also MCP_41.SCL, MCP_42.SCL, MCP_5.SCL, R194.1, R199.1, R204.1
- net I2C3_SDA: now also MCP_41.SDA, MCP_42.SDA, MCP_5.SDA, R198.1, R203.1, R205.1
- net PIXEL_81: now also TFT_EXT.9; no longer PIXEL_03.SDI
- net RST: now also MCP_41.!RESET, MCP_42.!RESET, MCP_5.!RESET
- net USART1_RX: no longer MIDI.1
- net USART1_TX: no longer MIDI.2
Other:
- note added: "MCP 41 & 42"
- note added: "MODULATION"
- note added: "TFT EXTENSION"
- note removed: "LFO"
- note removed: "STM32"

Commit message: Finished front pane and sent to production
Parts:
- removed JOYSTICK: (no value), MyComponents:MA05-1PL
- added ANALOG_IN: (no value), con-lstb:MA04-1
- added CONN_STH_BRD_1, CONN_STH_BRD_2: (no value), MyComponents:MA10-2
- added UART_ANALOG, UART_DISCO, UART_MIDI: (no value), con-lstb:MA03-1
- renumbered 3V3 to LED_3V3, 5V to LED_5V, MCP_11 to MCP_000, MCP_12 to MCP_001, MCP_2 to MCP_010, MCP_31 to MCP_011, MCP_32 to MCP_100, MCP_41 to MCP_101, MCP_42 to MCP_110, MCP_5 to MCP_111
Connections:
- removed net DATA_PIXEL31: PIXEL_31.SDO
- removed net GP: ENC_54.SW, ENC_61.SW, ENC_62.SW, ENC_63.SW, ENC_64.SW, ENC_81.SW, ENC_82.SW, ENC_83.SW, RB22.1, RB28.1, RB40.1, RB55.1, RB61.1, RB67.1, RB73.1, RB79.1, RPD11.1, RPD16.1, RPD18.1, RPD20.1, RPD22.1, RPD24.1, RPD5.1, RPD7.1
- removed net GPA: ENC_54.A, ENC_61.A, ENC_62.A, ENC_63.A, ENC_64.A, ENC_81.A, ENC_82.A, RB20.1, RB26.1, RB44.1, RB53.1, RB59.1, RB65.1, RB71.1, RB77.1, SW_65.3, SW_65.4
- removed net GPB: ENC_54.B, ENC_61.B, ENC_62.B, ENC_63.B, ENC_64.B, ENC_81.B, ENC_82.B, RB21.1, RB27.1, RB54.1, RB60.1, RB66.1, RB72.1, RB78.1
- removed net GPB0_12: MCP_001.GPB0
- removed net INTA_41: MCP_101.INTA
- removed net INTA_42: MCP_110.INTA
- removed net INTA_5: MCP_111.INTA
- removed net INTB_41: MCP_101.INTB
- removed net INTB_42: MCP_110.INTB
- removed net INTB_5: MCP_111.INTB
- removed net JOY_SEL: JOYSTICK.2
- removed net JOY_XOUT: JOYSTICK.4
- removed net JOY_YOUT: JOYSTICK.3
- removed net N$1: TFT_EXT.10, TFT_EXT.11, TFT_EXT.12, TFT_EXT.2, TFT_EXT.3, TFT_EXT.4, TFT_EXT.5, TFT_EXT.6, TFT_EXT.8
- removed net PIXEL_01: PIXEL_01.SDO
- removed net PIXEL_65: PIXEL_65.SDO
- removed net SPI1_SCK: F446.PA5
- removed net SPI2_SCK: F446.PB13
- removed net SPI3_SCK: F446.PC10
- new net GPIO_EXTI0: F446.PH0-OSC_IN, MCP_101.INTB
- new net GPIO_EXTI13: F446.PC13, MCP_101.INTA
- net 3V3: now also CONN_STH_BRD_1.2, CONN_STH_BRD_1.4, CONN_STH_BRD_2.2, CONN_STH_BRD_2.4, MCP_111.A0; no longer JOYSTICK.5
- net ADC1_IN1: now also ANALOG_IN.4
- net ADC1_IN10: now also ANALOG_IN.2
- net ADC1_IN4: now also ANALOG_IN.3
- net GND: now also ANALOG_IN.1, CONN_STH_BRD_1.1, CONN_STH_BRD_2.1, UART_ANALOG.1, UART_DISCO.1, UART_MIDI.1; no longer JOYSTICK.1, MCP_111.A0
- net GPA0_32: now also RB44.1, SW_65.3, SW_65.4
- net GPA0_41: now also ENC_81.SW, RB79.1, RPD24.1
- net GPA1_32: now also ENC_64.SW, RB73.1, RPD22.1
- net GPA1_41: now also ENC_82.SW, RB22.1, RPD5.1
- net GPA2_32: now also ENC_64.B, RB72.1
- net GPA2_41: now also ENC_82.A, RB20.1
- net GPA3_32: now also ENC_64.A, RB71.1
- net GPA3_41: now also ENC_82.B, RB21.1
- net GPA4_32: now also ENC_63.SW, RB67.1, RPD20.1
- net GPA4_41: now also ENC_83.SW, RB40.1, RPD11.1
- net GPA5_32: now also ENC_63.B, RB66.1
- net GPA5_41: now also TFT_EXT.5
- net GPA6_32: now also ENC_63.A, RB65.1
- net GPA6_41: now also TFT_EXT.3
- net GPA7_32: now also ENC_62.SW, RB61.1, RPD18.1
- net GPA7_41: now also TFT_EXT.2
- net GPB0_32: now also ENC_62.B, RB60.1
- net GPB0_41: now also TFT_EXT.11
- net GPB1_32: now also ENC_62.A, RB59.1
- net GPB1_41: now also TFT_EXT.12
- net GPB2_32: now also ENC_61.B, RB54.1
- net GPB2_41: now also TFT_EXT.10
- net GPB3_32: now also ENC_61.A, RB53.1
- net GPB3_41: now also TFT_EXT.8
- net GPB4_32: now also ENC_61.SW, RB55.1, RPD16.1
- net GPB4_41: now also TFT_EXT.6
- net GPB5_32: now also ENC_54.A, RB26.1
- net GPB5_41: now also TFT_EXT.4
- net GPB6_32: now also ENC_54.B, RB27.1
- net GPB6_41: now also ENC_81.A, RB77.1
- net GPB7_32: now also ENC_54.SW, RB28.1, RPD7.1
- net GPB7_41: now also ENC_81.B, RB78.1
- net GPIO_EXTI1: now also CONN_STH_BRD_1.17
- net GPIO_EXTI10: now also CONN_STH_BRD_1.10
- net GPIO_EXTI11: now also CONN_STH_BRD_1.7
- net GPIO_EXTI12: now also CONN_STH_BRD_1.8
- net GPIO_EXTI14: now also CONN_STH_BRD_1.18
- net GPIO_EXTI15: now also CONN_STH_BRD_1.15
- net GPIO_EXTI2: now also MCP_110.INTB
- net GPIO_EXTI3: now also MCP_110.INTA
- net GPIO_EXTI4: now also MCP_111.INTA
- net GPIO_EXTI5: now also MCP_111.INTB
- net GPIO_EXTI6: now also CONN_STH_BRD_1.16
- net GPIO_EXTI7: now also CONN_STH_BRD_1.13
- net GPIO_EXTI8: now also CONN_STH_BRD_1.14
- net GPIO_EXTI9: now also CONN_STH_BRD_1.9
- net I2C1_SCL: now also MCP_101.SCL, MCP_110.SCL, MCP_111.SCL, R194.1, R199.1, R204.1; no longer MCP_000.SCL, MCP_001.SCL, R186.1, R4.1
- net I2C1_SDA: now also MCP_101.SDA, MCP_110.SDA, MCP_111.SDA, R198.1, R203.1, R205.1; no longer MCP_000.SDA, MCP_001.SDA, R187.1, R5.1
- net I2C2_SCL: now also CONN_STH_BRD_1.20, CONN_STH_BRD_2.20
- net I2C2_SDA: now also CONN_STH_BRD_1.5, CONN_STH_BRD_2.5
- net I2C3_SCL: now also CONN_STH_BRD_1.12, CONN_STH_BRD_2.12, MCP_000.SCL, MCP_001.SCL, R186.1, R4.1; no longer MCP_101.SCL, MCP_110.SCL, MCP_111.SCL, R194.1, R199.1, R204.1
- net I2C3_SDA: now also CONN_STH_BRD_1.11, CONN_STH_BRD_2.11, MCP_000.SDA, MCP_001.SDA, R187.1, R5.1; no longer MCP_101.SDA, MCP_110.SDA, MCP_111.SDA, R198.1, R203.1, R205.1
- net INTA_11: now also CONN_STH_BRD_2.8
- net INTA_12: now also CONN_STH_BRD_2.9
- net INTA_2: now also CONN_STH_BRD_2.13
- net INTA_31: now also CONN_STH_BRD_2.18
- net INTA_32: now also CONN_STH_BRD_2.15
- net INTB_11: now also CONN_STH_BRD_2.7
- net INTB_12: now also CONN_STH_BRD_2.10
- net INTB_2: now also CONN_STH_BRD_2.14
- net INTB_31: now also CONN_STH_BRD_2.17
- net INTB_32: now also CONN_STH_BRD_2.16
- net RST: now also CONN_STH_BRD_1.3, CONN_STH_BRD_2.3
- net SPI1_MOSI: now also CONN_STH_BRD_1.6, CONN_STH_BRD_2.6
- net SPI2_MOSI: now also PIXEL_71.SDI; no longer PIXEL_51.SDI
- net SPI3_MOSI: now also CONN_STH_BRD_1.19, CONN_STH_BRD_2.19, PIXEL_51.SDI; no longer PIXEL_71.SDI
- net UART4_RX: now also UART_ANALOG.2
- net UART4_TX: now also UART_ANALOG.3
- net USART1_RX: now also UART_DISCO.2
- net USART1_TX: now also UART_DISCO.3
- net USART2_RX: now also UART_MIDI.2
- net USART2_TX: now also UART_MIDI.3
Other:
- moved on the sheet: RB2
