File: front-pane/eagle-schematics/v3/STM32F446 front pane - south - v3.brd (EAGLE design)
At the start: 370 x 140 mm, 435 parts, among them IC1 NEOPIXEL-TLC59731DR, IC10 NEOPIXEL-TLC59731DR, IC11 NEOPIXEL-TLC59731DR, IC12 NEOPIXEL-TLC59731DR, IC13 NEOPIXEL-TLC59731DR, IC14 NEOPIXEL-TLC59731DR, IC15 NEOPIXEL-TLC59731DR, IC16 NEOPIXEL-TLC59731DR, IC17 NEOPIXEL-TLC59731DR, IC18 NEOPIXEL-TLC59731DR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

Commit message: Fixed bug with MCP_XXX name
Parts:
- renumbered MCP_101 to MCP_010
