File: front-pane/eagle-schematics/v3/STM32F446 front pane - v3.1.brd (EAGLE design)
At the start: 450 x 300 mm, 707 parts

Commit message: added graphism proposal
Parts:
- moved RB104 10.0 mm to (53.6, 262.6)
- moved RB110 10.0 mm to (83.7, 262.6)
- moved RB116 10.0 mm to (113.7, 262.6)
- moved RB20 10.0 mm to (228.7, 262.6)
- moved RB38 10.0 mm to (258.6, 262.6)
- moved RB50 10.0 mm to (288.6, 262.6)
- moved RB62 10.0 mm to (318.6, 262.6)
- moved RB74 10.0 mm to (348.6, 262.6)
- moved RB77 10.0 mm to (198.7, 262.6)
- moved RB83 10.0 mm to (378.6, 262.6)
- moved RB89 10.0 mm to (408.6, 262.6)
- moved 0V/5V 10.0 mm to (245.1, 246.8)
- moved ANALOG_IN 10.0 mm to (205.0, 215.0)
- moved C55 10.0 mm to (236.1, 240.9)
- moved C60 10.0 mm to (246.5, 229.2)
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Other:
- board size 450 x 300 mm -> 405 x 260 mm
- board text added: "JOYSTICK"
- board text added: "Touchscreen"

Commit message: Slight translation of touch screen
This doesn't have any consequence on the electrical design
Parts:
- moved TFT_EXT_2 109.0 mm to (29.6, 287.3), turned to 0 degrees
- moved RB118 104.0 mm to (18.3, 271.9), turned to 270 degrees
- moved CDEC37 103.2 mm to (27.8, 280.7), turned to 180 degrees
- moved CB118 99.2 mm to (18.2, 266.2), turned to 270 degrees
- moved R197 98.1 mm to (25.4, 273.6), turned to 270 degrees
- moved RPD37 96.9 mm to (20.6, 266.7), turned to 270 degrees
- moved CB117 94.2 mm to (33.8, 277.4), turned to 90 degrees
- moved R196 92.8 mm to (25.4, 268.0), turned to 270 degrees
- moved CPOL37 90.6 mm to (34.1, 274.3), turned to 180 degrees
- moved RB117 90.5 mm to (37.5, 276.9), turned to 90 degrees
- moved ENC_3 90.0 mm to (30.0, 270.0), turned to 90 degrees
- moved R195 89.2 mm to (25.2, 263.6), turned to 0 degrees
- moved PIXEL_03 88.2 mm to (31.8, 270.0), turned to 180 degrees
- moved CB106 84.6 mm to (18.2, 206.2), turned to 270 degrees
- moved RB112 83.7 mm to (18.3, 241.9), turned to 270 degrees
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Other:
- board size 405 x 260 mm -> 500 x 300 mm
- board text added: "RAINBOW by SYD X. REY (c) 2022"
- board text removed: "RAINBOW by SYD X. REY (c) 2021"
