File: main-board/v2.0/eagle-schematics/STM32F446 Full Board SMD v7.brd (EAGLE design)
At the start: 101.3 x 99.1 mm, 275 parts, among them Q1 16MHz

Commit message: Added missing net label on BH2221 DAC
Connections:
- net N$23 renamed BH2221_AO5
Changed lines of the file:
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@@
 <wire x1="51.816" y1="22.1821875" x2="51.816" y2="16.764" width="0.254" layer="1"/>
 </signal>
-<signal name="N$23">
+<signal name="BH2221_AO5">
 <contactref element="A010/9/8/7/3/4/5/6" pad="7"/>
 <contactref element="BH2221" pad="4"/>

Commit message: pointing new errors on the board layout
Connections:
- net N$34 renamed AD5644_A
- net N$35 renamed AD5644_B
- net N$39 renamed AD5644_C
- net N$40 renamed AD5644_D
Changed lines of the file:
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@@
 <wire x1="39.624" y1="32.512" x2="39.624" y2="34.29" width="0.3048" layer="1"/>
 </signal>
-<signal name="N$34">
+<signal name="AD5644_A">
 <contactref element="AD5644" pad="1"/>
 <contactref element="ABCD" pad="1"/>
@@
 <wire x1="37.846" y1="62.992" x2="36.322" y2="64.516" width="0.254" layer="1"/>
 </signal>
-<signal name="N$35">
+<signal name="AD5644_B">
 <contactref element="ABCD" pad="2"/>
 <contactref element="AD5644" pad="2"/>
@@
 <wire x1="36.98" y1="60.81" x2="35.814" y2="61.976" width="0.254" layer="1"/>
 </signal>
-<signal name="N$39">
+<signal name="AD5644_C">
 <contactref element="AD5644" pad="4"/>
 <contactref element="ABCD" pad="3"/>
@@
 <wire x1="35.306" y1="59.436" x2="34.29" y2="59.436" width="0.254" layer="1"/>
 </signal>
-<signal name="N$40">
+<signal name="AD5644_D">
 <contactref element="ABCD" pad="4"/>
 <contactref element="AD5644" pad="5"/>
